File: kicker/kicker-v2.2/kicker-v2.2.brd (EAGLE design)
At the start: 152.8 x 55 mm, 53 parts, among them IC1 7818TV, IC2 MCP601OT, J1 XT-60BATT_LABEL, Q1 IGB50N60T, Q3 IGB50N60T, U1 LT3750EMSPBF, U2 ATMEGA328P-AU

Commit message: Completed Circuit
Routing:
- net GND: track 3.18 -> 10.4 mm, vias 0 -> 1
Changed lines of the file:
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@@
 <contactref element="R14" pad="1"/>
 <contactref element="IC2" pad="2"/>
-<wire x1="-29.44" y1="0.63" x2="-28.5748" y2="-3.5036" width="0" layer="19" extent="1-16"/>
+<wire x1="-28.5748" y1="-3.5036" x2="-30.4464" y2="-3.5036" width="0.3" layer="16"/>
+<wire x1="-30.4464" y1="-3.5036" x2="-31.35" y2="-2.6" width="0.3" layer="16"/>
+<via x="-31.35" y="-2.6" extent="1-16" drill="0.5"/>
+<wire x1="-31.35" y1="-2.6" x2="-31.35" y2="-1.28" width="0.3" layer="1"/>
+<wire x1="-31.35" y1="-1.28" x2="-29.44" y2="0.63" width="0.3" layer="1"/>
 </signal>
 <signal name="N$4">
@@
 <wire x1="-32.2" y1="3.55" x2="-32.2" y2="-1.45" width="0.4064" layer="1"/>
 <wire x1="-32.2" y1="-1.45" x2="-32.7" y2="-1.95" width="0.4064" layer="1"/>
-<via x="-32.7" y="-1.95" extent="1-16" drill="0.6" shape="square"/>
+<via x="-32.7" y="-1.95" extent="1-16" drill="0.6"/>
 <wire x1="-32.7" y1="-1.95" x2="-41.62" y2="-1.95" width="0.4064" layer="16"/>
 <wire x1="-41.62" y1="-1.95" x2="-47.76" y2="4.19" width="0.4064" layer="16"/>
@@
 <wire x1="-24.4" y1="-3.2" x2="-31" y2="-3.2" width="0.2" layer="1"/>
 <wire x1="-31" y1="-3.2" x2="-31.9" y2="-4.1" width="0.2" layer="1"/>
-<via x="-31.9" y="-4.1" extent="1-16" drill="0.6" shape="square"/>
+<via x="-31.9" y="-4.1" extent="1-16" drill="0.6"/>
 <wire x1="-31.9" y1="-4.1" x2="-44.75" y2="-4.1" width="0.2" layer="16"/>
 <wire x1="-44.75" y1="-4.1" x2="-44.75" y2="-3.9" width="0.2" layer="16"/>
@@
 <wire x1="-16.75" y1="-4.6" x2="-21.7" y2="-4.6" width="0.2" layer="1"/>
 <wire x1="-21.7" y1="-4.6" x2="-23.65" y2="-2.65" width="0.2" layer="1"/>
-<via x="-26.45" y="-1.65" extent="1-16" drill="0.6" shape="square"/>
+<via x="-26.45" y="-1.65" extent="1-16" drill="0.6"/>
 <wire x1="-26.45" y1="-1.65" x2="-26.85" y2="-1.65" width="0.2" layer="16"/>
 <wire x1="-26.85" y1="-1.65" x2="-27.3" y2="-1.2" width="0.2" layer="16"/>
