File: motor_driver/uc2950-v1/uc2950-v1.sch (EAGLE design)
At the start: 76 parts, among them IC1 ATMEGA2560-16AU, IC2 ATMEGA2560-16AU, IC3 ATMEGA2560-16AU, IC4 ACS712, IC5 ACS712, IC6 ACS712, Y2 16MHz, Y3 16MHz, Y4 16MHz

Commit message: added 12v, fixed previous issues
Parts:
- added C1: 10uF, SparkFun-Capacitors:10UF-POLAR-0603-6.3V-20%(TANT)
- added D1: Yellow, SparkFun-LED:LED-YELLOW0603
- added R1: 1k, SparkFun-Resistors:1KOHM-0603-1/10W-1%
Connections:
- removed net N$11: C2.1, IC1.AREF
- removed net N$24: C3.1, IC3.AREF
- removed net N$26: C14.1, IC2.AREF
- new net 12V: C1.+, D1.A, IC5.I+_0, IC5.I+_1, JP1.16
- new net N$1: D1.C, R1.1
- net 18V: now also IC4.I+_1, IC6.I+_1; no longer IC5.I+_0
- net 5V: now also C14.1, C2.1, C3.1, IC1.AREF, IC2.AREF, IC3.AREF
- net ACS1: now also IC4.I-_1, MIC1.P$5, MIC2.P$5, MIC3.P$5; no longer MIC1.P$1, MIC2.P$1, MIC3.P$1
- net ACS2: now also IC5.I-_1, MIC4.P$5, MIC5.P$5, MIC6.P$5; no longer MIC4.P$1, MIC5.P$1, MIC6.P$1
- net ACS3: now also IC6.I-_1, MIC7.P$5, MIC8.P$5, MIC9.P$5; no longer MIC7.P$1, MIC8.P$1, MIC9.P$1
- net GND: now also C1.-, R1.2
- net M11: now also MIC3.P$2; no longer MIC3.P$4
- net M12: now also MIC6.P$2; no longer MIC6.P$4
- net M13: now also MIC7.P$2; no longer MIC7.P$4
- net M21: now also MIC2.P$2; no longer MIC2.P$4
- net M22: now also MIC5.P$2; no longer MIC5.P$4
- net M23: now also MIC8.P$2; no longer MIC8.P$4
- net M31: now also MIC1.P$2; no longer MIC1.P$4
- net M32: now also MIC4.P$2; no longer MIC4.P$4
- net M33: now also MIC9.P$2; no longer MIC9.P$4
- net MISO: now also JP2.1, JP3.1, JP4.1; no longer JP2.3, JP3.3, JP4.3
- net MISO1: now also JP2.2; no longer JP2.4
- net MISO2: now also JP3.2; no longer JP3.4
- net MISO3: now also JP4.2; no longer JP4.4
- net MOSI: now also JP2.3, JP3.3, JP4.3; no longer JP2.1, JP3.1, JP4.1
- net MOSI1: now also JP2.4; no longer JP2.2
- net MOSI2: now also JP3.4; no longer JP3.2
- net MOSI3: now also JP4.4; no longer JP4.2
- net S11: now also MIC3.P$4; no longer MIC3.P$2
- net S12: now also MIC6.P$4; no longer MIC6.P$2
- net S13: now also MIC7.P$4; no longer MIC7.P$2
- net S21: now also MIC3.P$1; no longer MIC3.P$5
- net S22: now also MIC6.P$1; no longer MIC6.P$5
- net S23: now also MIC7.P$1; no longer MIC7.P$5
- net S31: now also MIC2.P$4; no longer MIC2.P$2
- net S32: now also MIC5.P$4; no longer MIC5.P$2
- net S33: now also MIC8.P$4; no longer MIC8.P$2
- net S41: now also MIC2.P$1; no longer MIC2.P$5
- net S42: now also MIC5.P$1; no longer MIC5.P$5
- net S43: now also MIC8.P$1; no longer MIC8.P$5
- net S51: now also MIC1.P$4; no longer MIC1.P$2
- net S52: now also MIC4.P$4; no longer MIC4.P$2
- net S53: now also MIC9.P$4; no longer MIC9.P$2
- net S61: now also MIC1.P$1; no longer MIC1.P$5
- net S62: now also MIC4.P$1; no longer MIC4.P$5
- net S63: now also MIC9.P$1; no longer MIC9.P$5
