File: main_board/main_board-v2.2/main_board-v2.2.brd (EAGLE design)
At the start: 174.2 x 59 mm, 59 parts, among them J1 XT-60BATT_LABEL, J2 F-1X02-SIP-100-32Y, J3 F-1X02-SIP-100-32Y, J4 F-1X08-SIP-100-32Y, T1 2N706

Commit message: Completed
Parts:
- 12V, 3.3V, 5V, BATTERY: device led:CHIPLED_1206 -> led:CHIPLED_0805
- moved TP5 109.7 mm to (-71.1, -3.89)
- moved TP4 106.5 mm to (-68.6, -1.34)
- moved TP3 99.2 mm to (-71.1, -1.34)
- moved TP10 56.2 mm to (-68.6, -8.99)
- moved TP9 51.2 mm to (-71.1, -8.96)
- moved TP8 47.7 mm to (-68.6, -6.41)
- moved TP7 44.3 mm to (-71.2, -6.46)
- moved TP6 41.0 mm to (-68.6, -3.91)
- moved R15 0.45 mm to (3.56, 11.8)
Routing:
- net 5V: track 102.3 -> 262.9 mm, vias 1 -> 6
- net SCK: track 0.00 -> 121.6 mm, vias 0 -> 2
- net SDA: track 0.00 -> 114.3 mm, vias 0 -> 3
- net CE: track 0.00 -> 102.8 mm, vias 0 -> 1
- net CSN: track 0.00 -> 98.3 mm, vias 0 -> 2
- net 3.3V: track 318.6 -> 416.7 mm, vias 1 -> 6
- net GND: track 198.0 -> 292.1 mm, vias 2 -> 5
- net SCL: track 0.00 -> 93.4 mm, vias 0 -> 2
- net MOSI_MOTOR: track 0.00 -> 92.0 mm, vias 0 -> 3
- net MISO: track 0.00 -> 87.7 mm, vias 0 -> 2
- net MOSI: track 0.00 -> 86.1 mm, vias 0 -> 3
- net SS4: track 0.00 -> 74.9 mm, vias 0 -> 3
- net RST5: track 9.00 -> 77.9 mm, vias 0 -> 2
- net MISO_MOTOR: track 0.00 -> 61.8 mm, vias 0 -> 3
- net RST2: track 0.00 -> 61.5 mm, vias 0 -> 1
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- added copper zone on layer 15, net 12V
- added copper zone on layer 15, net GND
- added copper zone on layer 2, net VDC_1
- added copper zone on layer 2, net VDC_2
