File: kicker/kicker-v2.1/kicker-v2.1.sch (EAGLE design)
At the start: 86 parts, among them IC1 MEGA8-AI, J1 1X2-3.5MM, J2 1X2-3.5MM, J3 XT-60BATT_LABEL, J4 1X2-3.5MM, J5 1X2-3.5MM, J6 1X2-3.5MM, J7 1X2-3.5MM, Q3 16MHz, T1 BC547, T2 BC547

Commit message: Kicker proto
Parts:
- removed !RESET: (no value), switch-omron:10-XX
- removed 5V, GND, GND12, GND_12V1, GND_5V, POWER_1, POWER_HEAD1, V_BAT: PINHEAD_1, pinhead_1:PINHEAD_1
- removed C1, C10, C11, C6, C8, C9: 0.01uF, rcl:C-EUC1206
- removed C12: 0.1uF, rcl:C-EUC1206
- removed C13, C14: 22pF, rcl:C-EUC1206
- removed C3: 4.7uF, rcl:C-EUC1206
- removed C4: 4.7uF, rcl:CPOL-EUE2.5-6
- removed D1, D2, DS, DS1: UF5400, diode-1:UF5400
- removed D3, D5: 1N4446, diode:1N4446
- removed FHEADER1, FHEADER4: F-1X04-SIP-100-32Y, con-headers-jp:F-1X04-SIP-100-32Y
- removed IGBT, MOSFET: NE555, st-microelectronics:NE555
- removed J1, J2, J4, J5, J6, J7: 1X2-3.5MM, adafruit:1X2-3.5MM
- removed J3: XT-60BATT_LABEL, RoboJackets-Connectors:XT-60BATT_LABEL
- removed LED_5V, LED_BATT, LED_TEST: (no value), led:LEDSML1206
- removed R10, R12, R4: 10K, resistor:R-EU_R1206
- removed R11, R6: 330, resistor:R-EU_R1206
- removed R13, R9: 1 K, adafruit:FLIPFLOP-RES
- removed R14, R15: 4.7 K, adafruit:FLIPFLOP-RES
- removed R7, RD2: 8.2K, resistor:R-EU_R1206
- removed R8, RD1: 1M, resistor:R-EU_R1206
- removed RS, RS1: 10/.5W, rcl:R-US_0411/15
- removed R_RELAY, R_RELAY1: 1K, resistor:R-EU_R1206
- removed S1, S2: (no value), switch:A68-A31
- removed SV5: (no value), con-lsta:FE06-1
- removed SV6: (no value), con-lsta:FE08-1
- removed T2: BC547, transistor:BC547
- removed U$10, U$11, U$12, U$13: REL, rel:REL
- removed U$16: SCREW, screw:SCREW
- removed U$7, U$8: POLYCAP, polycap:POLYCAP
- removed U$9: MOS, mosfet:MOS
- removed U4: (no value), LP38690DT-3.3:LP38690DT-3.3
- added C16, C2, C20: (no value), rcl:C-EUC1206
- added D4: (no value), diode:DIODE-DO214AA
- added IC2: AD7992, analog_devices_gaui:AD7992
- added IC4: NE555, st-microelectronics:NE555
- added J8: 1X2-3.5MM, adafruit:1X2-3.5MM
- added J9: XT-60BATT_LABEL, RoboJackets-Connectors:XT-60BATT_LABEL
- added JP1, JP2: (no value), adafruit:PINHD-1X3
- added Q2: SPB80P06P, transistor-fet:SPB80P06P
- added R16, R17, R18, R20: (no value), adafruit:R-US_R1206
- added R19: (no value), resistor:R-US_R1206
- added R21: 4.7 K, resistor:R-EU_0207/10
- added S3: (no value), switch:A68-A31
- added U$15: DA2033-AL, inductor-coilcraft-2:DA2033-AL
- added U$17: (no value), Electrolytic-Cap:CAPS
- added X1, X2: (no value), con-wago-500:W237-102
- IC1: value MEGA8-AI -> NE555; device atmel:MEGA8-AI -> st-microelectronics:NE555
- Q3: value 16MHz -> SPB80P06P; device crystal:CRYSTALHC49U70 -> transistor-fet:SPB80P06P
- R1, R3: value 1K -> (none); device resistor:R-EU_R1206 -> adafruit:R-US_R1206
- R2: value 10K -> (none); device resistor:R-EU_R1206 -> adafruit:R-US_R1206
- R5: value 10K -> 4.7 K; device resistor:R-EU_R1206 -> resistor:R-EU_0207/10
- T1: value BC547 -> (none); device transistor:BC547 -> transistor-neu-to92:-NPN-SOT223
- U$1: value DA2033-AL -> CAP; device inductor-coilcraft-2:DA2033-AL -> SVP_F12:CAP
- U$3: value MOS -> CAP; device mosfet:MOS -> SVP_F12:CAP
- U$4: value (none) -> CAP; device Electrolytic-Cap:CAPS -> SVP_F12:CAP
- U$5: value DA2033-AL -> MOSFET-LT3750; device inductor-coilcraft-2:DA2033-AL -> SON-8:MOSFET-LT3750
- U$6: value SCREW -> TC4426A; device screw:SCREW -> smd-footprints:TC4426A
Connections:
- removed net !RESET: !RESET.S, !RESET.S1, IC1.PC6(/RESET), R12.1, SV6.4
- removed net ATMEGA_POW: C12.2, D3.C, D5.C, IC1.AREF, IC1.AVCC, IC1.VCC@1, IC1.VCC@2, R12.2, R13.1, S2A.S, S2B.S, SV5.2, SV6.5, U$10.2, U$11.2, U$12.2, U$13.2
- removed net ATMEGA_POW_BS: 5V.P$1, S2A.P, S2B.P
- removed net BATT: C3.1, C4.+, IGBT.TRE, MOSFET.TRE, R14.1, S1A.S, S1B.S, U$1.10, U$1.7, U$1.8, U$1.9, U$5.10, U$5.7, U$5.8, U$5.9
- removed net C1+: D1.C, J2.1, RD1.2, U$16.+, U$2.P$2, U$6.+
- removed net C1-: D2.C, J1.1, J2.2, R8.2, U$1.1, U$2.P$1, U$4.P$2
- removed net COLLECTOR: D3.A, T1.C, U$10.1, U$12.1
- removed net COLLECTOR1: D5.A, T2.C, U$11.1, U$13.1
- removed net DRV_IN: J6.2, R6.1
- removed net DRV_IN1: J4.2, R11.1
- removed net EXT1: IC1.PD2(INT0), SV5.3
- removed net EXT2: IC1.PD3(INT1), SV5.4
- removed net FEED1: C9.1, IC1.PC1(ADC1), RD1.1, RD2.2
- removed net FEED2: C8.1, IC1.PC2(ADC2), R7.2, R8.1
- removed net GND1: GND.P$1, LED_5V.C, LED_TEST.C
- removed net GPIO: IC1.PD4(XCK/T0), SV5.5
- removed net GPIO1: IC1.PD5(T1), SV5.6
- removed net IGBT1: FHEADER1.2, IGBT.TRI
- removed net IGBT2: FHEADER4.2, IGBT./RES
- removed net MISO16: IC1.PB4(MISO), SV6.7
- removed net MOS1: IC1.PB2(SS/OC1B), MOSFET.TRI, R2.2
- removed net MOS2: IC1.PB1(OC1A), MOSFET./RES, R4.2
- removed net MOSI15: IC1.PB3(MOSI/OC2), SV6.8
- removed net N$11: R_RELAY1.2, T2.B
- removed net N$12: LED_BATT.A, R14.2
- removed net N$14: C13.2, IC1.PB6(XTAL1/TOSC1), Q3.2
- removed net N$15: LED_12V.A, R15.2
- removed net N$16: U4.K, V_BAT.P$1
- removed net N$17: C14.2, IC1.PB7(XTAL2/TOSC2), Q3.1
- removed net N$19: LED_TEST.A, R9.2
- removed net N$21: U$5.3, U$5.4, U$5.5, U$5.6, U$9.P$1
- removed net N$22: U$1.3, U$1.4, U$1.5, U$1.6, U$3.P$1
- removed net N$23: IC1.PB0(ICP), R9.1
- removed net N$6: LED_5V.A, R13.2
- removed net N$7: POWER_HEAD1.P$1, U1.K
- removed net N$8: D1.A, U$1.12
- removed net N$9: DS1.C, RS1.1, U$8.1
- removed net NC: IGBT.GND, IGBT.VCC+, MOSFET.GND, MOSFET.VCC+
- removed net OUTB: C1.1, IGBT.CON, R10.2, R11.2
- removed net POWER: POWER_1.P$1, R15.1, S1A.P, S1B.P
- removed net PWM1: C11.1, MOSFET.DIS, R1.2, U$3.P$2
- removed net PWM2: C10.1, MOSFET.CON, R3.2, U$9.P$2
- removed net RELAY: FHEADER1.4, R_RELAY.1
- removed net RELAY1: FHEADER4.4, R_RELAY1.1
- removed net RXD30: IC1.PD0(RXD), SV6.3
- removed net S+: DS.A, J6.1, RS.2, U$10.NO, U$12.NO, U$16.-
- removed net S1+: DS1.A, J4.1, RS1.2, U$11.NO, U$13.NO, U$6.-
- removed net SCK17: IC1.PB5(SCK), SV6.6
- removed net SWITCH: FHEADER1.3, IC1.PC0(ADC0)
- removed net SWITCH1: FHEADER4.3, IC1.PD6(AIN0)
- removed net TXD31: IC1.PD1(TXD), SV6.2
- new net 3.3V: IC4.GND, JP1.3
- new net 5.0V: JP1.2, R5.1
- new net ANODE(+)_1: IC1.TRI, R2.1
- new net C+: D4.C, J8.1, U$17.P$2, U$2.P$2, X1-2.KL, X2-2.KL
- new net CHARGE: IC2.VDD, JP2.1
- new net DONE: IC2.AGND, R16.1
- new net GATE: IC2.AGND0, T1.B, U$5.4
- new net GATE_IGBT_1: Q2.G, R1.2
- new net GATE_IGBT_2: Q3.G, R3.2
- new net MOS_TRIG: IC4.TRI, JP1.1
- new net N$28: D4.A, U$15.12
- new net N$29: LED_12V.A, R21.2
- new net PIN3: IC4.DIS, U$6.3
- new net RDCM: IC2.AL/BUSY, R18.2
- new net RGB: C20.2, IC2.SCL, R20.2
- new net RVOUT: IC2.SDA, R17.2
- new net SOURCE: IC2.AS, R19.1, T1.E, U$5.1, U$5.2, U$5.3
- new net SUPP_+: R21.1, S3A.P, S3B.P, U1.K
- new net TRIG_ON_1: JP2.2, R2.2
- new net TRIG_ON_2: JP2.3
- new net VO/NC_1: IC1.TRE
- new net VO_1: IC1.DIS, R1.1
- new net VO_2: R3.1, U$6.7
- new net VTRANS: C16.1, C2.1, IC1.VCC+, IC2.CONVST', IC2.V2/REF, R16.2, S3A.S, S3B.S, U$1.CAP+, U$15.10, U$15.7, U$15.8, U$15.9, U$3.CAP+, U$4.CAP+, U$6.6
- net GND: now also C16.2, C2.2, C20.1, IC1.CON, IC1.OUT, IC2.V1, J8.2, J9.-, Q2.D, Q3.D, R19.2, R20.1, U$1.CAP-, U$15.1, U$17.P$1, U$2.P$1, U$3.CAP-, U$4.CAP-; no longer !RESET.P, !RESET.P1, C1.2, C10.2, C11.2, C12.1, C13.1, C14.1, C3.2, C4.-, C6.2, C8.2, C9.2, FHEADER1.1, FHEADER4.1, GND12.P$1, GND_12V1.P$1, GND_5V.P$1, IC1.GND, IC1.GND@1, IC1.GND@2, IGBT.OUT, J1.2, J3.-, J5.1, J7.1, LED_BATT.C, MOSFET.OUT, R1.1, R10.1, R2.1, R3.1, R4.1, R5.1, R7.1, RD2.1, SV5.1, SV6.1, T1.E, T2.E, U$10.C, U$11.C, U$12.C, U$13.C, U$3.P$3, U$4.P$1, U$5.1, U$7.2, U$8.2, U$9.P$3
- net N$1: now also Q2.S, X1-1.KL; no longer DS.C, RS.1, U$7.1
- net N$2: now also Q3.S, X2-1.KL; no longer R_RELAY.2, T1.B
- net N$3: now also R17.1, R18.1, T1.C, U$15.3, U$15.4, U$15.5, U$15.6, U$5.5, U$5.6, U$5.7, U$5.8; no longer C6.1, IGBT.DIS, R5.2, R6.2
- net N$4: now also IC4.VCC+, R5.2, U$6.2; no longer D2.A, U$5.12
- net POWER_HEAD: now also J9.+; no longer J3.+, U4.A, U4.~A
Other:
- note removed: "CHARGING CKT 1"
- note removed: "CHARGING CKT 2"
- note removed: "CONNECTION HEADERS"
- note removed: "DRIVER AND SWITCH"
- note removed: "IGBT SWITCHING CIRCUIT"
- note removed: "POTENTIAL DIVIDER"
- note removed: "POWER SUPPLY 5v"
- note removed: "SNUBBER"
- moved on the sheet: LED_12V, R5, T1
