File: test boards/IR4427-v2/IR4427.sch (EAGLE design)
At the start: 36 parts, among them IC1 IR4427, IC2 IR4427, IC3 IR4427, IC5 ACS712-LC, Q1 IRF7389, Q2 IRF7389, Q3 IRF7389

Commit message: Update
Parts:
- removed C1A, C1B, C2A, C2B, C3A, C3B: 1n, eagle-ltspice:CC1206
Connections:
- net N$1 renamed SINK
- net GND: no longer C1A.2, C1B.2, C2A.2, C2B.2, C3A.2, C3B.2
- net OUT_1A: no longer C1A.1
- net OUT_1B: no longer C1B.1
- net OUT_2A: no longer C2A.1
- net OUT_2B: no longer C2B.1
- net OUT_3A: no longer C3A.1
- net OUT_3B: no longer C3B.1
Other:
- moved on the sheet: CL, CL1, CL2, CS, CS1, CS2, IC1, IC2, IC3, R10, R11, R12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

Commit message: IRS
Parts:
- added CL3, CL4, CL5: 4.7u, eagle-ltspice:CC1206
- added CS3, CS4, CS5: 0.1u, eagle-ltspice:CC1206
Connections:
- net GND: now also CL3.2, CL4.2, CL5.2, CS3.2, CS4.2, CS5.2
- net OUT_1A: now also CL3.1
- net OUT_1B: now also CS3.1
- net OUT_2A: now also CL4.1
- net OUT_2B: now also CS4.1
- net OUT_3A: now also CL5.1
- net OUT_3B: now also CS5.1
Changed lines of the file:
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@@
 <part name="R13" library="eagle-ltspice" library_urn="urn:adsk.eagle:library:217" deviceset="R" device="R1206" package3d_urn="urn:adsk.eagle:package:13301/1" value="1k"/>
 <part name="R14" library="eagle-ltspice" library_urn="urn:adsk.eagle:library:217" deviceset="R" device="R1206" package3d_urn="urn:adsk.eagle:package:13301/1" value="330"/>
+<part name="CL3" library="eagle-ltspice" library_urn="urn:adsk.eagle:library:217" deviceset="C" device="C1206" package3d_urn="urn:adsk.eagle:package:13279/1" value="4.7u"/>
+<part name="CS3" library="eagle-ltspice" library_urn="urn:adsk.eagle:library:217" deviceset="C" device="C1206" package3d_urn="urn:adsk.eagle:package:13279/1" value="0.1u"/>
+<part name="GND1" library="supply2" library_urn="urn:adsk.eagle:library:372" deviceset="GND" device=""/>
+<part name="CL4" library="eagle-ltspice" library_urn="urn:adsk.eagle:library:217" deviceset="C" device="C1206" package3d_urn="urn:adsk.eagle:package:13279/1" value="4.7u"/>
+<part name="CS4" library="eagle-ltspice" library_urn="urn:adsk.eagle:library:217" deviceset="C" device="C1206" package3d_urn="urn:adsk.eagle:package:13279/1" value="0.1u"/>
+<part name="GND2" library="supply2" library_urn="urn:adsk.eagle:library:372" deviceset="GND" device=""/>
+<part name="CL5" library="eagle-ltspice" library_urn="urn:adsk.eagle:library:217" deviceset="C" device="C1206" package3d_urn="urn:adsk.eagle:package:13279/1" value="4.7u"/>
+<part name="CS5" library="eagle-ltspice" library_urn="urn:adsk.eagle:library:217" deviceset="C" device="C1206" package3d_urn="urn:adsk.eagle:package:13279/1" value="0.1u"/>
+<part name="GND8" library="supply2" library_urn="urn:adsk.eagle:library:372" deviceset="GND" device=""/>
 </parts>
 <sheets>
@@
 <instance part="R13" gate="G$1" x="269.24" y="58.42"/>
 <instance part="R14" gate="G$1" x="281.94" y="63.5"/>
+<instance part="CL3" gate="G$1" x="156.73" y="-17.12"/>
+<instance part="CS3" gate="G$1" x="171.97" y="-17.12"/>
+<instance part="GND1" gate="GND" x="164.35" y="-27.28"/>
+<instance part="CL4" gate="G$1" x="188.03" y="-16.88"/>
+<instance part="CS4" gate="G$1" x="203.27" y="-16.88"/>
+<instance part="GND2" gate="GND" x="195.65" y="-27.04"/>
+<instance part="CL5" gate="G$1" x="219.53" y="-15.84"/>
+<instance part="CS5" gate="G$1" x="234.77" y="-15.84"/>
+<instance part="GND8" gate="GND" x="227.15" y="-26"/>
 </instances>
 <busses>
@@
 <label x="102.85" y="52.81" size="1.778" layer="95"/>
 </segment>
+<segment>
+<pinref part="CL3" gate="G$1" pin="1"/>
+<wire x1="156.73" y1="-14.58" x2="156.73" y2="-12.04" width="0.1524" layer="91"/>
+<label x="151.65" y="-12.04" size="1.778" layer="95"/>
+</segment>
 </net>
 <net name="OUT_1B" class="3">
@@
 <wire x1="115.55" y1="45.19" x2="113.01" y2="45.19" width="0.1524" layer="91"/>
 <label x="102.85" y="45.19" size="1.778" layer="95"/>
+</segment>
+<segment>
+<pinref part="CS3" gate="G$1" pin="1"/>
+<wire x1="171.97" y1="-14.58" x2="171.97" y2="-12.04" width="0.1524" layer="91"/>
+<label x="166.89" y="-12.04" size="1.778" layer="95"/>
 </segment>
 </net>
@@
 <label x="2.54" y="10.16" size="1.778" layer="95"/>
 </segment>
+<segment>
+<pinref part="CL3" gate="G$1" pin="2"/>
+<pinref part="GND1" gate="GND" pin="GND"/>
+<wire x1="156.73" y1="-22.2" x2="156.73" y2="-24.74" width="0.1524" layer="91"/>
+<wire x1="156.73" y1="-24.74" x2="164.35" y2="-24.74" width="0.1524" layer="91"/>
+<pinref part="CS3" gate="G$1" pin="2"/>
+<wire x1="171.97" y1="-22.2" x2="171.97" y2="-24.74" width="0.1524" layer="91"/>
+<wire x1="171.97" y1="-24.74" x2="164.35" y2="-24.74" width="0.1524" layer="91"/>
+<junction x="164.35" y="-24.74"/>
+</segment>
+<segment>
+<pinref part="CL4" gate="G$1" pin="2"/>
+<pinref part="GND2" gate="GND" pin="GND"/>
+<wire x1="188.03" y1="-21.96" x2="188.03" y2="-24.5" width="0.1524" layer="91"/>
+<wire x1="188.03" y1="-24.5" x2="195.65" y2="-24.5" width="0.1524" layer="91"/>
+<pinref part="CS4" gate="G$1" pin="2"/>
+<wire x1="203.27" y1="-21.96" x2="203.27" y2="-24.5" width="0.1524" layer="91"/>
+<wire x1="203.27" y1="-24.5" x2="195.65" y2="-24.5" width="0.1524" layer="91"/>
+<junction x="195.65" y="-24.5"/>
+</segment>
+<segment>
+<pinref part="CL5" gate="G$1" pin="2"/>
+<pinref part="GND8" gate="GND" pin="GND"/>
+<wire x1="219.53" y1="-20.92" x2="219.53" y2="-23.46" width="0.1524" layer="91"/>
+<wire x1="219.53" y1="-23.46" x2="227.15" y2="-23.46" width="0.1524" layer="91"/>
+<pinref part="CS5" gate="G$1" pin="2"/>
+<wire x1="234.77" y1="-20.92" x2="234.77" y2="-23.46" width="0.1524" layer="91"/>
+<wire x1="234.77" y1="-23.46" x2="227.15" y2="-23.46" width="0.1524" layer="91"/>
+<junction x="227.15" y="-23.46"/>
+</segment>
 </net>
 <net name="OUT_2A" class="3">
@@
 <label x="102.85" y="68.05" size="1.778" layer="95"/>
 </segment>
+<segment>
+<pinref part="CL4" gate="G$1" pin="1"/>
+<wire x1="188.03" y1="-14.34" x2="188.03" y2="-11.8" width="0.1524" layer="91"/>
+<label x="182.95" y="-11.8" size="1.778" layer="95"/>
+</segment>
 </net>
 <net name="OUT_2B" class="3">
@@
 <label x="102.85" y="60.43" size="1.778" layer="95"/>
 </segment>
+<segment>
+<pinref part="CS4" gate="G$1" pin="1"/>
+<wire x1="203.27" y1="-14.34" x2="203.27" y2="-11.8" width="0.1524" layer="91"/>
+<label x="198.19" y="-11.8" size="1.778" layer="95"/>
+</segment>
 </net>
 <net name="OUT_3A" class="3">
@@
 <label x="102.85" y="83.29" size="1.778" layer="95"/>
 </segment>
+<segment>
+<pinref part="CL5" gate="G$1" pin="1"/>
+<wire x1="219.53" y1="-13.3" x2="219.53" y2="-10.76" width="0.1524" layer="91"/>
+<label x="214.45" y="-10.76" size="1.778" layer="95"/>
+</segment>
 </net>
 <net name="OUT_3B" class="3">
@@
 <wire x1="115.55" y1="75.67" x2="113.01" y2="75.67" width="0.1524" layer="91"/>
 <label x="102.85" y="75.67" size="1.778" layer="95"/>
+</segment>
+<segment>
+<pinref part="CS5" gate="G$1" pin="1"/>
+<wire x1="234.77" y1="-13.3" x2="234.77" y2="-10.76" width="0.1524" layer="91"/>
+<label x="229.69" y="-10.76" size="1.778" layer="95"/>
 </segment>
 </net>
@@
 </segment>
 </net>
+<net name="N$1" class="0">
+<segment>
+<wire x1="147.05" y1="-2.1" x2="147.05" y2="-34.3" width="0.1524" layer="91" style="longdash"/>
+<wire x1="147.05" y1="-34.3" x2="243.95" y2="-34.3" width="0.1524" layer="91" style="longdash"/>
+<wire x1="243.95" y1="-34.3" x2="243.95" y2="-2.2" width="0.1524" layer="91" style="longdash"/>
+<wire x1="243.95" y1="-2.2" x2="147.2" y2="-2.2" width="0.1524" layer="91" style="longdash"/>
+</segment>
+</net>
