File: test boards/IR4427-v2/IR4427.brd (EAGLE design)
At the start: 50.6 x 37 mm, 30 parts, among them IC1 IR4427, IC2 IR4427, IC3 IR4427, IC5 ACS712-LC, Q1 IRF7389, Q2 IRF7389, Q3 IRF7389

Commit message: IRS
Parts:
- added CL3, CL4, CL5: 4.7u, eagle-ltspice:C1206
- added CS3, CS4, CS5: 0.1u, eagle-ltspice:C1206
Connections:
- net GND: now also CL3.2, CL4.2, CL5.2, CS3.2, CS4.2, CS5.2
- net OUT_1A: now also CL3.1
- net OUT_1B: now also CS3.1
- net OUT_2A: now also CL4.1
- net OUT_2B: now also CS4.1
- net OUT_3A: now also CL5.1
- net OUT_3B: now also CS5.1
Changed lines of the file:
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@@
 <attribute name="SPICEPREFIX" value="R" x="34" y="35.2" size="1.778" layer="27" display="off"/>
+</element>
+<element name="CL3" library="eagle-ltspice" library_urn="urn:adsk.eagle:library:217" package="C1206" package3d_urn="urn:adsk.eagle:package:13279/1" value="4.7u" x="12.6" y="12.8">
+<attribute name="SPICEMODEL" value="NONE" x="12.6" y="12.8" size="1.778" layer="27" display="off"/>
+<attribute name="SPICEPREFIX" value="C" x="12.6" y="12.8" size="1.778" layer="27" display="off"/>
+</element>
+<element name="CS3" library="eagle-ltspice" library_urn="urn:adsk.eagle:library:217" package="C1206" package3d_urn="urn:adsk.eagle:package:13279/1" value="0.1u" x="17.8" y="6.6">
+<attribute name="SPICEMODEL" value="NONE" x="12.6" y="6.6" size="1.778" layer="27" display="off"/>
+<attribute name="SPICEPREFIX" value="C" x="12.6" y="6.6" size="1.778" layer="27" display="off"/>
+</element>
+<element name="CL4" library="eagle-ltspice" library_urn="urn:adsk.eagle:library:217" package="C1206" package3d_urn="urn:adsk.eagle:package:13279/1" value="4.7u" x="17.8" y="12.8">
+<attribute name="SPICEMODEL" value="NONE" x="12.6" y="0.4" size="1.778" layer="27" display="off"/>
+<attribute name="SPICEPREFIX" value="C" x="12.6" y="0.4" size="1.778" layer="27" display="off"/>
+</element>
+<element name="CS4" library="eagle-ltspice" library_urn="urn:adsk.eagle:library:217" package="C1206" package3d_urn="urn:adsk.eagle:package:13279/1" value="0.1u" x="12.6" y="0.4">
+<attribute name="SPICEMODEL" value="NONE" x="12.6" y="-5.8" size="1.778" layer="27" display="off"/>
+<attribute name="SPICEPREFIX" value="C" x="12.6" y="-5.8" size="1.778" layer="27" display="off"/>
+</element>
+<element name="CL5" library="eagle-ltspice" library_urn="urn:adsk.eagle:library:217" package="C1206" package3d_urn="urn:adsk.eagle:package:13279/1" value="4.7u" x="12.6" y="6.6">
+<attribute name="SPICEMODEL" value="NONE" x="12.6" y="-12" size="1.778" layer="27" display="off"/>
+<attribute name="SPICEPREFIX" value="C" x="12.6" y="-12" size="1.778" layer="27" display="off"/>
+</element>
+<element name="CS5" library="eagle-ltspice" library_urn="urn:adsk.eagle:library:217" package="C1206" package3d_urn="urn:adsk.eagle:package:13279/1" value="0.1u" x="17.8" y="0.4">
+<attribute name="SPICEMODEL" value="NONE" x="12.6" y="-18.2" size="1.778" layer="27" display="off"/>
+<attribute name="SPICEPREFIX" value="C" x="12.6" y="-18.2" size="1.778" layer="27" display="off"/>
 </element>
 </elements>
@@
 <contactref element="Q2" pad="3"/>
 <contactref element="Q3" pad="3"/>
-<wire x1="27.4" y1="45" x2="38.4568" y2="43.365" width="0" layer="19" extent="1-1"/>
-<wire x1="29.81" y1="44.93" x2="27.4" y2="45" width="0" layer="19" extent="1-1"/>
-<wire x1="41.1" y1="45.4" x2="29.81" y2="44.93" width="0" layer="19" extent="1-1"/>
-<wire x1="13.5" y1="42.73" x2="41.1" y2="45.4" width="0" layer="19" extent="1-1"/>
-<wire x1="16.5" y1="42.8" x2="13.5" y2="42.73" width="0" layer="19" extent="1-1"/>
+<wire x1="38.4568" y1="43.365" x2="41.1" y2="45.4" width="0" layer="19" extent="1-16"/>
+<wire x1="29.81" y1="44.93" x2="38.4568" y2="43.365" width="0" layer="19" extent="1-1"/>
+<wire x1="27.4" y1="45" x2="29.81" y2="44.93" width="0" layer="19" extent="16-16"/>
+<wire x1="16.5" y1="42.8" x2="27.4" y2="45" width="0" layer="19" extent="1-16"/>
+<wire x1="13.5" y1="42.73" x2="16.5" y2="42.8" width="0" layer="19" extent="1-1"/>
 <wire x1="38.4568" y1="31.865" x2="38.4568" y2="43.365" width="0" layer="19" extent="1-1"/>
-<wire x1="27.4" y1="33" x2="38.4568" y2="31.865" width="0" layer="19" extent="1-1"/>
-<wire x1="29.81" y1="33.03" x2="27.4" y2="33" width="0" layer="19" extent="1-1"/>
+<wire x1="29.81" y1="33.03" x2="38.4568" y2="31.865" width="0" layer="19" extent="1-1"/>
+<wire x1="27.4" y1="33" x2="29.81" y2="33.03" width="0" layer="19" extent="16-16"/>
 <wire x1="38.4568" y1="21.365" x2="38.4568" y2="31.865" width="0" layer="19" extent="1-1"/>
-<wire x1="27.4" y1="21" x2="38.4568" y2="21.365" width="0" layer="19" extent="1-1"/>
-<wire x1="29.81" y1="21.03" x2="27.4" y2="21" width="0" layer="19" extent="1-1"/>
+<wire x1="29.81" y1="21.03" x2="38.4568" y2="21.365" width="0" layer="19" extent="1-1"/>
+<wire x1="27.4" y1="21" x2="29.81" y2="21.03" width="0" layer="19" extent="16-16"/>
+<wire x1="19.9" y1="24" x2="27.4" y2="21" width="0" layer="19" extent="1-16"/>
 <wire x1="48" y1="18.578" x2="38.4568" y2="21.365" width="0" layer="19" extent="1-1"/>
-<wire x1="19.9" y1="24" x2="29.81" y2="21.03" width="0" layer="19" extent="1-1"/>
 </signal>
 <signal name="OUT_1A" class="3">
 <contactref element="IC1" pad="7"/>
 <contactref element="R11" pad="1"/>
+<contactref element="CL3" pad="1"/>
 <wire x1="29.81" y1="47.47" x2="32.578" y2="47.5" width="0" layer="19" extent="1-1"/>
+<wire x1="11.2" y1="12.8" x2="29.81" y2="47.47" width="0" layer="19" extent="1-1"/>
 </signal>
 <signal name="OUT_1B" class="3">
 <contactref element="IC1" pad="5"/>
 <contactref element="R12" pad="1"/>
+<contactref element="CS3" pad="1"/>
 <wire x1="29.81" y1="42.39" x2="32.578" y2="42.5" width="0" layer="19" extent="1-1"/>
+<wire x1="16.4" y1="6.6" x2="29.81" y2="42.39" width="0" layer="19" extent="1-1"/>
 </signal>
 <signal name="GND" class="4">
@@
 <contactref element="POWER" pad="4"/>
 <contactref element="J1" pad="3"/>
+<contactref element="CL3" pad="2"/>
+<contactref element="CS3" pad="2"/>
+<contactref element="CL4" pad="2"/>
+<contactref element="CS4" pad="2"/>
+<contactref element="CL5" pad="2"/>
+<contactref element="CS5" pad="2"/>
 <wire x1="48" y1="39.73" x2="54.603" y2="43.54" width="0" layer="19" extent="1-1"/>
 <wire x1="43.6" y1="34.405" x2="48" y2="39.73" width="0" layer="19" extent="16-16"/>
@@
 <wire x1="22.19" y1="21.03" x2="17.1" y2="24" width="0" layer="19" extent="1-1"/>
 <wire x1="24.6" y1="21" x2="22.19" y2="21.03" width="0" layer="19" extent="16-16"/>
+<wire x1="19.2" y1="12.8" x2="22.19" y2="21.03" width="0" layer="19" extent="1-1"/>
+<wire x1="14" y1="12.8" x2="19.2" y2="12.8" width="0" layer="19" extent="1-1"/>
+<wire x1="19.2" y1="6.6" x2="19.2" y2="12.8" width="0" layer="19" extent="1-1"/>
+<wire x1="14" y1="6.6" x2="19.2" y2="6.6" width="0" layer="19" extent="1-1"/>
+<wire x1="19.2" y1="0.4" x2="19.2" y2="6.6" width="0" layer="19" extent="1-1"/>
+<wire x1="14" y1="0.4" x2="19.2" y2="0.4" width="0" layer="19" extent="1-1"/>
 </signal>
 <signal name="OUT_2A" class="3">
 <contactref element="IC2" pad="7"/>
 <contactref element="R9" pad="1"/>
+<contactref element="CL4" pad="1"/>
 <wire x1="32.578" y1="35.2" x2="29.81" y2="35.57" width="0" layer="19" extent="1-1"/>
+<wire x1="16.4" y1="12.8" x2="29.81" y2="35.57" width="0" layer="19" extent="1-1"/>
 </signal>
 <signal name="OUT_2B" class="3">
 <contactref element="IC2" pad="5"/>
 <contactref element="R10" pad="1"/>
+<contactref element="CS4" pad="1"/>
 <wire x1="32.578" y1="30.2" x2="29.81" y2="30.49" width="0" layer="19" extent="1-1"/>
+<wire x1="11.2" y1="0.4" x2="29.81" y2="30.49" width="0" layer="19" extent="1-1"/>
 </signal>
 <signal name="OUT_3A" class="3">
 <contactref element="IC3" pad="7"/>
 <contactref element="R7" pad="1"/>
+<contactref element="CL5" pad="1"/>
 <wire x1="29.81" y1="23.57" x2="32.578" y2="24" width="0" layer="19" extent="1-1"/>
+<wire x1="11.2" y1="6.6" x2="29.81" y2="23.57" width="0" layer="19" extent="1-1"/>
 </signal>
 <signal name="OUT_3B" class="3">
 <contactref element="IC3" pad="5"/>
 <contactref element="R8" pad="1"/>
+<contactref element="CS5" pad="1"/>
 <wire x1="29.81" y1="18.49" x2="32.578" y2="19" width="0" layer="19" extent="1-1"/>
+<wire x1="16.4" y1="0.4" x2="29.81" y2="18.49" width="0" layer="19" extent="1-1"/>
 </signal>
 <signal name="H1" class="3">

Commit message: Completed
Parts:
- removed HALL: (no value), con-lstb:MA03-2
- removed INPUT: (no value), con-lstb:MA06-1
- removed J1: (no value), SparkFun-Connectors:2X5-SHROUDED_LOCK
- removed MOTOR: (no value), con-lstb:MA08-1
- removed POWER: (no value), pinhead:1X04
- added SV1: (no value), con-lstb:MA10-1
- added SV2: (no value), con-lstb:MA08-1
- moved CL3 40.8 mm to (32.2, 48.6), flipped to the bottom, turned to 270 degrees
- moved CS3 39.0 mm to (32.2, 42.8), flipped to the bottom, turned to 270 degrees
- moved CS4 36.6 mm to (32.3, 31.3), flipped to the bottom, turned to 270 degrees
- moved R13 32.7 mm to (37.8, 51.1), turned to 0 degrees
- moved CL4 28.1 mm to (32.3, 36.9), flipped to the bottom, turned to 270 degrees
- moved CL5 26.9 mm to (32.3, 24.9), flipped to the bottom, turned to 270 degrees
- moved LED18V 25.7 mm to (43.3, 51.1), turned to 270 degrees
- moved CS5 23.9 mm to (32.3, 19.4), flipped to the bottom, turned to 270 degrees
- moved CS 15.5 mm to (26.0, 47.3), turned to 0 degrees
- moved R14 13.5 mm to (37.7, 17.6), turned to 0 degrees
- moved CS1 11.2 mm to (26.0, 35.4), flipped to the bottom, turned to 0 degrees
- moved LED5V 11.2 mm to (43.4, 17.6), turned to 270 degrees
- moved CS2 7.53 mm to (26.0, 23.3), flipped to the bottom, turned to 0 degrees
- moved CF 4.08 mm to (37.7, 39.2)
- moved Q1 3.89 mm to (37.6, 45.9)
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Connections:
- removed net A: HALL.5, J1.6
- removed net B: HALL.3, J1.8
- removed net H1: HALL.6, MOTOR.3
- removed net H2: HALL.4, MOTOR.2
- removed net H3: HALL.2, MOTOR.1
- net 1A: now also SV1.8; no longer INPUT.6
- net 1B: now also SV1.7; no longer INPUT.5
- net 2A: now also SV1.6; no longer INPUT.4
- net 2B: now also SV1.5; no longer INPUT.3
- net 3A: now also SV1.4; no longer INPUT.2
- net 3B: now also SV1.3; no longer INPUT.1
- net ACS_OUT: now also SV2.8; no longer POWER.2
- net GND: now also SV1.1, SV1.2; no longer HALL.1, J1.3, MOTOR.4, POWER.4
- net M1: now also SV2.6, SV2.7; no longer MOTOR.8
- net M2: now also SV2.4, SV2.5; no longer MOTOR.7
- net M3: now also SV2.2, SV2.3; no longer MOTOR.6
- net VCC_18: now also SV1.10, SV1.9; no longer POWER.3
- net VCC_5V: now also SV2.1; no longer J1.2, MOTOR.5, POWER.1
Routing:
- net SINK: track 0.00 -> 34.0 mm, vias 0 -> 1
- net VCC_5V: track 0.00 -> 28.6 mm
- net 3P: track 0.00 -> 19.7 mm
- net ACS_OUT: track 0.00 -> 17.6 mm
- net VCC_18: track 0.00 -> 14.3 mm
- net 3B: track 0.00 -> 11.4 mm
- net 3A: track 0.00 -> 9.22 mm
- net 1A: track 0.00 -> 9.15 mm
- net 1N: track 0.00 -> 8.10 mm
- net M1: track 0.00 -> 7.48 mm
- net N$3: track 0.00 -> 6.95 mm
- net 1B: track 0.00 -> 6.02 mm
- net M3: track 0.00 -> 5.71 mm
- net 2B: track 0.00 -> 5.24 mm
- net 2A: track 0.00 -> 4.19 mm
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- added copper zone on layer 16, net GND
- added copper zone on layer 1, net M1
- added copper zone on layer 1, net M2
- added copper zone on layer 1, net M3
- added copper zone on layer 1, net VCC_18
Other:
- board size 50.6 x 37 mm -> 34 x 37 mm
- board text removed: "HM"
- board text removed: "KRSSG"
- board text removed: "PD"
- board text removed: "TJ"
- board text removed: "¯\_(ツ)_/¯"
