File: test boards/MotorTestBoard/FPGA.brd (EAGLE design)
At the start: 160 x 100 mm, 2 parts, among them X1 87758-4016, X2 87758-4016

Commit message: FPGA Labelling
Connections:
- new net M11A: X1.3
- new net M11B: X1.5
- new net M12A: X1.7
- new net M12B: X1.9
- new net M13A: X1.11
- new net M13B: X1.13
- new net M1EA: X1.4
- new net M1EB: X1.6
- new net M1H1: X1.8
- new net M1H2: X1.10
- new net M1H3: X1.12
- new net M21A: X1.27
- new net M21B: X1.29
- new net M22A: X1.31
- new net M22B: X1.33
- new net M23A: X1.35
- new net M23B: X1.37
- new net M2EA: X1.30
- new net M2EB: X1.32
- new net M2H1: X1.34
- new net M2H2: X1.36
- new net M2H3: X1.38
- new net M31A: X2.4
- new net M31B: X2.6
- new net M32A: X2.8
- new net M32B: X2.10
- new net M33A: X2.12
- new net M33B: X2.14
- new net M3EA: X2.3
- new net M3EB: X2.5
- new net M3H1: X2.7
- new net M3H2: X2.9
- new net M3H3: X2.11
- new net M41A: X2.28
- new net M41B: X2.30
- new net M42A: X2.32
- new net M42B: X2.34
- new net M43A: X2.36
- new net M43B: X2.38
- new net M4EA: X2.29
- new net M4EB: X2.31
- new net M4H1: X2.33
- new net M4H2: X2.35
- new net M4H3: X2.37
Changed lines of the file:
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@@
 </elements>
 <signals>
+<signal name="M11A">
+<contactref element="X1" pad="3"/>
+</signal>
+<signal name="M11B">
+<contactref element="X1" pad="5"/>
+</signal>
+<signal name="M1EA">
+<contactref element="X1" pad="4"/>
+</signal>
+<signal name="M1EB">
+<contactref element="X1" pad="6"/>
+</signal>
+<signal name="M12A">
+<contactref element="X1" pad="7"/>
+</signal>
+<signal name="M1H1">
+<contactref element="X1" pad="8"/>
+</signal>
+<signal name="M12B">
+<contactref element="X1" pad="9"/>
+</signal>
+<signal name="M13A">
+<contactref element="X1" pad="11"/>
+</signal>
+<signal name="M13B">
+<contactref element="X1" pad="13"/>
+</signal>
+<signal name="M1H2">
+<contactref element="X1" pad="10"/>
+</signal>
+<signal name="M1H3">
+<contactref element="X1" pad="12"/>
+</signal>
+<signal name="M23B">
+<contactref element="X1" pad="37"/>
+</signal>
+<signal name="M23A">
+<contactref element="X1" pad="35"/>
+</signal>
+<signal name="M22B">
+<contactref element="X1" pad="33"/>
+</signal>
+<signal name="M22A">
+<contactref element="X1" pad="31"/>
+</signal>
+<signal name="M21B">
+<contactref element="X1" pad="29"/>
+</signal>
+<signal name="M21A">
+<contactref element="X1" pad="27"/>
+</signal>
+<signal name="M2H3">
+<contactref element="X1" pad="38"/>
+</signal>
+<signal name="M2H2">
+<contactref element="X1" pad="36"/>
+</signal>
+<signal name="M2H1">
+<contactref element="X1" pad="34"/>
+</signal>
+<signal name="M2EB">
+<contactref element="X1" pad="32"/>
+</signal>
+<signal name="M2EA">
+<contactref element="X1" pad="30"/>
+</signal>
+<signal name="M3EA">
+<contactref element="X2" pad="3"/>
+</signal>
+<signal name="M3EB">
+<contactref element="X2" pad="5"/>
+</signal>
+<signal name="M3H1">
+<contactref element="X2" pad="7"/>
+</signal>
+<signal name="M3H2">
+<contactref element="X2" pad="9"/>
+</signal>
+<signal name="M3H3">
+<contactref element="X2" pad="11"/>
+</signal>
+<signal name="M31A">
+<contactref element="X2" pad="4"/>
+</signal>
+<signal name="M31B">
+<contactref element="X2" pad="6"/>
+</signal>
+<signal name="M32A">
+<contactref element="X2" pad="8"/>
+</signal>
+<signal name="M32B">
+<contactref element="X2" pad="10"/>
+</signal>
+<signal name="M33A">
+<contactref element="X2" pad="12"/>
+</signal>
+<signal name="M33B">
+<contactref element="X2" pad="14"/>
+</signal>
+<signal name="M43B">
+<contactref element="X2" pad="38"/>
+</signal>
+<signal name="M43A">
+<contactref element="X2" pad="36"/>
+</signal>
+<signal name="M42B">
+<contactref element="X2" pad="34"/>
+</signal>
+<signal name="M42A">
+<contactref element="X2" pad="32"/>
+</signal>
+<signal name="M41B">
+<contactref element="X2" pad="30"/>
+</signal>
+<signal name="M41A">
+<contactref element="X2" pad="28"/>
+</signal>
+<signal name="M4H3">
+<contactref element="X2" pad="37"/>
+</signal>
+<signal name="M4H2">
+<contactref element="X2" pad="35"/>
+</signal>
+<signal name="M4H1">
+<contactref element="X2" pad="33"/>
+</signal>
+<signal name="M4EB">
+<contactref element="X2" pad="31"/>
+</signal>
+<signal name="M4EA">
+<contactref element="X2" pad="29"/>
+</signal>
 </signals>
 <mfgpreviewcolors>
