File: test boards/MotorTestBoard/FPGA.brd (EAGLE design)
At the start: 160 x 100 mm, 14 parts, among them X1 87758-4016, X2 87758-4016

Commit message: encoders
Parts:
- added J1, J2, J3, J4: (no value), SparkFun-Connectors:2X5-SHROUDED_LOCK
Connections:
- net 5V: now also J1.2, J2.2, J3.2, J4.2
- net GND: now also J1.3, J2.3, J3.3, J4.3
- net M1EA: now also J1.6
- net M1EB: now also J1.8
- net M2EA: now also J2.6
- net M2EB: now also J2.8
- net M3EA: now also J3.6
- net M3EB: now also J3.8
- net M4EA: now also J4.6
- net M4EB: now also J4.8
Changed lines of the file:
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@@
 <layer number="115" name="ReferenceISLANDS" color="7" fill="1" visible="yes" active="yes"/>
 <layer number="116" name="Patch_BOT" color="9" fill="4" visible="yes" active="yes"/>
+<layer number="117" name="BACKMAAT1" color="7" fill="1" visible="yes" active="yes"/>
 <layer number="118" name="Rect_Pads" color="7" fill="1" visible="no" active="no"/>
+<layer number="119" name="KAP_TEKEN" color="7" fill="1" visible="yes" active="yes"/>
+<layer number="120" name="KAP_MAAT1" color="7" fill="1" visible="yes" active="yes"/>
 <layer number="121" name="_tsilk" color="7" fill="1" visible="no" active="yes"/>
 <layer number="122" name="_bsilk" color="7" fill="1" visible="no" active="yes"/>
@@
 <layer number="128" name="_bValues" color="7" fill="1" visible="yes" active="yes"/>
 <layer number="129" name="Mask" color="7" fill="1" visible="yes" active="yes"/>
+<layer number="130" name="SMDSTROOK" color="7" fill="1" visible="yes" active="yes"/>
 <layer number="131" name="tAdjust" color="7" fill="1" visible="yes" active="yes"/>
 <layer number="132" name="bAdjust" color="7" fill="1" visible="yes" active="yes"/>
+<layer number="133" name="bottom_silk" color="7" fill="1" visible="yes" active="yes"/>
+<layer number="134" name="silk_top" color="7" fill="1" visible="yes" active="yes"/>
+<layer number="135" name="silk_bottom" color="7" fill="1" visible="yes" active="yes"/>
+<layer number="136" name="silktop" color="7" fill="1" visible="yes" active="yes"/>
+<layer number="137" name="silkbottom" color="7" fill="1" visible="yes" active="yes"/>
 <layer number="144" name="Drill_legend" color="7" fill="1" visible="no" active="yes"/>
+<layer number="145" name="DrillLegend_01-16" color="7" fill="1" visible="yes" active="yes"/>
+<layer number="146" name="DrillLegend_01-20" color="7" fill="1" visible="yes" active="yes"/>
 <layer number="150" name="Notes" color="7" fill="1" visible="yes" active="yes"/>
 <layer number="151" name="HeatSink" color="7" fill="1" visible="no" active="yes"/>
@@
 <layer number="154" name="FabDoc2" color="7" fill="1" visible="yes" active="yes"/>
 <layer number="155" name="FabDoc3" color="7" fill="1" visible="yes" active="yes"/>
+<layer number="166" name="AntennaArea" color="7" fill="1" visible="yes" active="yes"/>
+<layer number="168" name="4mmHeightArea" color="7" fill="1" visible="yes" active="yes"/>
 <layer number="199" name="Contour" color="7" fill="1" visible="yes" active="yes"/>
 <layer number="200" name="200bmp" color="1" fill="10" visible="no" active="no"/>
@@
 <classes>
 <class number="0" name="default" width="0" drill="0">
+</class>
+<class number="1" name="5v" width="0.4" drill="0.4">
+<clearance class="1" value="0.1524"/>
+</class>
+<class number="3" name="signal" width="0.3" drill="0.4">
+<clearance class="3" value="0.1524"/>
+</class>
+<class number="4" name="gnd" width="1.4" drill="0.4">
+<clearance class="4" value="0.1524"/>
 </class>
 </classes>
@@
 <attribute name="OC_NEWARK" value="unknown" x="125.73" y="34.89" size="1.778" layer="27" display="off"/>
 </element>
+<element name="J1" library="SparkFun-Connectors" library_urn="urn:adsk.eagle:library:513" package="2X5-SHROUDED_LOCK" package3d_urn="urn:adsk.eagle:package:38007/1" value="" x="5.08" y="-41.91">
+<attribute name="PROD_ID" value="CONN-08671" x="-5.08" y="-17.78" size="1.778" layer="27" display="off"/>
+<attribute name="SF_ID" value="PRT-08506" x="-5.08" y="-17.78" size="1.778" layer="27" display="off"/>
+</element>
+<element name="J2" library="SparkFun-Connectors" library_urn="urn:adsk.eagle:library:513" package="2X5-SHROUDED_LOCK" package3d_urn="urn:adsk.eagle:package:38007/1" value="" x="5.08" y="-64.77">
+<attribute name="PROD_ID" value="CONN-08671" x="-5.08" y="-39.37" size="1.778" layer="27" display="off"/>
+<attribute name="SF_ID" value="PRT-08506" x="-5.08" y="-39.37" size="1.778" layer="27" display="off"/>
+</element>
+<element name="J3" library="SparkFun-Connectors" library_urn="urn:adsk.eagle:library:513" package="2X5-SHROUDED_LOCK" package3d_urn="urn:adsk.eagle:package:38007/1" value="" x="5.08" y="-87.63">
+<attribute name="PROD_ID" value="CONN-08671" x="-5.08" y="-62.23" size="1.778" layer="27" display="off"/>
+<attribute name="SF_ID" value="PRT-08506" x="-5.08" y="-62.23" size="1.778" layer="27" display="off"/>
+</element>
+<element name="J4" library="SparkFun-Connectors" library_urn="urn:adsk.eagle:library:513" package="2X5-SHROUDED_LOCK" package3d_urn="urn:adsk.eagle:package:38007/1" value="" x="5.08" y="-110.49">
+<attribute name="PROD_ID" value="CONN-08671" x="-5.08" y="-85.09" size="1.778" layer="27" display="off"/>
+<attribute name="SF_ID" value="PRT-08506" x="-5.08" y="-85.09" size="1.778" layer="27" display="off"/>
+</element>
 </elements>
 <signals>
@@
 <signal name="M1EA">
 <contactref element="X1" pad="4"/>
+<contactref element="J1" pad="6"/>
+<wire x1="6.477" y1="-41.91" x2="65.55" y2="25.13" width="0" layer="19" extent="1-1"/>
 </signal>
 <signal name="M1EB">
 <contactref element="X1" pad="6"/>
+<contactref element="J1" pad="8"/>
+<wire x1="6.477" y1="-44.45" x2="67.55" y2="25.13" width="0" layer="19" extent="1-1"/>
 </signal>
 <signal name="M12A">
@@
 <signal name="M2EB">
 <contactref element="X1" pad="32"/>
+<contactref element="J2" pad="8"/>
+<wire x1="6.477" y1="-67.31" x2="93.55" y2="25.13" width="0" layer="19" extent="1-1"/>
 </signal>
 <signal name="M2EA">
 <contactref element="X1" pad="30"/>
+<contactref element="J2" pad="6"/>
+<wire x1="6.477" y1="-64.77" x2="91.55" y2="25.13" width="0" layer="19" extent="1-1"/>
 </signal>
 <signal name="M3EA">
 <contactref element="X2" pad="3"/>
+<contactref element="J3" pad="6"/>
+<wire x1="6.477" y1="-87.63" x2="65.55" y2="77.49" width="0" layer="19" extent="1-1"/>
 </signal>
 <signal name="M3EB">
 <contactref element="X2" pad="5"/>
+<contactref element="J3" pad="8"/>
+<wire x1="6.477" y1="-90.17" x2="67.55" y2="77.49" width="0" layer="19" extent="1-1"/>
 </signal>
 <signal name="M3H1">
@@
 <signal name="M4EB">
 <contactref element="X2" pad="31"/>
+<contactref element="J4" pad="8"/>
+<wire x1="6.477" y1="-113.03" x2="93.55" y2="77.49" width="0" layer="19" extent="1-1"/>
 </signal>
 <signal name="M4EA">
 <contactref element="X2" pad="29"/>
+<contactref element="J4" pad="6"/>
+<wire x1="6.477" y1="-110.49" x2="91.55" y2="77.49" width="0" layer="19" extent="1-1"/>
 </signal>
 <signal name="M11">
@@
 <contactref element="SV15" pad="1"/>
 <contactref element="SV9" pad="1"/>
+<contactref element="J1" pad="2"/>
+<contactref element="J2" pad="2"/>
+<contactref element="J3" pad="2"/>
+<contactref element="J4" pad="2"/>
 <wire x1="116.84" y1="8.89" x2="119.38" y2="58.42" width="0" layer="19" extent="1-1"/>
 <wire x1="15.24" y1="59.69" x2="119.38" y2="58.42" width="0" layer="19" extent="1-1"/>
@@
 <wire x1="12.7" y1="-19.05" x2="12.7" y2="-11.43" width="0" layer="19" extent="1-1"/>
 <wire x1="12.7" y1="-26.67" x2="12.7" y2="-19.05" width="0" layer="19" extent="1-1"/>
+<wire x1="6.477" y1="-36.83" x2="12.7" y2="-26.67" width="0" layer="19" extent="1-1"/>
+<wire x1="6.477" y1="-59.69" x2="6.477" y2="-36.83" width="0" layer="19" extent="1-1"/>
+<wire x1="6.477" y1="-82.55" x2="6.477" y2="-59.69" width="0" layer="19" extent="1-1"/>
+<wire x1="6.477" y1="-105.41" x2="6.477" y2="-82.55" width="0" layer="19" extent="1-1"/>
 </signal>
 <signal name="GND">
@@
 <contactref element="SV10" pad="2"/>
 <contactref element="SV10" pad="1"/>
+<contactref element="J1" pad="3"/>
+<contactref element="J2" pad="3"/>
+<contactref element="J3" pad="3"/>
+<contactref element="J4" pad="3"/>
 <wire x1="116.84" y1="84.42" x2="119.38" y2="84.42" width="0" layer="19" extent="1-1"/>
 <wire x1="116.84" y1="34.89" x2="116.84" y2="84.42" width="0" layer="19" extent="1-1"/>
@@
 <wire x1="10.16" y1="-19.05" x2="10.16" y2="-11.43" width="0" layer="19" extent="1-1"/>
 <wire x1="10.16" y1="-26.67" x2="10.16" y2="-19.05" width="0" layer="19" extent="1-1"/>
+<wire x1="3.683" y1="-39.37" x2="10.16" y2="-26.67" width="0" layer="19" extent="1-1"/>
+<wire x1="3.683" y1="-62.23" x2="3.683" y2="-39.37" width="0" layer="19" extent="1-1"/>
+<wire x1="3.683" y1="-85.09" x2="3.683" y2="-62.23" width="0" layer="19" extent="1-1"/>
+<wire x1="3.683" y1="-107.95" x2="3.683" y2="-85.09" width="0" layer="19" extent="1-1"/>
 </signal>
 <signal name="M21">

Commit message: update
Parts:
- added C1, C2, C3, C4, C5, C9: 47uF, rcl:C1206
- added IC1, IC2: 7805T, linear:TO220H
- added U1: (no value), SparkFun-PowerIC:SOT223
Connections:
- new net 3.3V: C9.1, U1.2, U1.4
- new net 5VI: C2.1, C5.1, IC2.3, U1.3
- new net VCKT: C1.1, C4.1, IC1.1, IC2.1
- net 5V: now also C3.1, IC1.3
- net GND: now also C1.2, C2.2, C3.2, C4.2, C5.2, C9.2, IC1.2, IC2.2, U1.1
Changed lines of the file:
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@@
 <attribute name="SF_ID" value="PRT-08506" x="-5.08" y="-85.09" size="1.778" layer="27" display="off"/>
 </element>
+<element name="U1" library="SparkFun-PowerIC" package="SOT223" value="" x="3.81" y="-149.86">
+<attribute name="PROD_ID" value="VREG-08170" x="-3.81" y="-138.43" size="1.778" layer="27" display="off"/>
+</element>
+<element name="C2" library="rcl" package="C1206" value="47uF" x="10.16" y="-147.32"/>
+<element name="C9" library="rcl" package="C1206" value="47uF" x="16.51" y="-147.32"/>
+<element name="IC1" library="linear" library_urn="urn:adsk.eagle:library:262" package="TO220H" package3d_urn="urn:adsk.eagle:package:16414/1" value="7805T" x="-8.89" y="-140.97"/>
+<element name="IC2" library="linear" library_urn="urn:adsk.eagle:library:262" package="TO220H" package3d_urn="urn:adsk.eagle:package:16414/1" value="7805T" x="-25.4" y="-140.97"/>
+<element name="C1" library="rcl" package="C1206" value="47uF" x="-30.48" y="-157.48"/>
+<element name="C3" library="rcl" package="C1206" value="47uF" x="-30.48" y="-163.83"/>
+<element name="C4" library="rcl" package="C1206" value="47uF" x="-30.48" y="-170.18"/>
+<element name="C5" library="rcl" package="C1206" value="47uF" x="-30.48" y="-176.53"/>
 </elements>
 <signals>
@@
 <contactref element="J3" pad="2"/>
 <contactref element="J4" pad="2"/>
+<contactref element="IC1" pad="3"/>
+<contactref element="C3" pad="1"/>
+<wire x1="-6.35" y1="-151.13" x2="-31.88" y2="-163.83" width="0" layer="19" extent="1-1"/>
+<wire x1="6.477" y1="-105.41" x2="-6.35" y2="-151.13" width="0" layer="19" extent="1-1"/>
+<wire x1="6.477" y1="-82.55" x2="6.477" y2="-105.41" width="0" layer="19" extent="1-1"/>
+<wire x1="6.477" y1="-59.69" x2="6.477" y2="-82.55" width="0" layer="19" extent="1-1"/>
+<wire x1="6.477" y1="-36.83" x2="6.477" y2="-59.69" width="0" layer="19" extent="1-1"/>
+<wire x1="12.7" y1="-26.67" x2="6.477" y2="-36.83" width="0" layer="19" extent="1-1"/>
+<wire x1="12.7" y1="-19.05" x2="12.7" y2="-26.67" width="0" layer="19" extent="1-1"/>
+<wire x1="12.7" y1="-11.43" x2="12.7" y2="-19.05" width="0" layer="19" extent="1-1"/>
+<wire x1="12.7" y1="-3.81" x2="12.7" y2="-11.43" width="0" layer="19" extent="1-1"/>
+<wire x1="11.43" y1="11.43" x2="12.7" y2="-3.81" width="0" layer="19" extent="1-1"/>
+<wire x1="15.24" y1="59.69" x2="11.43" y2="11.43" width="0" layer="19" extent="1-1"/>
+<wire x1="119.38" y1="58.42" x2="15.24" y2="59.69" width="0" layer="19" extent="1-1"/>
 <wire x1="116.84" y1="8.89" x2="119.38" y2="58.42" width="0" layer="19" extent="1-1"/>
-<wire x1="15.24" y1="59.69" x2="119.38" y2="58.42" width="0" layer="19" extent="1-1"/>
-<wire x1="11.43" y1="11.43" x2="15.24" y2="59.69" width="0" layer="19" extent="1-1"/>
-<wire x1="12.7" y1="-3.81" x2="11.43" y2="11.43" width="0" layer="19" extent="1-1"/>
-<wire x1="12.7" y1="-11.43" x2="12.7" y2="-3.81" width="0" layer="19" extent="1-1"/>
-<wire x1="12.7" y1="-19.05" x2="12.7" y2="-11.43" width="0" layer="19" extent="1-1"/>
-<wire x1="12.7" y1="-26.67" x2="12.7" y2="-19.05" width="0" layer="19" extent="1-1"/>
-<wire x1="6.477" y1="-36.83" x2="12.7" y2="-26.67" width="0" layer="19" extent="1-1"/>
-<wire x1="6.477" y1="-59.69" x2="6.477" y2="-36.83" width="0" layer="19" extent="1-1"/>
-<wire x1="6.477" y1="-82.55" x2="6.477" y2="-59.69" width="0" layer="19" extent="1-1"/>
-<wire x1="6.477" y1="-105.41" x2="6.477" y2="-82.55" width="0" layer="19" extent="1-1"/>
 </signal>
 <signal name="GND">
@@
 <contactref element="J3" pad="3"/>
 <contactref element="J4" pad="3"/>
+<contactref element="C2" pad="2"/>
+<contactref element="C9" pad="2"/>
+<contactref element="U1" pad="1"/>
+<contactref element="C3" pad="2"/>
+<contactref element="IC1" pad="2"/>
+<contactref element="C1" pad="2"/>
+<contactref element="C4" pad="2"/>
+<contactref element="C5" pad="2"/>
+<contactref element="IC2" pad="2"/>
 <wire x1="116.84" y1="84.42" x2="119.38" y2="84.42" width="0" layer="19" extent="1-1"/>
 <wire x1="116.84" y1="34.89" x2="116.84" y2="84.42" width="0" layer="19" extent="1-1"/>
@@
 <wire x1="3.683" y1="-85.09" x2="3.683" y2="-62.23" width="0" layer="19" extent="1-1"/>
 <wire x1="3.683" y1="-107.95" x2="3.683" y2="-85.09" width="0" layer="19" extent="1-1"/>
+<wire x1="11.56" y1="-147.32" x2="3.683" y2="-107.95" width="0" layer="19" extent="1-1"/>
+<wire x1="17.91" y1="-147.32" x2="11.56" y2="-147.32" width="0" layer="19" extent="1-1"/>
+<wire x1="1.4986" y1="-152.9588" x2="11.56" y2="-147.32" width="0" layer="19" extent="1-1"/>
+<wire x1="-8.89" y1="-151.13" x2="1.4986" y2="-152.9588" width="0" layer="19" extent="1-1"/>
+<wire x1="-25.4" y1="-151.13" x2="-8.89" y2="-151.13" width="0" layer="19" extent="1-1"/>
+<wire x1="-29.08" y1="-157.48" x2="-25.4" y2="-151.13" width="0" layer="19" extent="1-1"/>
+<wire x1="-29.08" y1="-163.83" x2="-29.08" y2="-157.48" width="0" layer="19" extent="1-1"/>
+<wire x1="-29.08" y1="-170.18" x2="-29.08" y2="-163.83" width="0" layer="19" extent="1-1"/>
+<wire x1="-29.08" y1="-176.53" x2="-29.08" y2="-170.18" width="0" layer="19" extent="1-1"/>
 </signal>
 <signal name="M21">
@@
 <contactref element="SV9" pad="8"/>
 </signal>
+<signal name="3.3V">
+<contactref element="U1" pad="2"/>
+<contactref element="U1" pad="4"/>
+<contactref element="C9" pad="1"/>
+<wire x1="3.81" y1="-146.761" x2="3.81" y2="-152.9588" width="0" layer="19" extent="1-1"/>
+<wire x1="15.11" y1="-147.32" x2="3.81" y2="-146.761" width="0" layer="19" extent="1-1"/>
+</signal>
+<signal name="5VI">
+<contactref element="U1" pad="3"/>
+<contactref element="C2" pad="1"/>
+<contactref element="IC2" pad="3"/>
+<contactref element="C5" pad="1"/>
+<wire x1="-22.86" y1="-151.13" x2="-31.88" y2="-176.53" width="0" layer="19" extent="1-1"/>
+<wire x1="6.1214" y1="-152.9588" x2="-22.86" y2="-151.13" width="0" layer="19" extent="1-1"/>
+<wire x1="8.76" y1="-147.32" x2="6.1214" y2="-152.9588" width="0" layer="19" extent="1-1"/>
+</signal>
+<signal name="VCKT">
+<contactref element="IC1" pad="1"/>
+<contactref element="C1" pad="1"/>
+<contactref element="IC2" pad="1"/>
+<contactref element="C4" pad="1"/>
+<wire x1="-31.88" y1="-157.48" x2="-31.88" y2="-170.18" width="0" layer="19" extent="1-1"/>
+<wire x1="-27.94" y1="-151.13" x2="-31.88" y2="-157.48" width="0" layer="19" extent="1-1"/>
+<wire x1="-11.43" y1="-151.13" x2="-27.94" y2="-151.13" width="0" layer="19" extent="1-1"/>
+</signal>
 </signals>

Commit message: Board file layout
Parts:
- added J5: XT-60BATT_LABEL, RoboJackets-Connectors:XT-60
- added S2: (no value), switch:A68-A31
- moved C5 300.8 mm to (152.4, 62.2), turned to 180 degrees
- moved C3 277.6 mm to (148.6, 48.3), turned to 180 degrees
- moved C1 275.9 mm to (146.1, 54.6), turned to 90 degrees
- moved C4 273.7 mm to (148.6, 36.8), turned to 180 degrees
- moved IC2 273.1 mm to (163.8, 55.9), flipped to the bottom, turned to 90 degrees
- moved IC1 251.5 mm to (163.8, 41.9), flipped to the bottom, turned to 90 degrees
- moved J4 225.6 mm to (100.3, 94.0), turned to 90 degrees
- moved U1 221.8 mm to (92.7, 53.3)
- moved C2 208.5 mm to (88.9, 45.7), turned to 180 degrees
- moved C9 208.5 mm to (95.2, 45.7), turned to 180 degrees
- moved J3 189.3 mm to (58.4, 94.0), turned to 90 degrees
- moved SV4 141.8 mm to (100.3, 83.8), turned to 180 degrees
- moved SV11 117.4 mm to (133.3, 43.2), turned to 180 degrees
- moved J2 114.8 mm to (101.6, -2.54), turned to 90 degrees
- moved SV12 114.8 mm to (133.3, 17.2), turned to 180 degrees
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Connections:
- new net N$1: J5.BATT, S2.2, S2.5
- net GND: now also J5.GND
- net VCKT: now also S2.3, S2.6
Other:
- board size 160 x 100 mm -> 172.7 x 110.2 mm

Commit message: Tst Board Comp
Parts:
- added U3: (no value), LP38690DT-3.3:TO228P1042X238-3N
- added X3: 22-23-2021, con-molex:22-23-2021
- added X4: 332-14, con-garry:332-14
Connections:
- removed net VCKT: C1.1, C4.1, IC1.1, IC2.1, S2.3, S2.6
- new net INPUT: J5.BATT, U3.1, U3.3
- new net N$10: X2.23, X4.10
- new net N$11: X2.21, X4.8
- new net N$12: X2.19, X4.6
- new net N$13: X2.17, X4.4
- new net N$14: X2.15, X4.2
- new net N$2: X1.18, X4.3
- new net N$25: S2.2, S2.5, U3.2
- new net N$3: X1.20, X4.5
- new net N$4: X1.22, X4.7
- new net N$5: X1.24, X4.9
- new net N$6: X1.26, X4.11
- new net N$7: X1.28, X4.13
- new net N$8: X2.27, X4.14
- new net N$9: X2.25, X4.12
- net 18V: now also C1.1, C4.1, IC1.1, IC2.1, S2.3, S2.6
- net 3.3V: now also X3.1
- net GND: now also X1.1, X1.39, X2.2, X2.40, X3.2
- net N$1: now also X1.16, X4.1; no longer J5.BATT, S2.2, S2.5
Routing:
- net 5V: track 0.00 -> 352.8 mm
- net GND: track 0.00 -> 305.9 mm, vias 0 -> 8
- net M12A: track 0.00 -> 164.6 mm, vias 0 -> 2
- net N$25: track 0.00 -> 117.3 mm
- net 5VI: track 0.00 -> 74.6 mm, vias 0 -> 1
- net 3.3V: track 0.00 -> 67.3 mm
- net M4EB: track 0.00 -> 65.6 mm, vias 0 -> 1
- net M32A: track 0.00 -> 65.4 mm, vias 0 -> 1
- net M4EA: track 0.00 -> 64.0 mm, vias 0 -> 2
- net M23: track 0.00 -> 58.8 mm
- net M22: track 0.00 -> 57.3 mm
- net M43B: track 0.00 -> 56.1 mm, vias 0 -> 1
- net M42B: track 0.00 -> 55.0 mm, vias 0 -> 2
- net M42A: track 0.00 -> 54.5 mm, vias 0 -> 1
- net M43A: track 0.00 -> 54.1 mm, vias 0 -> 1
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- added copper zone on layer 1, net 18V
- added copper zone on layer 16, net GND
Other:
- board size 172.7 x 110.2 mm -> 168.9 x 110.2 mm
