File: test boards/MotorTestBoard/FPGA.sch (EAGLE design)
At the start: 27 parts, among them IC1 7805T, IC2 7805T, X1 87758-4016, X2 87758-4016

Commit message: Board file layout
Parts:
- added J5: XT-60BATT_LABEL, RoboJackets-Connectors:XT-60BATT_LABEL
- added S2: (no value), switch:A68-A31
Connections:
- new net N$1: J5.+, S2A.P, S2B.P
- net GND: now also J5.-
- net VCKT: now also S2A.S, S2B.S
Other:
- note added: "POWER SUPPLY"
Changed lines of the file:
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@@
 <part name="C4" library="rcl" deviceset="C-EU" device="C1206" value="47uF"/>
 <part name="C5" library="rcl" deviceset="C-EU" device="C1206" value="47uF"/>
+<part name="GND12" library="SparkFun" deviceset="GND" device=""/>
+<part name="S2" library="switch" deviceset="A68-A31" device=""/>
+<part name="J5" library="RoboJackets-Connectors" deviceset="XT-60" device="BATT_LABEL"/>
 </parts>
 <sheets>
@@
 <wire x1="57.88" y1="-100.62" x2="58.03" y2="-66.33" width="0.1524" layer="94" style="longdash"/>
 <text x="66.63" y="-97" size="3.81" layer="94">POWER SUPPLY 3.3V</text>
+<text x="-99.06" y="-68.58" size="3.81" layer="94" ratio="31">POWER SUPPLY</text>
 </plain>
 <instances>
@@
 <instance part="C4" gate="G$1" x="110.82" y="-23.48"/>
 <instance part="C5" gate="G$1" x="133.68" y="-23.48"/>
+<instance part="GND12" gate="1" x="-124.46" y="-86.36" rot="MR0"/>
+<instance part="S2" gate="B" x="-106.68" y="-88.9" rot="R270"/>
+<instance part="S2" gate="A" x="-106.68" y="-76.2" rot="R270"/>
+<instance part="J5" gate="G$1" x="-142.24" y="-81.28"/>
 </instances>
 <busses>
@@
 <label x="119.38" y="-33.02" size="1.778" layer="95"/>
 </segment>
+<segment>
+<wire x1="-137.16" y1="-83.82" x2="-124.46" y2="-83.82" width="0.1524" layer="91"/>
+<pinref part="GND12" gate="1" pin="GND"/>
+<junction x="-124.46" y="-83.82"/>
+<pinref part="J5" gate="G$1" pin="-"/>
+</segment>
 </net>
 <net name="M21" class="0">
@@
 <segment>
 <pinref part="IC1" gate="A1" pin="VI"/>
-<wire x1="58.42" y1="-17.78" x2="60.96" y2="-17.78" width="0.1524" layer="91"/>
 <pinref part="C1" gate="G$1" pin="1"/>
 <wire x1="62.56" y1="-17.78" x2="68.58" y2="-17.78" width="0.1524" layer="91"/>
@@
 <wire x1="110.82" y1="-17.78" x2="111.76" y2="-17.78" width="0.1524" layer="91"/>
 <junction x="111.76" y="-17.78"/>
-<label x="106.68" y="-17.78" size="1.778" layer="95"/>
-</segment>
-</net>
+<label x="104.14" y="-17.78" size="1.778" layer="95"/>
+</segment>
+<segment>
+<pinref part="S2" gate="B" pin="S"/>
+<wire x1="-101.6" y1="-91.44" x2="-99.06" y2="-91.44" width="0.1524" layer="91"/>
+<wire x1="-99.06" y1="-91.44" x2="-99.06" y2="-86.36" width="0.1524" layer="91"/>
+<wire x1="-99.06" y1="-86.36" x2="-88.9" y2="-86.36" width="0.1524" layer="91"/>
+<pinref part="S2" gate="A" pin="S"/>
+<wire x1="-99.06" y1="-86.36" x2="-99.06" y2="-81.28" width="0.1524" layer="91"/>
+<wire x1="-99.06" y1="-81.28" x2="-101.6" y2="-81.28" width="0.1524" layer="91"/>
+<junction x="-99.06" y="-86.36"/>
+<label x="-93.98" y="-86.36" size="1.778" layer="95"/>
+</segment>
+</net>
+<net name="N$1" class="0">
+<segment>
+<pinref part="J5" gate="G$1" pin="+"/>
+<wire x1="-137.16" y1="-78.74" x2="-116.84" y2="-78.74" width="0.1524" layer="91"/>
+<pinref part="S2" gate="B" pin="P"/>
+<pinref part="S2" gate="A" pin="P"/>
+<wire x1="-111.76" y1="-78.74" x2="-111.76" y2="-88.9" width="0.1524" layer="91"/>
+<wire x1="-116.84" y1="-78.74" x2="-111.76" y2="-78.74" width="0.1524" layer="91"/>
+<junction x="-111.76" y="-78.74"/>
+</segment>
+</net>

Commit message: Tst Board Comp
Parts:
- added U3: (no value), LP38690DT-3.3:LP38690DT-3.3
- added X3: 22-23-2021, con-molex:22-23-2021
- added X4: 332-14, con-garry:332-14
Connections:
- removed net VCKT: C1.1, C4.1, IC1.VI, IC2.VI, S2A.S, S2B.S
- new net INPUT: J5.+, U3.A, U3.~A
- new net N$10: X2-23.S, X4-10.S
- new net N$11: X2-21.S, X4-8.S
- new net N$12: X2-19.S, X4-6.S
- new net N$13: X2-17.S, X4-4.S
- new net N$14: X2-15.S, X4-2.S
- new net N$2: X1-18.S, X4-3.S
- new net N$25: S2A.P, S2B.P, U3.K
- new net N$3: X1-20.S, X4-5.S
- new net N$4: X1-22.S, X4-7.S
- new net N$5: X1-24.S, X4-9.S
- new net N$6: X1-26.S, X4-11.S
- new net N$7: X1-28.S, X4-13.S
- new net N$8: X2-27.S, X4-14.S
- new net N$9: X2-25.S, X4-12.S
- net 18V: now also C1.1, C4.1, IC1.VI, IC2.VI, S2A.S, S2B.S
- net 3.3V: now also X3-1.S
- net GND: now also X1-1.S, X1-39.S, X2-2.S, X2-40.S, X3-2.S
- net N$1: now also X1-16.S, X4-1.S; no longer J5.+, S2A.P, S2B.P
Other:
- moved on the sheet: X2-1, X2-10, X2-11, X2-12, X2-13, X2-14, X2-15, X2-16, X2-17, X2-18, X2-19, X2-2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
