File: main_board/main_board-v3.1/main_board-v2.1.brd (EAGLE design)
At the start: 174.1 x 159 mm, 0 parts

Commit message: Mimas Added
Parts:
- added X3, X4: 87758-4016, con-molex:87758-4016
Changed lines of the file:
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@@
 <layer number="59" name="tCarbon" color="7" fill="1" visible="no" active="no"/>
 <layer number="60" name="bCarbon" color="7" fill="1" visible="no" active="no"/>
+<layer number="88" name="SimResults" color="9" fill="1" visible="no" active="no"/>
+<layer number="89" name="SimProbes" color="9" fill="1" visible="no" active="no"/>
 <layer number="90" name="Modules" color="5" fill="1" visible="no" active="no"/>
 <layer number="91" name="Nets" color="2" fill="1" visible="no" active="no"/>
@@
 </autorouter>
 <elements>
+<element name="X3" library="con-molex" library_urn="urn:adsk.eagle:library:165" package="87758-4016" value="87758-4016" x="61.491665625" y="82.29841875" locked="yes" rot="R90">
+<attribute name="MF" value="MOLEX" x="61.491665625" y="82.29841875" size="1.778" layer="27" rot="R90" display="off"/>
+<attribute name="MPN" value="87758-4016" x="61.491665625" y="82.29841875" size="1.778" layer="27" rot="R90" display="off"/>
+<attribute name="OC_FARNELL" value="unknown" x="61.491665625" y="82.29841875" size="1.778" layer="27" rot="R90" display="off"/>
+<attribute name="OC_NEWARK" value="25M5691" x="61.491665625" y="82.29841875" size="1.778" layer="27" rot="R90" display="off"/>
+</element>
+<element name="X4" library="con-molex" library_urn="urn:adsk.eagle:library:165" package="87758-4016" value="87758-4016" x="115.847665625" y="82.29841875" locked="yes" rot="R90">
+<attribute name="MF" value="MOLEX" x="115.847665625" y="82.29841875" size="1.778" layer="27" rot="R90" display="off"/>
+<attribute name="MPN" value="87758-4016" x="115.847665625" y="82.29841875" size="1.778" layer="27" rot="R90" display="off"/>
+<attribute name="OC_FARNELL" value="unknown" x="115.847665625" y="82.29841875" size="1.778" layer="27" rot="R90" display="off"/>
+<attribute name="OC_NEWARK" value="25M5691" x="115.847665625" y="82.29841875" size="1.778" layer="27" rot="R90" display="off"/>
+</element>
 </elements>
 <signals>
@@
 </drawing>
 <compatibility>
+<note version="8.2" severity="warning">
+Since Version 8.2, EAGLE supports online libraries. The ids
+of those online libraries will not be understood (or retained)
+with this version.
+</note>
 <note version="8.5" severity="warning">
 Since Version 8.5, EAGLE supports locking for holes, vias, wires and polygons.

Commit message: Components
Parts:
- added 12V, 3.3V, 5V1, BATTERY, BATTERY1, BATTERY2: (no value), led:CHIPLED_0805
- added C2, C9: 47uF, rcl:C1206
- added D2: 1N5817-B, diode:DO41-7.6
- added J1: XT-60BATT_LABEL, RoboJackets-Connectors:XT-60
- added J2, J3: F-1X02-SIP-100-32Y, con-headers-jp:SIP-100-02-32Y
- added R1, R25, R4, R7: 1k, resistor:R1206
- added R14, R2, R3: 4.7k, resistor:R1206
- added S2: (no value), switch:A68-A31
- added T1: 2N706, transistor:TO18
- added U$2: REL, rel:REL
- added U$3, U$4: BUCK, BUCK:BUCK
- added U$6: NODEMCU32S, nodeMCU:NODEMCU32
- added U1: (no value), SparkFun-PowerIC:SOT223
- added U2, U3, U4: (no value), LP38690DT-3.3:TO228P1042X238-3N
Connections:
- new net 12V: R7.1, U$4.VOUT
- new net 3.3V: C9.1, J3.2, R1.1, R25.2, U1.2, U1.4
- new net 3VESP: J3.1, U$6.P$38
- new net 5V: C2.1, J2.2, R4.2, T1.3, U$3.VOUT, U1.3
- new net 5VESP: J2.1, U$6.P$20
- new net BATT_LEVEL: U$2.NO, U2.1, U2.3, U4.1, U4.3
- new net ESP_ENABLE: U$6.P$37
- new net GND: 12V.C, 3.3V.C, 5V1.C, BATTERY.C, BATTERY1.C, BATTERY2.C, C2.2, C9.2, D2.A, J1.GND, U$2.2, U$3.GND, U$3.GNDO, U$4.GND, U$4.GNDO, U$6.P$13, U$6.P$19, U$6.P$21, U$6.P$25, U1.1
- new net INPUT: J1.BATT, U$2.C, U3.1, U3.3
- new net KICKER_RX: U$6.P$9
- new net KICKER_TX: U$6.P$8
- new net N$1: BATTERY1.A, R2.2
- new net N$14: 12V.A, R7.2
- new net N$18: BATTERY.A, R14.2
- new net N$19: 3.3V.A, R25.1
- new net N$2: BATTERY2.A, R3.2
- new net N$21: R1.2, T1.2
- new net N$22: D2.C, T1.1, U$2.1
- new net N$25: S2.2, S2.5, U3.2
- new net N$3: 5V1.A, R4.1
- new net U6_RX: U$6.P$16
- new net U6_TX: U$6.P$15
- new net VDC_1: R14.1, U$4.VIN, U4.2
- new net VDC_2: R2.1, U2.2
- new net V_CIRCUIT: R3.1, S2.3, S2.6, U$3.VIN

Commit message: Update
Parts:
- removed X3, X4: 87758-4016, con-molex:87758-4016
- added J4, J5, J6, J7: (no value), SparkFun-Connectors:2X5-SHROUDED_LOCK
- added SV10, SV12, SV16, SV8: (no value), con-lstb:MA10-1
- added SV11, SV15, SV3, SV4, SV5, SV6, SV7, SV9: (no value), con-lstb:MA08-1
Connections:
- new net 18V: SV10.10, SV10.9, SV12.10, SV12.9, SV16.10, SV16.9, SV8.10, SV8.9
- new net M11: SV3.8, SV7.6, SV7.7
- new net M11A: SV8.8
- new net M11B: SV8.7
- new net M12: SV3.7, SV7.4, SV7.5
- new net M12A: SV8.6
- new net M12B: SV8.5
- new net M13: SV3.6, SV7.2, SV7.3
- new net M13A: SV8.4
- new net M13B: SV8.3
- new net M1ACS_OUT: SV7.8
- new net M1EA: J4.6
- new net M1EB: J4.8
- new net M1H1: SV3.3
- new net M1H2: SV3.2
- new net M1H3: SV3.1
- new net M21: SV11.6, SV11.7, SV4.8
- new net M21A: SV12.8
- new net M21B: SV12.7
- new net M22: SV11.4, SV11.5, SV4.7
- new net M22A: SV12.6
- new net M22B: SV12.5
- new net M23: SV11.2, SV11.3, SV4.6
- new net M23A: SV12.4
- new net M23B: SV12.3
- new net M2ACS_OUT: SV11.8
- new net M2EA: J5.6
- new net M2EB: J5.8
- new net M2H1: SV4.3
- new net M2H2: SV4.2
- new net M2H3: SV4.1
- new net M31: SV15.6, SV15.7, SV5.8
- new net M31A: SV16.8
- new net M31B: SV16.7
- new net M32: SV15.4, SV15.5, SV5.7
- new net M32A: SV16.6
- new net M32B: SV16.5
- new net M33: SV15.2, SV15.3, SV5.6
- new net M33A: SV16.4
- new net M33B: SV16.3
- new net M3ACS_OUT: SV15.8
- new net M3EA: J6.6
- new net M3EB: J6.8
- new net M3H1: SV5.3
- new net M3H2: SV5.2
- new net M3H3: SV5.1
- new net M41: SV6.8, SV9.6, SV9.7
- new net M41A: SV10.8
- new net M41B: SV10.7
- new net M42: SV6.7, SV9.4, SV9.5
- new net M42A: SV10.6
- new net M42B: SV10.5
- new net M43: SV6.6, SV9.2, SV9.3
- new net M43A: SV10.4
- new net M43B: SV10.3
- new net M4ACS_OUT: SV9.8
- new net M4EA: J7.6
- new net M4EB: J7.8
- new net M4H1: SV6.3
- new net M4H2: SV6.2
- new net M4H3: SV6.1
- net 5V: now also J4.2, J5.2, J6.2, J7.2, SV11.1, SV15.1, SV3.5, SV4.5, SV5.5, SV6.5, SV7.1, SV9.1
- net GND: now also J4.3, J5.3, J6.3, J7.3, SV10.1, SV10.2, SV12.1, SV12.2, SV16.1, SV16.2, SV3.4, SV4.4, SV5.4, SV6.4, SV8.1, SV8.2
