File: main_board/MotorTestBoard/FPGA.brd (EAGLE design)
At the start: 174.1 x 159 mm, 32 parts, among them IC1 7805T, IC2 7805T, J5 XT-60BATT_LABEL, X3 22-23-2021, X4 332-14

Commit message: New Main CKt
Parts:
- moved J2 673.5 mm to (-181.5, 106.0), flipped to the bottom
- moved J5 647.2 mm to (-155.7, 113.9), flipped to the bottom, turned to 90 degrees
- moved SV3 574.8 mm to (-181.1, 96.2), flipped to the bottom
- moved SV1 563.4 mm to (-177.8, 8.03), flipped to the bottom, turned to 0 degrees
- moved J1 562.6 mm to (-177.7, -3.11), flipped to the bottom
- moved J4 555.8 mm to (-112.9, 106.2), flipped to the bottom
- moved SV4 555.5 mm to (-112.2, 96.4), flipped to the bottom
- moved SV2 547.4 mm to (-113.0, 7.75)
- moved J3 451.7 mm to (-113.0, -3.05), flipped to the bottom
- moved SV10 227.9 mm to (-94.5, 62.4)
- moved SV9 227.9 mm to (-94.5, 88.4)
- moved SV11 227.6 mm to (-94.3, 42.2)
- moved SV12 227.6 mm to (-94.3, 16.2)
- moved SV7 220.4 mm to (-196.3, 42.7)
- moved SV8 220.4 mm to (-196.3, 16.7)
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
Commit message: Update main board
Parts:
- removed C2, C9: 47uF, rcl:C1206
- removed U1: (no value), SparkFun-PowerIC:SOT223
- removed X3: 22-23-2021, con-molex:22-23-2021
- removed X4: 332-14, con-garry:332-14
- added SV5: (no value), con-lstb:MA08-1
- added U$1: NODEMCU32S, nodeMCU:NODEMCU32
- moved SV15 4.49 mm to (-192.0, 88.0)
- moved SV16 4.49 mm to (-192.0, 62.0)
- moved SV7 4.31 mm to (-192.0, 42.0)
- moved SV8 4.31 mm to (-192.0, 16.0)
- moved J1 3.79 mm to (-181.0, -5.00)
- moved SV1 3.20 mm to (-181.0, 8.00)
- moved J3 1.95 mm to (-113.0, -5.00)
- moved SV2 1.75 mm to (-113.0, 6.00)
- moved SV12 1.73 mm to (-96.0, 16.0)
- moved SV11 1.73 mm to (-96.0, 42.0)
- moved SV10 1.51 mm to (-96.0, 62.0)
- moved SV9 1.51 mm to (-96.0, 88.0)
- moved SV3 0.17 mm to (-181.0, 96.0)
Connections:
- removed net 3.3V: C9.1, U1.2, U1.4, X3.1
- removed net 5VI: C2.1, C5.1, IC2.3, U1.3
- removed net N$1: X4.1
- removed net N$10: X4.10
- removed net N$11: X4.8
- removed net N$12: X4.6
- removed net N$13: X4.4
- removed net N$14: X4.2
- removed net N$3: X4.5
- removed net N$4: X4.7
- removed net N$5: X4.9
- removed net N$6: X4.11
- removed net N$7: X4.13
- removed net N$8: X4.14
- removed net N$9: X4.12
- new net 5V1: C5.1, IC2.3, U$1.P$20
- new net CHARGE: JP2.16, SV5.1
- new net DONE: JP2.18, SV5.2
- new net ESP_EN: JP2.25, U$1.P$37
- new net ESP_RX: JP2.21, U$1.P$15
- new net ESP_TX: JP2.23, U$1.P$16
- new net IR1: JP2.24, SV5.7
- new net IR2: JP2.26, SV5.6
- new net IR3: JP2.15, SV5.5
- new net KICK: JP2.20, SV5.4
- new net KICK_CHIP: JP2.22, SV5.3
- net GND: now also JP1.1, JP1.39, JP2.2, JP2.40, SV5.8, U$1.P$13, U$1.P$19, U$1.P$21, U$1.P$25; no longer C2.2, C9.2, U1.1, X3.2
- net M11A: now also JP1.3
- net M11B: now also JP1.5
- net M12A: now also JP1.7
- net M12B: now also JP1.9
- net M13A: now also JP1.11
- net M13B: now also JP1.13
- net M1EA: now also JP1.4
- net M1EB: now also JP1.6
- net M1H1: now also JP1.8
- net M1H2: now also JP1.10
- net M1H3: now also JP1.12
- net M21A: now also JP1.27
- net M21B: now also JP1.29
- net M22A: now also JP1.31
- net M22B: now also JP1.33
- net M23A: now also JP1.35
- net M23B: now also JP1.37
- net M2EA: now also JP1.30
- net M2EB: now also JP1.32
- net M2H1: now also JP1.34
- net M2H2: now also JP1.36
- net M2H3: now also JP1.38
- net M31A: now also JP2.4
- net M31B: now also JP2.6
- net M32A: now also JP2.8
- net M32B: now also JP2.10
- net M33A: now also JP2.12
- net M33B: now also JP2.14
- net M3EA: now also JP2.3
- net M3EB: now also JP2.5
- net M3H1: now also JP2.7
- net M3H2: now also JP2.9
- net M3H3: now also JP2.11
- net M41A: now also JP2.28
- net M41B: now also JP2.30
- net M42A: now also JP2.32
- net M42B: now also JP2.34
- net M43A: now also JP2.36
- net M43B: now also JP2.38
- net M4EA: now also JP2.29
- net M4EB: now also JP2.31
- net M4H1: now also JP2.33
- net M4H2: now also JP2.35
- net M4H3: now also JP2.37
- net N$2: now also U$1.P$17; no longer X4.3

Commit message: New Dimensions for Main CKT
Parts:
- added SV14: (no value), con-lstb:MA10-1
- added SV17, SV18: (no value), con-lstb:MA08-1
- moved U3 483.9 mm to (-6.11, 54.2), flipped to the bottom, turned to 180 degrees
- moved U$1 403.9 mm to (12.2, 2.51), flipped to the bottom
- moved SV5 376.5 mm to (1.67, -74.2), flipped to the bottom
- moved J4 158.1 mm to (34.3, 48.7)
- moved JP1 158.1 mm to (-25.7, -8.00)
- moved SV4 158.1 mm to (35.1, 38.9)
- moved J1 158.1 mm to (-33.8, -62.5)
- moved J2 158.1 mm to (-34.3, 48.5)
- moved J3 158.1 mm to (34.2, -62.5)
- moved JP2 158.1 mm to (28.6, -8.00)
- moved SV1 158.1 mm to (-33.8, -49.5)
- moved SV10 158.1 mm to (51.2, 4.51)
- moved SV11 158.1 mm to (51.2, -15.5)
- moved SV12 158.1 mm to (51.2, -41.5)
- moved SV15 158.1 mm to (-44.8, 30.5)
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Other:
- board size 174.1 x 159 mm -> 278 x 208.3 mm

Commit message: Placements
Parts:
- added U$4: BUCK, BUCK:BUCK
- added U1, U2: (no value), LP38690DT-3.3:TO228P1042X238-3N
- moved J4 108.9 mm to (40.0, -60.0)
- moved SV11 101.2 mm to (-50.0, -15.0)
- moved SV12 101.2 mm to (-50.0, -41.0)
- moved J2 97.3 mm to (50.0, 0.00)
- moved SV15 95.9 mm to (50.0, 45.0)
- moved SV16 95.9 mm to (50.0, 19.0)
- moved SV4 90.0 mm to (40.0, -51.0), turned to 0 degrees
- moved SV3 88.8 mm to (50.0, 9.00), turned to 0 degrees
- moved J3 74.3 mm to (-40.0, -60.0)
- moved SV2 74.2 mm to (-40.0, -51.0), flipped to the bottom, turned to 0 degrees
- moved J1 64.6 mm to (-50.0, 0.00)
- moved SV7 60.7 mm to (-50.0, 45.0)
- moved SV8 60.7 mm to (-50.0, 19.0)
- moved SV1 60.7 mm to (-50.0, 9.00)
- moved SV9 45.5 mm to (50.0, -15.0)
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Connections:
- new net 12V: C1.1, C4.1, IC1.1, IC2.1, SV14.10, SV14.9, U$4.VOUT
- new net MD1: SV17.6, SV17.7, SV18.8
- new net MD1A: JP1.15, SV14.8
- new net MD1B: JP1.17, SV14.7
- new net MD2: SV17.4, SV17.5, SV18.7
- new net MD2A: JP1.19, SV14.6
- new net MD2B: JP1.21, SV14.5
- new net MD3: SV17.2, SV17.3, SV18.6
- new net MD3A: JP1.23, SV14.4
- new net MD3B: JP1.25, SV14.3
- new net MDACS_OUT: SV17.8
- new net MDH1: JP1.16, SV18.3
- new net MDH2: JP1.18, SV18.2
- new net MDH3: JP1.20, SV18.1
- net 18V: now also U$4.VIN; no longer C1.1, C4.1, IC1.1, IC2.1
- net 5V: now also SV17.1, SV18.5; no longer SV11.1, SV15.1, SV7.1, SV9.1
- net 5V1: now also SV11.1, SV15.1, SV7.1, SV9.1
- net GND: now also SV14.1, SV14.2, SV18.4, U$4.GND, U$4.GNDO
- net INPUT: now also U1.1, U1.3, U2.1, U2.3
Other:
- outline, holes or cut-outs redrawn

Commit message: Sch Comp
Parts:
- removed S2: (no value), switch:A68-A31
- added LED1, LED2, LED3, LED4, LED5, LED6, LED7: (no value), led:1206
- added R1, R2, R3, R4, R5, R6, R7: (no value), resistor:R1206
- added U$5: (no value), switch_DA10:DA10
Connections:
- removed net N$25: S2.2, S2.5, U3.2
- new net ESP_REC: R7.1, U$1.P$33
- new net ESP_TRANS: R6.1, U$1.P$34
- new net FPGA_REC: JP1.22, R5.1
- new net N$1: J5.BATT, U$5.P$2
- new net N$10: LED3.A, R3.2
- new net N$13: LED4.A, R4.2
- new net N$16: LED5.A, R5.2
- new net N$19: LED6.A, R6.2
- new net N$22: LED7.A, R7.2
- new net N$4: LED1.A, R1.2
- new net N$7: LED2.A, R2.2
- net 12V: now also R4.1
- net 18V: now also R3.1, U1.2, U2.2, U3.2; no longer S2.3, S2.6
- net 5V: now also R2.1
- net 5V1: now also R1.1
- net GND: now also LED1.C, LED2.C, LED3.C, LED4.C, LED5.C, LED6.C, LED7.C
- net INPUT: now also U$5.P$1; no longer J5.BATT

Commit message: Route Complete
Parts:
- moved LED7 532.3 mm to (80.8, 10.0)
- moved R7 531.2 mm to (72.8, 10.0)
- moved LED6 523.0 mm to (80.8, 7.00)
- moved R6 521.8 mm to (72.8, 7.00)
- moved LED5 513.8 mm to (80.8, 4.00)
- moved R5 512.5 mm to (72.8, 4.00)
- moved LED4 504.7 mm to (80.8, 1.00)
- moved R4 503.3 mm to (72.8, 1.00)
- moved IC1 500.5 mm to (43.2, 61.7), turned to 0 degrees
- moved IC2 496.0 mm to (32.6, 61.7), turned to 0 degrees
- moved LED3 493.3 mm to (80.8, -5.00)
- moved R3 491.7 mm to (72.8, -5.00)
- moved C4 489.3 mm to (45.7, 55.8), flipped to the bottom, turned to 0 degrees
- moved LED1 485.8 mm to (80.8, -2.00)
- moved LED2 484.4 mm to (80.8, -8.00)
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Connections:
- net N$1 renamed SUPP
Routing:
- net 5V: track 0.00 -> 383.5 mm
- net 5V1: track 0.00 -> 264.1 mm, vias 0 -> 1
- net 12V: track 0.00 -> 150.9 mm
- net M3EA: track 0.00 -> 112.5 mm
- net FPGA_REC: track 0.00 -> 110.5 mm, vias 0 -> 1
- net M3EB: track 0.00 -> 107.9 mm
- net ESP_REC: track 0.00 -> 103.7 mm, vias 0 -> 1
- net ESP_TRANS: track 0.00 -> 101.6 mm, vias 0 -> 1
- net DONE: track 0.00 -> 100.3 mm
- net M2EB: track 0.00 -> 97.4 mm
- net IR1: track 0.00 -> 88.4 mm
- net M2EA: track 0.00 -> 87.3 mm, vias 0 -> 1
- net CHARGE: track 0.00 -> 80.0 mm
- net IR3: track 0.00 -> 79.6 mm
- net KICK: track 0.00 -> 78.3 mm, vias 0 -> 2
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- added copper zone on layer 1, net 18V
- added copper zone on layer 2, net 18V
- added copper zone on layer 1, net GND
- added copper zone on layer 15, net GND
- added copper zone on layer 1, net INPUT
- added copper zone on layer 1, net SUPP
Other:
- board size 278 x 208.3 mm -> 171.1 x 156.6 mm
