File: main_board/FPGA_board-v1/FPGA.sch (EAGLE design)
At the start: 35 parts, among them IC1 7805T, IC2 7805T, J5 XT-60BATT_LABEL

Commit message: Updates
Parts:
- removed S2: (no value), switch:A68-A31
- added LED1, LED2, LED3, LED4, LED5, LED6, LED7: (no value), led:LEDSMT1206
- added R1, R2, R3, R4, R5, R6, R7: (no value), resistor:R-EU_R1206
- added U$5: (no value), switch_DA10:SWITCH_DA10
- added X1: 22-23-2021, con-molex:22-23-2021
Connections:
- removed net N$25: S2A.P, S2B.P, U3.K
- new net ESP_REC: R7.1, U$1.P35
- new net ESP_TRANS: R6.1, U$1.P34
- new net FPGA_REC: JP1.22, R5.1
- new net N$10: LED3.A, R3.2
- new net N$13: LED4.A, R4.2
- new net N$16: LED5.A, R5.2
- new net N$19: LED6.A, R6.2
- new net N$22: LED7.A, R7.2
- new net N$4: LED1.A, R1.2
- new net N$7: LED2.A, R2.2
- new net SUPP: J5.+, U$5.P
- net 12V: now also R4.1
- net 18V: now also R3.1, U1.K, U2.K, U3.K; no longer S2A.S, S2B.S
- net 5V: now also R2.1
- net 5V1: now also R1.1, X1-2.S
- net GND: now also LED1.C, LED2.C, LED3.C, LED4.C, LED5.C, LED6.C, LED7.C, X1-1.S
- net INPUT: now also U$5.S; no longer J5.+
Other:
- moved on the sheet: C1, C3, C4, C5, IC1, IC2, J5
