File: main_board/FPGA_board-v1/FPGA_board-v1.sch (EAGLE design)
At the start: 50 parts, among them IC1 7805T, IC2 7805T, J5 XT-60BATT_LABEL, X1 22-23-2021

Commit message: ESP Update
Parts:
- removed U$1: NODEMCU32S, nodeMCU:NODEMCU32S
- added JP5, JP6: (no value), pinhead:PINHD-2X15
Connections:
- removed net N$2: U$1.P22
- new net N$1: JP5.1, JP5.2
- new net N$11: JP5.11, JP5.12
- new net N$12: JP5.13, JP5.14
- new net N$14: JP5.15, JP5.16
- new net N$15: JP5.17, JP5.18
- new net N$17: JP5.19, JP5.20
- new net N$18: JP5.21, JP5.22
- new net N$23: JP5.27, JP5.28
- new net N$24: JP5.29, JP5.30
- new net N$27: JP6.5, JP6.6
- new net N$28: JP6.7, JP6.8
- new net N$29: JP6.10, JP6.9
- new net N$30: JP6.11, JP6.12
- new net N$31: JP6.13, JP6.14
- new net N$34: JP6.19, JP6.20
- new net N$35: JP6.21, JP6.22
- new net N$38: JP6.27, JP6.28
- new net N$39: JP6.29, JP6.30
- new net N$6: JP5.5, JP5.6
- new net N$8: JP5.7, JP5.8
- new net N$9: JP5.10, JP5.9
- net 5V1: now also JP6.1, JP6.2; no longer U$1.5V
- net ESP_EN: no longer U$1.SEN
- net ESP_REC: now also JP6.15, JP6.16; no longer U$1.P35
- net ESP_RX: now also JP5.23, JP5.24; no longer U$1.RX
- net ESP_TRANS: now also JP6.17, JP6.18; no longer U$1.P34
- net ESP_TX: now also JP5.25, JP5.26; no longer U$1.TX
- net GND: now also JP5.3, JP5.4, JP6.3, JP6.4; no longer U$1.GND, U$1.GND1, U$1.GND2, U$1.GND3
Other:
- note added: "12V"
- note added: "5V"
- note added: "5V1"
- note added: "Dribbler"
- note added: "ESP32"
- note added: "FPGA"
- note added: "Input"
- note added: "Kicker"
- note added: "Motor Driver"
- note added: "Power Supply"
- note added: "Status LED"
- note removed: "POWER SUPPLY"
- moved on the sheet: C1, C3, C4, C5, IC1, IC2, J1, J2, J3, J4, J5, JP1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

Commit message: Current Sensing
Parts:
- added C2, C6, C7, C8: 47uF, rcl:C-EUC1206
Connections:
- removed net N$31: JP6.13, JP6.14
- removed net N$34: JP6.19, JP6.20
- removed net N$35: JP6.21, JP6.22
- new net N$41: JP6.25, JP6.26
- net ESP_TRANS: now also JP6.13, JP6.14; no longer JP6.17, JP6.18
- net GND: now also C2.1, C6.1, C7.1, C8.1
- net M1ACS_OUT: now also C2.2, JP6.17, JP6.18
- net M2ACS_OUT: now also C6.2, JP6.19, JP6.20
- net M3ACS_OUT: now also C7.2, JP6.21, JP6.22
- net M4ACS_OUT: now also C8.2, JP6.23, JP6.24
Changed lines of the file:
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@@
 <part name="JP5" library="pinhead" library_urn="urn:adsk.eagle:library:325" deviceset="PINHD-2X15" device="" package3d_urn="urn:adsk.eagle:package:22427/2"/>
 <part name="JP6" library="pinhead" library_urn="urn:adsk.eagle:library:325" deviceset="PINHD-2X15" device="" package3d_urn="urn:adsk.eagle:package:22427/2"/>
+<part name="C2" library="rcl" deviceset="C-EU" device="C1206" value="47uF"/>
+<part name="C6" library="rcl" deviceset="C-EU" device="C1206" value="47uF"/>
+<part name="C7" library="rcl" deviceset="C-EU" device="C1206" value="47uF"/>
+<part name="C8" library="rcl" deviceset="C-EU" device="C1206" value="47uF"/>
 </parts>
 <sheets>
@@
 <instance part="JP5" gate="A" x="-233.68" y="-129.54"/>
 <instance part="JP6" gate="A" x="-200.66" y="-129.54"/>
+<instance part="C2" gate="G$1" x="-230.2" y="-169.56" rot="R180"/>
+<instance part="C6" gate="G$1" x="-222.58" y="-169.56" rot="R180"/>
+<instance part="C7" gate="G$1" x="-214.96" y="-169.56" rot="R180"/>
+<instance part="C8" gate="G$1" x="-207.34" y="-169.56" rot="R180"/>
 </instances>
 <busses>
@@
 <label x="-251.46" y="-114.3" size="1.778" layer="95"/>
 </segment>
+<segment>
+<pinref part="C2" gate="G$1" pin="1"/>
+<pinref part="C6" gate="G$1" pin="1"/>
+<wire x1="-230.2" y1="-172.1" x2="-222.58" y2="-172.1" width="0.1524" layer="91"/>
+<pinref part="C7" gate="G$1" pin="1"/>
+<wire x1="-222.58" y1="-172.1" x2="-214.96" y2="-172.1" width="0.1524" layer="91"/>
+<junction x="-222.58" y="-172.1"/>
+<pinref part="C8" gate="G$1" pin="1"/>
+<wire x1="-214.96" y1="-172.1" x2="-207.34" y2="-172.1" width="0.1524" layer="91"/>
+<junction x="-214.96" y="-172.1"/>
+<label x="-223.52" y="-175.26" size="1.778" layer="95"/>
+</segment>
 </net>
 <net name="M21" class="6">
@@
 <label x="-73.66" y="-10.16" size="1.778" layer="95"/>
 </segment>
+<segment>
+<pinref part="JP6" gate="A" pin="18"/>
+<pinref part="JP6" gate="A" pin="17"/>
+<wire x1="-195.58" y1="-132.08" x2="-203.2" y2="-132.08" width="0.1524" layer="91"/>
+<wire x1="-203.2" y1="-132.08" x2="-213.36" y2="-132.08" width="0.1524" layer="91"/>
+<junction x="-203.2" y="-132.08"/>
+<label x="-223.52" y="-132.08" size="1.778" layer="95"/>
+</segment>
+<segment>
+<pinref part="C2" gate="G$1" pin="2"/>
+<wire x1="-230.2" y1="-164.48" x2="-230.2" y2="-160.02" width="0.1524" layer="91"/>
+<wire x1="-230.2" y1="-160.02" x2="-228.6" y2="-160.02" width="0.1524" layer="91"/>
+<label x="-231.14" y="-165.1" size="1.778" layer="95" rot="R90"/>
+</segment>
 </net>
 <net name="M2ACS_OUT" class="0">
@@
 <label x="-73.66" y="-43.18" size="1.778" layer="95"/>
 </segment>
+<segment>
+<pinref part="JP6" gate="A" pin="19"/>
+<pinref part="JP6" gate="A" pin="20"/>
+<wire x1="-203.2" y1="-134.62" x2="-195.58" y2="-134.62" width="0.1524" layer="91"/>
+<wire x1="-203.2" y1="-134.62" x2="-213.36" y2="-134.62" width="0.1524" layer="91"/>
+<junction x="-203.2" y="-134.62"/>
+<label x="-223.52" y="-134.62" size="1.778" layer="95"/>
+</segment>
+<segment>
+<pinref part="C6" gate="G$1" pin="2"/>
+<wire x1="-222.58" y1="-164.48" x2="-222.58" y2="-160.02" width="0.1524" layer="91"/>
+<wire x1="-222.58" y1="-160.02" x2="-220.98" y2="-160.02" width="0.1524" layer="91"/>
+<label x="-223.52" y="-165.1" size="1.778" layer="95" rot="R90"/>
+</segment>
 </net>
 <net name="M3ACS_OUT" class="0">
@@
 <label x="-73.66" y="-76.2" size="1.778" layer="95"/>
 </segment>
+<segment>
+<pinref part="JP6" gate="A" pin="22"/>
+<pinref part="JP6" gate="A" pin="21"/>
+<wire x1="-195.58" y1="-137.16" x2="-203.2" y2="-137.16" width="0.1524" layer="91"/>
+<wire x1="-203.2" y1="-137.16" x2="-213.36" y2="-137.16" width="0.1524" layer="91"/>
+<junction x="-203.2" y="-137.16"/>
+<label x="-223.52" y="-137.16" size="1.778" layer="95"/>
+</segment>
+<segment>
+<pinref part="C7" gate="G$1" pin="2"/>
+<wire x1="-214.96" y1="-164.48" x2="-214.96" y2="-160.02" width="0.1524" layer="91"/>
+<wire x1="-214.96" y1="-160.02" x2="-213.36" y2="-160.02" width="0.1524" layer="91"/>
+<label x="-215.9" y="-165.1" size="1.778" layer="95" rot="R90"/>
+</segment>
 </net>
 <net name="M4ACS_OUT" class="0">
@@
 <wire x1="-73.66" y1="-109.22" x2="-66.04" y2="-109.22" width="0.1524" layer="91"/>
 <label x="-73.66" y="-109.22" size="1.778" layer="95"/>
+</segment>
+<segment>
+<pinref part="JP6" gate="A" pin="24"/>
+<pinref part="JP6" gate="A" pin="23"/>
+<wire x1="-195.58" y1="-139.7" x2="-203.2" y2="-139.7" width="0.1524" layer="91"/>
+<wire x1="-203.2" y1="-139.7" x2="-213.36" y2="-139.7" width="0.1524" layer="91"/>
+<junction x="-203.2" y="-139.7"/>
+<label x="-223.52" y="-139.7" size="1.778" layer="95"/>
+</segment>
+<segment>
+<pinref part="C8" gate="G$1" pin="2"/>
+<wire x1="-207.34" y1="-164.48" x2="-207.34" y2="-160.02" width="0.1524" layer="91"/>
+<wire x1="-207.34" y1="-160.02" x2="-205.74" y2="-160.02" width="0.1524" layer="91"/>
+<label x="-208.28" y="-165.1" size="1.778" layer="95" rot="R90"/>
 </segment>
 </net>
@@
 </segment>
 <segment>
-<pinref part="JP6" gate="A" pin="18"/>
-<pinref part="JP6" gate="A" pin="17"/>
-<wire x1="-195.58" y1="-132.08" x2="-203.2" y2="-132.08" width="0.1524" layer="91"/>
-<wire x1="-203.2" y1="-132.08" x2="-213.36" y2="-132.08" width="0.1524" layer="91"/>
-<junction x="-203.2" y="-132.08"/>
-<label x="-223.52" y="-132.08" size="1.778" layer="95"/>
+<pinref part="JP6" gate="A" pin="14"/>
+<pinref part="JP6" gate="A" pin="13"/>
+<wire x1="-195.58" y1="-127" x2="-203.2" y2="-127" width="0.1524" layer="91"/>
+<wire x1="-203.2" y1="-127" x2="-213.36" y2="-127" width="0.1524" layer="91"/>
+<junction x="-203.2" y="-127"/>
+<label x="-223.52" y="-127" size="1.778" layer="95"/>
 </segment>
 </net>
@@
 </segment>
 </net>
-<net name="N$31" class="0">
-<segment>
-<pinref part="JP6" gate="A" pin="14"/>
-<pinref part="JP6" gate="A" pin="13"/>
-<wire x1="-195.58" y1="-127" x2="-203.2" y2="-127" width="0.1524" layer="91"/>
-<wire x1="-203.2" y1="-127" x2="-213.36" y2="-127" width="0.1524" layer="91"/>
-<junction x="-203.2" y="-127"/>
-</segment>
-</net>
-<net name="N$34" class="0">
-<segment>
-<pinref part="JP6" gate="A" pin="19"/>
-<pinref part="JP6" gate="A" pin="20"/>
-<wire x1="-203.2" y1="-134.62" x2="-195.58" y2="-134.62" width="0.1524" layer="91"/>
-<wire x1="-203.2" y1="-134.62" x2="-213.36" y2="-134.62" width="0.1524" layer="91"/>
-<junction x="-203.2" y="-134.62"/>
-</segment>
-</net>
-<net name="N$35" class="0">
-<segment>
-<pinref part="JP6" gate="A" pin="22"/>
-<pinref part="JP6" gate="A" pin="21"/>
-<wire x1="-195.58" y1="-137.16" x2="-203.2" y2="-137.16" width="0.1524" layer="91"/>
-<wire x1="-203.2" y1="-137.16" x2="-213.36" y2="-137.16" width="0.1524" layer="91"/>
-<junction x="-203.2" y="-137.16"/>
-</segment>
-</net>
 <net name="N$38" class="0">
 <segment>
@@
 </segment>
 </net>
+<net name="N$41" class="0">
+<segment>
+<pinref part="JP6" gate="A" pin="25"/>
+<pinref part="JP6" gate="A" pin="26"/>
+<wire x1="-203.2" y1="-142.24" x2="-195.58" y2="-142.24" width="0.1524" layer="91"/>
+</segment>
+</net>
