File: kicker/kicker-v2.3/kicker-v2.3.brd (EAGLE design)
At the start: 152.8 x 55 mm, 43 parts, among them IC1 7818TV, IC2 MCP601OT, J1 XT-60BATT_LABEL, Q1 IGB50N60T, Q3 IGB50N60T, U1 LT3750EMSPBF

Commit message: Error Correction
Parts:
- moved R1 3.80 mm to (-15.2, -1.77)
- moved R2 3.35 mm to (-18.5, -1.82)
- moved R5 2.35 mm to (-39.2, 5.25)
Connections:
- removed net VTRANS: U$6.8, U$7.8
- net V_TRANS: now also U$6.8, U$7.8
Routing:
- net VTRANS: track 22.1 -> 0.00 mm
- net V_TRANS: track 177.4 -> 197.8 mm
- net SINK: track 9.76 -> 28.9 mm
- net 5V: track 137.9 -> 145.2 mm
- net DONE: track 14.1 -> 19.9 mm, vias 2 -> 0
- net RVOUT: track 8.42 -> 13.1 mm
- net RDCM: track 13.0 -> 9.72 mm
- net CHARGE: track 10.8 -> 12.1 mm
Other:
- board size 152.8 x 55 mm -> 152.9 x 55 mm
