File: kicker/kicker-v2.3/kicker-V2.3.sch (EAGLE design)
At the start: 43 parts, among them IC1 7818TV, IC2 MCP601OT, J1 XT-60BATT_LABEL, Q1 IGB50N60T, Q3 IGB50N60T, U1 LT3750EMSPBF

Commit message: Error Correction
Connections:
- removed net VTRANS: U$6.VCC, U$7.VCC
- net V_TRANS: now also U$6.VCC, U$7.VCC
Changed lines of the file:
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@@
 <?xml version="1.0" encoding="utf-8"?>
 <!DOCTYPE eagle SYSTEM "eagle.dtd">
-<eagle version="7.7.0">
+<eagle version="9.1.3">
 <drawing>
 <settings>
 <setting alwaysvectorfont="no"/>
+<setting keepoldvectorfont="yes"/>
 <setting verticaltext="up"/>
 </settings>
@@
 <label x="-184.15" y="-15.24" size="1.27" layer="95" rot="R180" xref="yes"/>
 </segment>
+<segment>
+<pinref part="U$6" gate="G$1" pin="VCC"/>
+<wire x1="110.49" y1="48.26" x2="114.3" y2="48.26" width="0.1524" layer="91"/>
+<wire x1="114.3" y1="48.26" x2="114.3" y2="54.61" width="0.1524" layer="91"/>
+<label x="114.3" y="54.61" size="1.778" layer="95" rot="R90" xref="yes"/>
+</segment>
+<segment>
+<pinref part="U$7" gate="G$1" pin="VCC"/>
+<wire x1="237.49" y1="48.26" x2="241.3" y2="48.26" width="0.1524" layer="91"/>
+<wire x1="241.3" y1="48.26" x2="241.3" y2="54.61" width="0.1524" layer="91"/>
+<label x="241.3" y="54.61" size="1.778" layer="95" rot="R90" xref="yes"/>
+</segment>
 </net>
 <net name="CHARGE" class="0">
@@
 </segment>
 </net>
-<net name="VTRANS" class="0">
-<segment>
-<pinref part="U$6" gate="G$1" pin="VCC"/>
-<wire x1="110.49" y1="48.26" x2="114.3" y2="48.26" width="0.1524" layer="91"/>
-<wire x1="114.3" y1="48.26" x2="114.3" y2="54.61" width="0.1524" layer="91"/>
-<label x="114.3" y="54.61" size="1.778" layer="95" rot="R90" xref="yes"/>
-</segment>
-<segment>
-<pinref part="U$7" gate="G$1" pin="VCC"/>
-<wire x1="237.49" y1="48.26" x2="241.3" y2="48.26" width="0.1524" layer="91"/>
-<wire x1="241.3" y1="48.26" x2="241.3" y2="54.61" width="0.1524" layer="91"/>
-<label x="241.3" y="54.61" size="1.778" layer="95" rot="R90" xref="yes"/>
-</segment>
-</net>

Commit message: Update Kicker
Parts:
- added R15, R16, R9: 2.49K, resistor:R-US_M1206
Connections:
- net CHARGE: now also R16.2
- net GND: now also R15.1, R16.1, R9.1
- net TRIGGER: now also R15.2
- net TRIGGER_CHIP: now also R9.2
