File: main_board/main_board-v1/main_board-v1.brd (EAGLE design)
At the start: 163.3 x 159.3 mm, 108 parts, among them J1 XT-60BATT_LABEL, T1 2N706, T6 BC547, T7 BC547, T8 BC547, T9 BC547

Commit message: main board
Parts:
- removed 3.3V, BATTERY, TESTLED1, TESTLED2: (no value), led:CHIPLED_1206
- removed C14, C15: 20pF, rcl:C1206
- removed C16, C17, C18, C19, C20: 50uF, adafruit:E3,5-8
- removed D2: 1N5817-B, diode:DO41-7.6
- removed JP12, JP13: FRC_25, mohit:FRC2*5
- removed R14: 4.7k, resistor:R1206
- removed R2: 220, resistor:R1206
- removed R3: 10k, resistor:R1206
- removed R6, R7: 1k, resistor:R1206
- removed S10, S2, S7, S8, S9: (no value), switch:A68-A31
- removed SV13: (no value), con-lsta:FE06
- removed SV16, SV17, SV18: (no value), con-lsta:FE13-2
- removed SV5: (no value), con-lstb:MA08-1
- removed T6, T7, T8, T9: BC547, transistor:TO92
- removed TP10, TP19, TP20, TP21, TP22, TP23, TP24, TP25, TP26, TP3, TP4, TP5, TP6, TP7, TP8, TP9: PTR1PAD1-13, testpad:P1-13
- removed U$5: (no value), switch_DA10:DA10
- added D3: BYD13, diode:SOD81
- added GND, GND2, GND_12V, GND_5V, V_BAT, V_BAT_12V: PINHEAD_1, pinhead_1:PINHEAD_1
- added JP1, JP2, JP5, JP7, JP9: FRC_SSL, frc:FRC
- added JP11: (no value), adafruit:1X03
- added LED1, LED8, LED9, LED_12V, LED_3.3V, LED_5V, LED_8V: (no value), led:CHIPLED_1206
- added M1: WIRELESS-NRF24L01, diy-modules:WIRELESS-NRF24L01
- added R11: 1k, resistor:R1206
- added R16, R17, R18, R19, R20, R21, R22, R23: 10k, resistor:R1206
- added R8: 47k, resistor:R1206
- added SV15: (no value), con-lsta:FE05-1
- added SW1: (no value), special:EDG-04
- added T2, T3, T4: BC547, transistor:TO92
- 12V, 5V: value (none) -> PINHEAD_1; device led:CHIPLED_1206 -> pinhead_1:PINHEAD_1
- Q1: device crystal:HC49U-V -> TRANSISTOR-NPN:TO-92
- R1: value 1k -> (none); device resistor:R1206 -> resistor:M0805
- R12: value 1k -> (none)
- R24, R28: value 10k -> 1k
- R26: value 10k -> 27k
- R27: value 10k -> 140k
- R29: value 10k -> 4.7k
- R4, R5: value 10k -> 22
- SV1: device con-lstb:MA08-1 -> con-lstb:MA05-1
- SV10: device con-lsta:FE13-2 -> con-lsta:FE05-1
- SV11, SV3, SV7, SV9: device con-lsta:FE05-2 -> con-lsta:FE13
- SV12: device con-lsta:FE05-2 -> con-lsta:FE05-1
- SV14: device con-lstb:MA03-1 -> con-lsta:FE13
- SV2: device con-lstb:MA08-1 -> con-lsta:FE08
- SV4, SV8: device con-lstb:MA08-1 -> con-lsta:FE05-1
- SV6: device con-lsta:FE13-2 -> con-lstb:MA06-1
- T1: value 2N706 -> BC547; device transistor:TO18 -> transistor:TO92
- U$2: value REL -> XBEE-1B2; device rel:REL -> SparkFun:XBEE-SILK
- U$3: value BUCK -> (none); device BUCK:BUCK -> switch_DA10:DA10
- U$4: value BUCK -> USB-MICRO-B-FEMALE; device BUCK:BUCK -> USB-MICRO-B-FEMALE:USB-MICRO-B-FEMALE
- moved SV11 176.6 mm to (51.3, 138.0), turned to 225 degrees
- moved SV12 163.4 mm to (63.9, 118.3), turned to 45 degrees
- moved R1 158.8 mm to (73.4, 130.8), turned to 180 degrees
- moved SV14 157.5 mm to (56.0, 87.0), turned to 270 degrees
- moved C9 150.2 mm to (85.6, 126.2), turned to 0 degrees
- moved R28 146.2 mm to (27.7, 127.9), flipped to the top, turned to 90 degrees
- moved C10 140.9 mm to (85.6, 143.1), flipped to the bottom
- moved C5 140.6 mm to (85.6, 138.9), flipped to the bottom
- moved R29 137.5 mm to (34.8, 126.3), flipped to the top
- moved R15 137.5 mm to (143.0, 122.9), turned to 270 degrees
- moved SV10 129.3 mm to (104.7, 129.6), turned to 315 degrees
- moved PB1'1 127.1 mm to (110.4, 109.7), turned to 90 degrees
- moved R24 126.4 mm to (43.8, 123.2), flipped to the top, turned to 180 degrees
- moved T1 124.8 mm to (113.3, 94.7), turned to 90 degrees
- moved U3 124.1 mm to (61.7, 73.8), flipped to the bottom, turned to 270 degrees
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Connections:
- removed net CE_SPI2: TP21.TP, U$1.58
- removed net CSN_SPI2: TP22.TP, U$1.57
- removed net IRQ_SPI2: U$1.8
- removed net IR_SENSOR_ADC: SV14.2, U$1.24
- removed net KICKER_GPIO1: T6.1, U$1.15
- removed net KICKER_GPIO2: T7.1, U$1.16
- removed net KICKER_GPIO3: T8.1, U$1.17
- removed net KICKER_GPIO4: T9.1, U$1.18
- removed net KICKER_USART1_RX: JP13.P$1, U$1.93
- removed net KICKER_USART1_TX: JP13.P$3, U$1.92
- removed net MISO_SPI2: TP25.TP, U$1.53
- removed net MOSI_SPI2: TP24.TP, U$1.54
- removed net N$35: R5.2, T8.2
- removed net N$37: R3.2, T6.2
- removed net N$38: R4.2, T7.2
- removed net N$39: R24.2, T9.2
- removed net N$40: JP13.P$2, R26.1, T6.3
- removed net N$41: JP13.P$4, R27.1, T7.3
- removed net N$42: JP13.P$6, R28.1, T8.3
- removed net N$43: JP13.P$8, R29.2, T9.3
- removed net PH0: C14.2, Q1.1, U$1.12
- removed net PH1: R2.2, U$1.13
- removed net SCK_SPI2: TP23.TP, U$1.52
- removed net SD_CARD_CMD: SV13.4, U$1.83
- removed net SD_CARD_DAT0: SV13.3, U$1.65
- removed net SD_CARD_SCK: SV13.5, U$1.80
- removed net V_CIRCUIT: S2.3, S2.6, U$3.VIN
- new net ADC: JP11.2, U$1.24
- new net ADD: SV2.7
- new net BATTERY: J1.BATT, U$3.P$2
- new net BAT_ADC: R26.1, R27.2, U$1.25
- new net INT: SV2.8, U$1.33
- new net KICKER_1: T1.1, U$1.81
- new net KICKER_2: T2.1, U$1.82
- new net KICKER_3: T3.1, U$1.83
- new net KICKER_4: T4.1, U$1.84
- new net N$1: R5.2, U$4.D+
- new net N$11: LED1.C, Q1.3
- new net N$16: U$1.17
- new net N$17: U$1.18
- new net N$23: R16.2, T1.2
- new net N$26: R19.2, T4.2
- new net N$31: R20.1, SV1.1, T1.3
- new net N$32: R21.1, SV1.2, T2.3
- new net N$33: R22.1, SV1.3, T3.3
- new net N$34: R23.2, SV1.4, T4.3
- new net N$5: R4.2, U$4.D-
- new net PA10: U$1.69, U$4.ID
- new net PA9: R8.1, U$1.68, U$4.VCC
- new net SCL: SV2.3, U$1.92
- new net SDA: SV2.4, U$1.93
- new net TRACESWO: SV6.3, U$1.89
- new net USB_DM: R4.1, U$1.70
- new net USB_DP: R5.1, U$1.71
- new net V_BAT: R27.1, R29.2, U2.2, V_BAT.P$1, V_BAT_12V.P$1
- new net XCL: SV2.6
- new net XDA: SV2.5
- net 12V: now also 12V.P$1, R24.1, SV14.4; no longer C18.+, R7.1, SV10.7, SV10.8, U$4.VOUT
- net 3.3V: now also M1.2, Q1.1, R1.1, R12.2, R16.1, R17.1, R18.1, R19.1, SV2.1, SV6.6, U$2.1; no longer JP12.P$7, JP12.P$8, R24.1, R3.1, R4.1, R5.1, R6.1, S10.3, S10.6, S7.3, S7.6, S8.3, S8.6, S9.3, S9.6, SV13.2, TP20.TP, TP4.TP
- net 5V: now also 5V.P$1, JP11.1, R11.1, R20.2, R21.2, R22.2, R23.1; no longer R12.2, R26.2, R27.2, R29.1, SV14.3, T1.3, U$3.VOUT
- net 5VM: now also JP1.P$4, SV9.6; no longer SV1.5, SV16.11, SV16.12
- net 5VM2: now also JP5.P$4, SV11.6; no longer SV2.5, SV6.11, SV6.12
- net 5VM3: now also JP2.P$4, SV3.6; no longer SV18.11, SV18.12, SV8.5
- net 5VM4: now also JP7.P$4, SV7.6; no longer SV17.11, SV17.12, SV5.5
- net 5VM5: now also JP9.P$4, SV14.6; no longer SV10.11, SV10.12, SV4.5
- net A_1: now also SV9.10; no longer SV16.19, SV16.20
- net A_2: now also SV11.10; no longer SV6.19, SV6.20
- net A_3: now also SV3.10; no longer SV18.19, SV18.20
- net A_4: now also SV7.10; no longer SV17.19, SV17.20
- net A_5: now also SV14.10; no longer SV10.19, SV10.20
- net BATT_LEVEL: now also U$3.P$1, U3.1, U3.3; no longer U$2.NO, U$5.P$1
- net BOT_COLOR: now also SW1.1, U$1.4; no longer S10.2, S10.5, U$1.1
- net B_1: now also SV9.12; no longer SV16.23, SV16.24
- net B_2: now also SV11.12; no longer SV6.23, SV6.24
- net B_3: now also SV3.12; no longer SV18.23, SV18.24
- net B_4: now also SV7.12; no longer SV17.23, SV17.24
- net B_5: now also SV14.12; no longer SV10.23, SV10.24
- net CE: now also M1.3; no longer TP5.TP
- net CSN: now also M1.4; no longer TP6.TP
- net DIN1_1: now also SV10.4; no longer SV9.7, SV9.8
- net DIN1_2: now also SV12.4; no longer SV3.7, SV3.8
- net DIN1_3: now also SV4.4; no longer SV11.7, SV11.8
- net DIN1_4: now also SV8.4; no longer SV12.7, SV12.8
- net DIN1_5: now also SV15.4; no longer SV7.7, SV7.8
- net DIN2_1: now also SV10.3; no longer SV9.5, SV9.6
- net DIN2_2: now also SV12.3; no longer SV3.5, SV3.6
- net DIN2_3: now also SV4.3; no longer SV11.5, SV11.6
- net DIN2_4: now also SV8.3; no longer SV12.5, SV12.6
- net DIN2_5: now also SV15.3; no longer SV7.5, SV7.6
- net DIN3_1: now also SV10.2; no longer SV9.3, SV9.4
- net DIN3_2: now also SV12.2; no longer SV3.3, SV3.4
- net DIN3_3: now also SV4.2; no longer SV11.3, SV11.4
- net DIN3_4: now also SV8.2; no longer SV12.3, SV12.4
- net DIN3_5: now also SV15.2; no longer SV7.3, SV7.4
- net DIN4_1: now also SV10.1; no longer SV9.1, SV9.2
- net DIN4_2: now also SV12.1; no longer SV3.1, SV3.2
- net DIN4_3: now also SV4.1; no longer SV11.1, SV11.2
- net DIN4_4: now also SV8.1, U$1.65; no longer SV12.1, SV12.2, U$1.69
- net DIN4_5: now also SV15.1, U$1.66; no longer SV7.1, SV7.2, U$1.70
- net GND: now also GND.P$1, GND2.P$1, GND_12V.P$1, GND_5V.P$1, JP11.3, JP6.P$2, LED8.C, LED9.C, LED_12V.C, LED_3.3V.C, LED_5V.C, LED_8V.C, M1.1, R26.2, SV1.5, SV10.5, SV11.5, SV12.5, SV14.5, SV15.5, SV2.2, SV3.5, SV4.5, SV6.5, SV7.5, SV8.5, SV9.5, SW1.5, SW1.6, SW1.7, SW1.8, U$2.10; no longer 12V.C, 3.3V.C, 5V.C, BATTERY.C, C14.1, C15.1, C16.-, C17.-, C18.-, C19.-, C20.-, D2.A, JP12.P$3, JP12.P$4, JP13.P$10, JP6.P$4, S10.1, S10.4, S7.1, S7.4, S8.1, S8.4, S9.1, S9.4, SV1.4, SV10.10, SV10.9, SV11.10, SV11.9, SV12.10, SV12.9, SV13.1, SV14.1, SV16.10, SV16.9, SV17.10, SV17.9, SV18.10, SV18.9, SV2.4, SV3.10, SV3.9, SV4.4, SV5.4, SV6.10, SV6.9, SV7.10, SV7.9, SV8.4, SV9.10, SV9.9, TESTLED1.C, TESTLED2.C, TP19.TP, TP3.TP, U$2.2, U$3.GND, U$3.GNDO, U$4.GNDO
- net H1_1: now also JP1.P$6, SV9.7; no longer SV1.3, SV16.13, SV16.14
- net H1_2: now also JP5.P$6, SV11.7; no longer SV2.3, SV6.13, SV6.14
- net H1_3: now also JP2.P$6, SV3.7; no longer SV18.13, SV18.14, SV8.3
- net H1_4: now also JP7.P$6, SV7.7; no longer SV17.13, SV17.14, SV5.3
- net H1_5: now also JP9.P$6, SV14.7; no longer SV10.13, SV10.14, SV4.3
- net H2_1: now also JP1.P$7, SV9.8; no longer SV1.2, SV16.15, SV16.16
- net H2_2: now also JP5.P$7, SV11.8; no longer SV2.2, SV6.15, SV6.16
- net H2_3: now also JP2.P$7, SV3.8; no longer SV18.15, SV18.16, SV8.2
- net H2_4: now also JP7.P$7, SV7.8; no longer SV17.15, SV17.16, SV5.2
- net H2_5: now also JP9.P$7, SV14.8; no longer SV10.15, SV10.16, SV4.2
- net H3_1: now also JP1.P$8, SV9.9; no longer SV1.1, SV16.17, SV16.18
- net H3_2: now also JP5.P$8, SV11.9; no longer SV2.1, SV6.17, SV6.18
- net H3_3: now also JP2.P$8, SV3.9; no longer SV18.17, SV18.18, SV8.1
- net H3_4: now also JP7.P$8, SV7.9; no longer SV17.17, SV17.18, SV5.1
- net H3_5: now also JP9.P$8, SV14.9; no longer SV10.17, SV10.18, SV4.1
- net ID_0: now also SW1.2, U$1.3; no longer S9.2, S9.5, U$1.2
- net ID_1: now also SW1.3, U$1.2; no longer S8.2, S8.5, U$1.3
- net ID_2: now also SW1.4, U$1.1; no longer S7.2, S7.5, U$1.4
- net IRQ: now also M1.8, U$1.7; no longer TP10.TP
- net M1_1: now also JP1.P$1, SV9.1; no longer SV1.8, SV16.1, SV16.2
- net M1_2: now also JP5.P$1, SV11.1; no longer SV2.8, SV6.1, SV6.2
- net M1_3: now also JP2.P$1, SV3.1; no longer SV18.1, SV18.2, SV8.8
- net M1_4: now also JP7.P$1, SV7.1; no longer SV17.1, SV17.2, SV5.8
- net M1_5: now also JP9.P$1, SV14.1; no longer SV10.1, SV10.2, SV4.8
- net M2_1: now also JP1.P$2, SV9.2; no longer SV1.7, SV16.3, SV16.4
- net M2_2: now also JP5.P$2, SV11.2; no longer SV2.7, SV6.3, SV6.4
- net M2_3: now also JP2.P$2, SV3.2; no longer SV18.3, SV18.4, SV8.7
- net M2_4: now also JP7.P$2, SV7.2; no longer SV17.3, SV17.4, SV5.7
- net M2_5: now also JP9.P$2, SV14.2; no longer SV10.3, SV10.4, SV4.7
- net M3_1: now also JP1.P$3, SV9.3; no longer SV1.6, SV16.5, SV16.6
- net M3_2: now also JP5.P$3, SV11.3; no longer SV2.6, SV6.5, SV6.6
- net M3_3: now also JP2.P$3, SV3.3; no longer SV18.5, SV18.6, SV8.6
- net M3_4: now also JP7.P$3, SV7.3; no longer SV17.5, SV17.6, SV5.6
- net M3_5: now also JP9.P$3, SV14.3; no longer SV10.5, SV10.6, SV4.6
- net MISO: now also M1.7, U$1.79, U$2.2; no longer TP9.TP, U$1.90
- net MOSI: now also M1.6, U$1.80; no longer TP8.TP, U$1.91
- net N$10: now also R12.1, R8.2; no longer C15.2, R2.1
- net N$12: now also D3.A, U$2.3; no longer 5V.A, R12.1
- net N$13: now also LED1.A, R11.2; no longer J1.BATT, U$2.C, U$5.P$2, U3.1, U3.3
- net N$14: now also LED_12V.A, R24.2; no longer 12V.A, R7.2
- net N$15: now also LED_8V.A, R29.1; no longer SV13.6
- net N$18: now also LED_5V.A, R28.1; no longer BATTERY.A, R14.2
- net N$19: now also LED_3.3V.A; no longer 3.3V.A
- net N$2: now also LED9.A; no longer TESTLED2.A
- net N$21: now also R18.2, T3.2; no longer R1.2, T1.2
- net N$22: now also U$1.91; no longer D2.C, T1.1, U$2.1
- net N$24: now also U$1.67; no longer TP26.TP
- net N$25: now also R17.2, T2.2; no longer S2.2, S2.5, U3.2
- net N$9: now also LED8.A; no longer TESTLED1.A
- net NRST: now also R1.2, SV6.4; no longer JP12.P$2, R6.2
- net SCK: now also D3.C, M1.5, U$1.78; no longer TP7.TP, U$1.89
- net SWCLK: now also SV6.2; no longer JP12.P$5
- net SWDIO: now also SV6.1; no longer JP12.P$1
- net VDC_1: now also SV7.4, SV9.4; no longer C16.+, C17.+, R14.1, SV16.7, SV16.8, SV6.7, SV6.8, U$4.VIN
- net VDC_2: now also SV11.4, SV3.4, U3.2; no longer C19.+, C20.+, SV17.7, SV17.8, SV18.7, SV18.8, U2.2
- net ~A_1: now also SV9.11; no longer SV16.21, SV16.22
- net ~A_2: now also SV11.11; no longer SV6.21, SV6.22
- net ~A_3: now also SV3.11; no longer SV18.21, SV18.22
- net ~A_4: now also SV7.11; no longer SV17.21, SV17.22
- net ~A_5: now also SV14.11; no longer SV10.21, SV10.22
- net ~B_1: now also SV9.13; no longer SV16.25, SV16.26
- net ~B_2: now also SV11.13; no longer SV6.25, SV6.26
- net ~B_3: now also SV3.13; no longer SV18.25, SV18.26
- net ~B_4: now also SV7.13; no longer SV17.25, SV17.26
- net ~B_5: now also SV14.13; no longer SV10.25, SV10.26
Routing:
- net GND: track 877.6 -> 415.3 mm, vias 4 -> 3
- net V_BAT: track 0.00 -> 421.2 mm
- net PA10: track 0.00 -> 199.2 mm
- net PA9: track 0.00 -> 198.2 mm
- net PE1: track 200.1 -> 27.8 mm, vias 2 -> 0
- net IR_SENSOR_ADC: track 170.2 -> 0.00 mm, vias 1 -> 0
- net SD_CARD_DAT0: track 154.5 -> 0.00 mm, vias 2 -> 0
- net SDA: track 0.00 -> 152.9 mm
- net SCL: track 0.00 -> 152.3 mm
- net 3.3V: track 656.4 -> 513.2 mm, vias 9 -> 3
- net SD_CARD_CMD: track 122.4 -> 0.00 mm
- net SWDIO: track 148.0 -> 28.1 mm
- net BATTERY: track 0.00 -> 119.8 mm
- net SD_CARD_SCK: track 117.0 -> 0.00 mm
- net USB_DM: track 0.00 -> 114.1 mm, vias 0 -> 2
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- added copper zone on layer 15, net BATT_LEVEL
- removed copper zone on layer 15, net GND
Other:
- board size 163.3 x 159.3 mm -> 163.3 x 159 mm
