File: main_board/main_board-v1/main_board-v1.sch (EAGLE design)
At the start: 108 parts, among them J1 XT-60BATT_LABEL, T1 2N706, T6 BC547, T7 BC547, T8 BC547, T9 BC547

Commit message: main board
Parts:
- removed 3.3V, BATTERY, TESTLED1, TESTLED2: (no value), led:LEDCHIPLED_1206
- removed C14, C15: 20pF, rcl:C-EUC1206
- removed C16, C17, C18, C19, C20: 50uF, adafruit:CPOL-USE3.5-8
- removed D2: 1N5817-B, diode:1N5817-B
- removed JP12, JP13: FRC_25, mohit:FRC_25
- removed R14: 4.7k, resistor:R-EU_R1206
- removed R2: 220, resistor:R-EU_R1206
- removed R3: 10k, resistor:R-EU_R1206
- removed R6, R7: 1k, resistor:R-EU_R1206
- removed S10, S2, S7, S8, S9: (no value), switch:A68-A31
- removed SV13: (no value), con-lsta:FE06-1
- removed SV16, SV17, SV18: (no value), con-lsta:FE13-2
- removed SV5: (no value), con-lstb:MA08-1
- removed T6, T7, T8, T9: BC547, transistor:BC547
- removed TP10, TP19, TP20, TP21, TP22, TP23, TP24, TP25, TP26, TP3, TP4, TP5, TP6, TP7, TP8, TP9: PTR1PAD1-13, testpad:PTR1PAD1-13
- removed U$5: (no value), switch_DA10:SWITCH_DA10
- added D3: BYD13, diode:BYD13
- added GND, GND2, GND_12V, GND_5V, V_BAT, V_BAT_12V: PINHEAD_1, pinhead_1:PINHEAD_1
- added JP1, JP2, JP5, JP7, JP9: FRC_SSL, frc:FRC_SSL
- added JP11: (no value), adafruit:PINHD-1X3
- added LED1, LED8, LED9, LED_12V, LED_3.3V, LED_5V, LED_8V: (no value), led:LEDCHIPLED_1206
- added M1: WIRELESS-NRF24L01, diy-modules:WIRELESS-NRF24L01
- added R11: 1k, resistor:R-EU_R1206
- added R16, R17, R18, R19, R20, R21, R22, R23: 10k, resistor:R-EU_R1206
- added R8: 47k, resistor:R-EU_R1206
- added SV15: (no value), con-lsta:FE05-1
- added SW1: (no value), special:SW_DIP-4
- added T2, T3, T4: BC547, transistor:BC547
- 12V, 5V: value (none) -> PINHEAD_1; device led:LEDCHIPLED_1206 -> pinhead_1:PINHEAD_1
- Q1: device crystal:CRYSTALHC49U-V -> TRANSISTOR-NPN:TRANSISTOR-NPN-TO-92-EBC
- R1: value 1k -> (none); device resistor:R-EU_R1206 -> resistor:R-EU_M0805
- R12: value 1k -> (none)
- R24, R28: value 10k -> 1k
- R26: value 10k -> 27k
- R27: value 10k -> 140k
- R29: value 10k -> 4.7k
- R4, R5: value 10k -> 22
- SV1: device con-lstb:MA08-1 -> con-lstb:MA05-1
- SV10: device con-lsta:FE13-2 -> con-lsta:FE05-1
- SV11, SV3, SV7, SV9: device con-lsta:FE05-2 -> con-lsta:FE13-1
- SV12: device con-lsta:FE05-2 -> con-lsta:FE05-1
- SV14: device con-lstb:MA03-1 -> con-lsta:FE13-1
- SV2: device con-lstb:MA08-1 -> con-lsta:FE08-1
- SV4, SV8: device con-lstb:MA08-1 -> con-lsta:FE05-1
- SV6: device con-lsta:FE13-2 -> con-lstb:MA06-1
- T1: value 2N706 -> BC547; device transistor:2N706 -> transistor:BC547
- U$2: value REL -> XBEE-1B2; device rel:REL -> SparkFun:XBEE-1B2
- U$3: value BUCK -> (none); device BUCK:BUCK -> switch_DA10:SWITCH_DA10
- U$4: value BUCK -> USB-MICRO-B-FEMALE; device BUCK:BUCK -> USB-MICRO-B-FEMALE:USB-MICRO-B-FEMALE
Connections:
- removed net CE_SPI2: TP21.TP, U$1G$3.PD11/USART3_CTS
- removed net CSN_SPI2: TP22.TP, U$1G$3.PD10/USART3_CK
- removed net IRQ_SPI2: U$1G$1.PC14/OSC32_IN
- removed net IR_SENSOR_ADC: SV14.2, U$1G$1.PA1/USART2_RTS/USART4_RX
- removed net KICKER_GPIO1: T6.E, U$1G$1.PC0
- removed net KICKER_GPIO2: T7.E, U$1G$1.PC1
- removed net KICKER_GPIO3: T8.E, U$1G$1.PC2/SPI2_MISO
- removed net KICKER_GPIO4: T9.E, U$1G$1.PC3/SPI2_MOSI
- removed net KICKER_USART1_RX: JP13.1, U$1G$4.PB7/I2C1_SDA/USART1_RX
- removed net KICKER_USART1_TX: JP13.3, U$1G$4.PB6/I2C1_SCL/CAN2_TX/USART1_TX
- removed net MISO_SPI2: TP25.TP, U$1G$3.PB14/SPI2_MISO/USART3_RTS
- removed net MOSI_SPI2: TP24.TP, U$1G$3.PB15/SPI2_MOSI
- removed net N$35: R5.2, T8.B
- removed net N$37: R3.2, T6.B
- removed net N$38: R4.2, T7.B
- removed net N$39: R24.2, T9.B
- removed net N$40: JP13.2, R26.1, T6.C
- removed net N$41: JP13.4, R27.1, T7.C
- removed net N$42: JP13.6, R28.1, T8.C
- removed net N$43: JP13.8, R29.2, T9.C
- removed net PH0: C14.2, Q1.1, U$1G$1.PH0/OSC_IN
- removed net PH1: R2.2, U$1G$1.PH1/OSC_OUT
- removed net SCK_SPI2: TP23.TP, U$1G$3.PB13/SPI2_SCK_USART3_CTS_CAN2_TX
- removed net SD_CARD_CMD: SV13.4, U$1G$4.PD2/UART5_RX
- removed net SD_CARD_DAT0: SV13.3, U$1G$3.PC8/USART6_CK
- removed net SD_CARD_SCK: SV13.5, U$1G$4.PC12/UART5_TX/SPI3_MOSI/USART3_CK
- removed net V_CIRCUIT: S2A.S, S2B.S, U$3.VIN
- new net ADC: JP11.2, U$1G$1.PA1/USART2_RTS/USART4_RX
- new net ADD: SV2.7
- new net BATTERY: J1.+, U$3.P
- new net BAT_ADC: R26.1, R27.2, U$1G$1.PA2/USART2_TX
- new net INT: SV2.8, U$1G$2.PC4
- new net KICKER_1: T1.E, U$1G$4.PD0/CAN1_RX
- new net KICKER_2: T2.E, U$1G$4.PD1/CAN1_TX
- new net KICKER_3: T3.E, U$1G$4.PD2/UART5_RX
- new net KICKER_4: T4.E, U$1G$4.PD3/USART2_CTS
- new net N$1: R5.2, U$4.3
- new net N$11: LED1.C, Q1.C
- new net N$16: U$1G$1.PC2/SPI2_MISO
- new net N$17: U$1G$1.PC3/SPI2_MOSI
- new net N$23: R16.2, T1.B
- new net N$26: R19.2, T4.B
- new net N$31: R20.1, SV1.1, T1.C
- new net N$32: R21.1, SV1.2, T2.C
- new net N$33: R22.1, SV1.3, T3.C
- new net N$34: R23.2, SV1.4, T4.C
- new net N$5: R4.2, U$4.2
- new net PA10: U$1G$3.PA10/USART1_RX, U$4.4
- new net PA9: R8.1, U$1G$3.PA9/USART1_TX/I2C3_SMBA, U$4.1
- new net SCL: SV2.3, U$1G$4.PB6/I2C1_SCL/CAN2_TX/USART1_TX
- new net SDA: SV2.4, U$1G$4.PB7/I2C1_SDA/USART1_RX
- new net TRACESWO: SV6.3, U$1G$4.PB3/JTDO/TRACESWO/SPI3_SCK/SPI1_SCK
- new net USB_DM: R4.1, U$1G$3.PA11/USART1_CTS/CAN1_RX/OTG_FS_D-
- new net USB_DP: R5.1, U$1G$3.PA12/USART1_RTS/CAN1_TX/OTG_FS_DP+
- new net V_BAT: R27.1, R29.2, U2.K, V_BAT.P$1, V_BAT_12V.P$1
- new net XCL: SV2.6
- new net XDA: SV2.5
- net 12V: now also 12V.P$1, R24.1, SV14.4; no longer C18.+, R7.1, SV10.7, SV10.8, U$4.VOUT
- net 3.3V: now also M1.VCC, Q1.E, R1.1, R12.2, R16.1, R17.1, R18.1, R19.1, SV2.1, SV6.6, U$2.VDD; no longer JP12.7, JP12.8, R24.1, R3.1, R4.1, R5.1, R6.1, S10A.S, S10B.S, S7A.S, S7B.S, S8A.S, S8B.S, S9A.S, S9B.S, SV13.2, TP20.TP, TP4.TP
- net 5V: now also 5V.P$1, JP11.1, R11.1, R20.2, R21.2, R22.2, R23.1; no longer R12.2, R26.2, R27.2, R29.1, SV14.3, T1.C, U$3.VOUT
- net 5VM: now also JP1.4, SV9.6; no longer SV1.5, SV16.11, SV16.12
- net 5VM2: now also JP5.4, SV11.6; no longer SV2.5, SV6.11, SV6.12
- net 5VM3: now also JP2.4, SV3.6; no longer SV18.11, SV18.12, SV8.5
- net 5VM4: now also JP7.4, SV7.6; no longer SV17.11, SV17.12, SV5.5
- net 5VM5: now also JP9.4, SV14.6; no longer SV10.11, SV10.12, SV4.5
- net A_1: now also SV9.10; no longer SV16.19, SV16.20
- net A_2: now also SV11.10; no longer SV6.19, SV6.20
- net A_3: now also SV3.10; no longer SV18.19, SV18.20
- net A_4: now also SV7.10; no longer SV17.19, SV17.20
- net A_5: now also SV14.10; no longer SV10.19, SV10.20
- net BATT_LEVEL: now also U$3.S, U3.A, U3.~A; no longer U$2.NO, U$5.S
- net BOT_COLOR: now also SW1.1, U$1G$1.PE5; no longer S10A.P, S10B.P, U$1G$1.PE2
- net B_1: now also SV9.12; no longer SV16.23, SV16.24
- net B_2: now also SV11.12; no longer SV6.23, SV6.24
- net B_3: now also SV3.12; no longer SV18.23, SV18.24
- net B_4: now also SV7.12; no longer SV17.23, SV17.24
- net B_5: now also SV14.12; no longer SV10.23, SV10.24
- net CE: now also M1.CE; no longer TP5.TP
- net CSN: now also M1.CSN; no longer TP6.TP
- net DIN1_1: now also SV10.4; no longer SV9.7, SV9.8
- net DIN1_2: now also SV12.4; no longer SV3.7, SV3.8
- net DIN1_3: now also SV4.4; no longer SV11.7, SV11.8
- net DIN1_4: now also SV8.4; no longer SV12.7, SV12.8
- net DIN1_5: now also SV15.4; no longer SV7.7, SV7.8
- net DIN2_1: now also SV10.3; no longer SV9.5, SV9.6
- net DIN2_2: now also SV12.3; no longer SV3.5, SV3.6
- net DIN2_3: now also SV4.3; no longer SV11.5, SV11.6
- net DIN2_4: now also SV8.3; no longer SV12.5, SV12.6
- net DIN2_5: now also SV15.3; no longer SV7.5, SV7.6
- net DIN3_1: now also SV10.2; no longer SV9.3, SV9.4
- net DIN3_2: now also SV12.2; no longer SV3.3, SV3.4
- net DIN3_3: now also SV4.2; no longer SV11.3, SV11.4
- net DIN3_4: now also SV8.2; no longer SV12.3, SV12.4
- net DIN3_5: now also SV15.2; no longer SV7.3, SV7.4
- net DIN4_1: now also SV10.1; no longer SV9.1, SV9.2
- net DIN4_2: now also SV12.1; no longer SV3.1, SV3.2
- net DIN4_3: now also SV4.1; no longer SV11.1, SV11.2
- net DIN4_4: now also SV8.1, U$1G$3.PC8/USART6_CK; no longer SV12.1, SV12.2, U$1G$3.PA10/USART1_RX
- net DIN4_5: now also SV15.1, U$1G$3.PC9/I2C3_SDA; no longer SV7.1, SV7.2, U$1G$3.PA11/USART1_CTS/CAN1_RX/OTG_FS_D-
- net GND: now also GND.P$1, GND2.P$1, GND_12V.P$1, GND_5V.P$1, JP11.3, JP6.2, LED8.C, LED9.C, LED_12V.C, LED_3.3V.C, LED_5V.C, LED_8V.C, M1.GND, R26.2, SV1.5, SV10.5, SV11.5, SV12.5, SV14.5, SV15.5, SV2.2, SV3.5, SV4.5, SV6.5, SV7.5, SV8.5, SV9.5, SW1.5, SW1.6, SW1.7, SW1.8, U$2.GND, U$4.5; no longer 12V.C, 3.3V.C, 5V.C, BATTERY.C, C14.1, C15.1, C16.-, C17.-, C18.-, C19.-, C20.-, D2.A, JP12.3, JP12.4, JP13.10, JP6.4, S10A.O, S10B.O, S7A.O, S7B.O, S8A.O, S8B.O, S9A.O, S9B.O, SV1.4, SV10.10, SV10.9, SV11.10, SV11.9, SV12.10, SV12.9, SV13.1, SV14.1, SV16.10, SV16.9, SV17.10, SV17.9, SV18.10, SV18.9, SV2.4, SV3.10, SV3.9, SV4.4, SV5.4, SV6.10, SV6.9, SV7.10, SV7.9, SV8.4, SV9.10, SV9.9, TESTLED1.C, TESTLED2.C, TP19.TP, TP3.TP, U$2.2, U$3.GND, U$3.GNDO, U$4.GND, U$4.GNDO
- net H1_1: now also JP1.6, SV9.7; no longer SV1.3, SV16.13, SV16.14
- net H1_2: now also JP5.6, SV11.7; no longer SV2.3, SV6.13, SV6.14
- net H1_3: now also JP2.6, SV3.7; no longer SV18.13, SV18.14, SV8.3
- net H1_4: now also JP7.6, SV7.7; no longer SV17.13, SV17.14, SV5.3
- net H1_5: now also JP9.6, SV14.7; no longer SV10.13, SV10.14, SV4.3
- net H2_1: now also JP1.7, SV9.8; no longer SV1.2, SV16.15, SV16.16
- net H2_2: now also JP5.7, SV11.8; no longer SV2.2, SV6.15, SV6.16
- net H2_3: now also JP2.7, SV3.8; no longer SV18.15, SV18.16, SV8.2
- net H2_4: now also JP7.7, SV7.8; no longer SV17.15, SV17.16, SV5.2
- net H2_5: now also JP9.7, SV14.8; no longer SV10.15, SV10.16, SV4.2
- net H3_1: now also JP1.8, SV9.9; no longer SV1.1, SV16.17, SV16.18
- net H3_2: now also JP5.8, SV11.9; no longer SV2.1, SV6.17, SV6.18
- net H3_3: now also JP2.8, SV3.9; no longer SV18.17, SV18.18, SV8.1
- net H3_4: now also JP7.8, SV7.9; no longer SV17.17, SV17.18, SV5.1
- net H3_5: now also JP9.8, SV14.9; no longer SV10.17, SV10.18, SV4.1
- net ID_0: now also SW1.2, U$1G$1.PE4; no longer S9A.P, S9B.P, U$1G$1.PE3
- net ID_1: now also SW1.3, U$1G$1.PE3; no longer S8A.P, S8B.P, U$1G$1.PE4
- net ID_2: now also SW1.4, U$1G$1.PE2; no longer S7A.P, S7B.P, U$1G$1.PE5
- net IRQ: now also M1.IRQ, U$1G$1.PC13/RTC_AF1; no longer TP10.TP
- net M1_1: now also JP1.1, SV9.1; no longer SV1.8, SV16.1, SV16.2
- net M1_2: now also JP5.1, SV11.1; no longer SV2.8, SV6.1, SV6.2
- net M1_3: now also JP2.1, SV3.1; no longer SV18.1, SV18.2, SV8.8
- net M1_4: now also JP7.1, SV7.1; no longer SV17.1, SV17.2, SV5.8
- net M1_5: now also JP9.1, SV14.1; no longer SV10.1, SV10.2, SV4.8
- net M2_1: now also JP1.2, SV9.2; no longer SV1.7, SV16.3, SV16.4
- net M2_2: now also JP5.2, SV11.2; no longer SV2.7, SV6.3, SV6.4
- net M2_3: now also JP2.2, SV3.2; no longer SV18.3, SV18.4, SV8.7
- net M2_4: now also JP7.2, SV7.2; no longer SV17.3, SV17.4, SV5.7
- net M2_5: now also JP9.2, SV14.2; no longer SV10.3, SV10.4, SV4.7
- net M3_1: now also JP1.3, SV9.3; no longer SV1.6, SV16.5, SV16.6
- net M3_2: now also JP5.3, SV11.3; no longer SV2.6, SV6.5, SV6.6
- net M3_3: now also JP2.3, SV3.3; no longer SV18.5, SV18.6, SV8.6
- net M3_4: now also JP7.3, SV7.3; no longer SV17.5, SV17.6, SV5.6
- net M3_5: now also JP9.3, SV14.3; no longer SV10.5, SV10.6, SV4.6
- net MISO: now also M1.MISO, U$1G$4.PC11/UART4_RX/SPI3_MISO/USART3_RX, U$2.DOUT; no longer TP9.TP, U$1G$4.PB4/NJTRST/SPI3_MISO/SPI1_MISO
- net MOSI: now also M1.MOSI, U$1G$4.PC12/UART5_TX/SPI3_MOSI/USART3_CK; no longer TP8.TP, U$1G$4.PB5/I2C1_SMBA/CAN2_RX/SPI1_MOSI/SPI3_MOSI
- net N$10: now also Q1.B, R12.1, R8.2; no longer C15.2, Q1.2, R2.1
- net N$12: now also D3.A, U$2.DIN; no longer 5V.A, R12.1
- net N$13: now also LED1.A, R11.2; no longer J1.+, U$2.C, U$5.P, U3.A, U3.~A
- net N$14: now also LED_12V.A, R24.2; no longer 12V.A, R7.2
- net N$15: now also LED_8V.A, R29.1; no longer SV13.6
- net N$18: now also LED_5V.A, R28.1; no longer BATTERY.A, R14.2
- net N$19: now also LED_3.3V.A; no longer 3.3V.A
- net N$2: now also LED9.A; no longer TESTLED2.A
- net N$21: now also R18.2, T3.B; no longer R1.2, T1.B
- net N$22: now also U$1G$4.PB5/I2C1_SMBA/CAN2_RX/SPI1_MOSI/SPI3_MOSI; no longer D2.C, T1.E, U$2.1
- net N$24: now also U$1G$3.PA8/USART1_CK/I2C3_SCL; no longer TP26.TP
- net N$25: now also R17.2, T2.B; no longer S2A.P, S2B.P, U3.K
- net N$9: now also LED8.A; no longer TESTLED1.A
- net NRST: now also R1.2, SV6.4; no longer JP12.2, R6.2
- net SCK: now also D3.C, M1.SCK, U$1G$4.PC10/SPI3_SCK/UART4_TX/USART3_CK; no longer TP7.TP, U$1G$4.PB3/JTDO/TRACESWO/SPI3_SCK/SPI1_SCK
- net SWCLK: now also SV6.2; no longer JP12.5
- net SWDIO: now also SV6.1; no longer JP12.1
- net VDC_1: now also SV7.4, SV9.4; no longer C16.+, C17.+, R14.1, SV16.7, SV16.8, SV6.7, SV6.8, U$4.VIN
- net VDC_2: now also SV11.4, SV3.4, U3.K; no longer C19.+, C20.+, SV17.7, SV17.8, SV18.7, SV18.8, U2.K
- net ~A_1: now also SV9.11; no longer SV16.21, SV16.22
- net ~A_2: now also SV11.11; no longer SV6.21, SV6.22
- net ~A_3: now also SV3.11; no longer SV18.21, SV18.22
- net ~A_4: now also SV7.11; no longer SV17.21, SV17.22
- net ~A_5: now also SV14.11; no longer SV10.21, SV10.22
- net ~B_1: now also SV9.13; no longer SV16.25, SV16.26
- net ~B_2: now also SV11.13; no longer SV6.25, SV6.26
- net ~B_3: now also SV3.13; no longer SV18.25, SV18.26
- net ~B_4: now also SV7.13; no longer SV17.25, SV17.26
- net ~B_5: now also SV14.13; no longer SV10.25, SV10.26
Other:
- note added: "IMU MPU6050"
- note added: "NRF24L01+"
- note added: "POWER SUPPLY 5v"
- note added: "Proximity"
- note added: "USB MICRO"
- note added: "X-Bee"
- note removed: "CRYSTAL"
- note removed: "IR SENSOR"
- note removed: "NRF24L01+ receiver"
- note removed: "NRF24L01+ transmitter"
- note removed: "POWER SUPPLY"
- note removed: "Power Supply 5V"
- note removed: "SD CARD MODULE"
- moved on the sheet: C1, C10, C11, C12, C13, C2, C3, C4, C5, C6, C69, C7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
