File: main_board/main_board-v2.1/main_board-v2.1.brd (EAGLE design)
At the start: 163.3 x 159 mm, 94 parts, among them J1 XT-60BATT_LABEL, M1 WIRELESS-NRF24L01, T1 BC547, T2 BC547, T3 BC547, T4 BC547

Commit message: main board
Parts:
- removed D3: BYD13, diode:SOD81
- removed GND, GND2, GND_12V, GND_5V, V_BAT, V_BAT_12V: PINHEAD_1, pinhead_1:PINHEAD_1
- removed JP1, JP2, JP5, JP7, JP9: FRC_SSL, frc:FRC
- removed JP11: (no value), adafruit:1X03
- removed LED1, LED8, LED9, LED_12V, LED_3.3V, LED_5V, LED_8V: (no value), led:CHIPLED_1206
- removed M1: WIRELESS-NRF24L01, diy-modules:WIRELESS-NRF24L01
- removed R11: 1k, resistor:R1206
- removed R16, R17, R18, R19, R20, R21, R22, R23: 10k, resistor:R1206
- removed R8: 47k, resistor:R1206
- removed SV15: (no value), con-lsta:FE05-1
- removed SW1: (no value), special:EDG-04
- removed T2, T3, T4: BC547, transistor:TO92
- added 3.3V, BATTERY, TESTLED1, TESTLED2: (no value), led:CHIPLED_1206
- added C14, C15: 20pF, rcl:C1206
- added C16, C17, C18, C19, C20: 50uF, adafruit:E3,5-8
- added D2: 1N5817-B, diode:DO41-7.6
- added JP12, JP13: FRC_25, mohit:FRC2*5
- added R14: 4.7k, resistor:R1206
- added R2: 220, resistor:R1206
- added R3: 10k, resistor:R1206
- added R6, R7: 1k, resistor:R1206
- added S10, S2, S7, S8, S9: (no value), switch:A68-A31
- added SV13: (no value), con-lsta:FE06
- added SV16, SV17, SV18: (no value), con-lsta:FE13-2
- added SV5: (no value), con-lstb:MA08-1
- added T6, T7, T8, T9: BC547, transistor:TO92
- added TP10, TP19, TP20, TP21, TP22, TP23, TP24, TP25, TP26, TP3, TP4, TP5, TP6, TP7, TP8, TP9: PTR1PAD1-13, testpad:P1-13
- added U$5: (no value), switch_DA10:DA10
- 12V, 5V: value PINHEAD_1 -> (none); device pinhead_1:PINHEAD_1 -> led:CHIPLED_1206
- Q1: device TRANSISTOR-NPN:TO-92 -> crystal:HC49U-V
- R1: value (none) -> 1k; device resistor:M0805 -> resistor:R1206
- R12: value (none) -> 1k
- R24, R28: value 1k -> 10k
- R26: value 27k -> 10k
- R27: value 140k -> 10k
- R29: value 4.7k -> 10k
- R4, R5: value 22 -> 10k
- SV1: device con-lstb:MA05-1 -> con-lstb:MA08-1
- SV10: device con-lsta:FE05-1 -> con-lsta:FE13-2
- SV11, SV3, SV7, SV9: device con-lsta:FE13 -> con-lsta:FE05-2
- SV12: device con-lsta:FE05-1 -> con-lsta:FE05-2
- SV14: device con-lsta:FE13 -> con-lstb:MA03-1
- SV2: device con-lsta:FE08 -> con-lstb:MA08-1
- SV4, SV8: device con-lsta:FE05-1 -> con-lstb:MA08-1
- SV6: device con-lstb:MA06-1 -> con-lsta:FE13-2
- T1: value BC547 -> 2N706; device transistor:TO92 -> transistor:TO18
- U$2: value XBEE-1B2 -> REL; device SparkFun:XBEE-SILK -> rel:REL
- U$3: value (none) -> BUCK; device switch_DA10:DA10 -> BUCK:BUCK
- U$4: value USB-MICRO-B-FEMALE -> BUCK; device USB-MICRO-B-FEMALE:USB-MICRO-B-FEMALE -> BUCK:BUCK
- moved SV11 176.6 mm to (92.5, -33.7), turned to 135 degrees
- moved SV12 163.4 mm to (133.2, -29.7), turned to 225 degrees
- moved R1 158.8 mm to (93.2, -26.8), turned to 0 degrees
- moved SV14 157.5 mm to (80.3, -68.7), turned to 157.1 degrees
- moved C9 150.2 mm to (93.2, -23.9), turned to 180 degrees
- moved R28 146.2 mm to (122.9, 16.9), flipped to the bottom, turned to 0 degrees
- moved C10 140.9 mm to (93.7, 2.46), flipped to the top
- moved C5 140.6 mm to (93.7, -1.43), flipped to the top
- moved R29 137.5 mm to (122.9, 20.7), flipped to the bottom
- moved R15 137.5 mm to (93.6, -5.40), turned to 0 degrees
- moved SV10 129.3 mm to (80.9, 2.54), turned to 270 degrees
- moved PB1'1 127.1 mm to (91.8, -16.1), turned to 180 degrees
- moved R24 126.4 mm to (122.9, 24.6), flipped to the bottom, turned to 0 degrees
- moved T1 124.8 mm to (98.7, -29.2), turned to 0 degrees
- moved U3 124.1 mm to (90.1, -47.0), flipped to the top, turned to 90 degrees
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Connections:
- removed net ADC: JP11.2, U$1.24
- removed net ADD: SV2.7
- removed net BATTERY: J1.BATT, U$3.P$2
- removed net BAT_ADC: R26.1, R27.2, U$1.25
- removed net INT: SV2.8, U$1.33
- removed net KICKER_1: T1.1, U$1.81
- removed net KICKER_2: T2.1, U$1.82
- removed net KICKER_3: T3.1, U$1.83
- removed net KICKER_4: T4.1, U$1.84
- removed net N$1: R5.2, U$4.D+
- removed net N$11: LED1.C, Q1.3
- removed net N$16: U$1.17
- removed net N$17: U$1.18
- removed net N$23: R16.2, T1.2
- removed net N$26: R19.2, T4.2
- removed net N$31: R20.1, SV1.1, T1.3
- removed net N$32: R21.1, SV1.2, T2.3
- removed net N$33: R22.1, SV1.3, T3.3
- removed net N$34: R23.2, SV1.4, T4.3
- removed net N$5: R4.2, U$4.D-
- removed net PA10: U$1.69, U$4.ID
- removed net PA9: R8.1, U$1.68, U$4.VCC
- removed net SCL: SV2.3, U$1.92
- removed net SDA: SV2.4, U$1.93
- removed net TRACESWO: SV6.3, U$1.89
- removed net USB_DM: R4.1, U$1.70
- removed net USB_DP: R5.1, U$1.71
- removed net V_BAT: R27.1, R29.2, U2.2, V_BAT.P$1, V_BAT_12V.P$1
- removed net XCL: SV2.6
- removed net XDA: SV2.5
- new net CE_SPI2: TP21.TP, U$1.58
- new net CSN_SPI2: TP22.TP, U$1.57
- new net IRQ_SPI2: U$1.8
- new net IR_SENSOR_ADC: SV14.2, U$1.24
- new net KICKER_GPIO1: T6.1, U$1.15
- new net KICKER_GPIO2: T7.1, U$1.16
- new net KICKER_GPIO3: T8.1, U$1.17
- new net KICKER_GPIO4: T9.1, U$1.18
- new net KICKER_USART1_RX: JP13.P$1, U$1.93
- new net KICKER_USART1_TX: JP13.P$3, U$1.92
- new net MISO_SPI2: TP25.TP, U$1.53
- new net MOSI_SPI2: TP24.TP, U$1.54
- new net N$35: R5.2, T8.2
- new net N$37: R3.2, T6.2
- new net N$38: R4.2, T7.2
- new net N$39: R24.2, T9.2
- new net N$40: JP13.P$2, R26.1, T6.3
- new net N$41: JP13.P$4, R27.1, T7.3
- new net N$42: JP13.P$6, R28.1, T8.3
- new net N$43: JP13.P$8, R29.2, T9.3
- new net PH0: C14.2, Q1.1, U$1.12
- new net PH1: R2.2, U$1.13
- new net SCK_SPI2: TP23.TP, U$1.52
- new net SD_CARD_CMD: SV13.4, U$1.83
- new net SD_CARD_DAT0: SV13.3, U$1.65
- new net SD_CARD_SCK: SV13.5, U$1.80
- new net V_CIRCUIT: S2.3, S2.6, U$3.VIN
- net 12V: now also C18.+, R7.1, SV10.7, SV10.8, U$4.VOUT; no longer 12V.P$1, R24.1, SV14.4
- net 3.3V: now also JP12.P$7, JP12.P$8, R24.1, R3.1, R4.1, R5.1, R6.1, S10.3, S10.6, S7.3, S7.6, S8.3, S8.6, S9.3, S9.6, SV13.2, TP20.TP, TP4.TP; no longer M1.2, Q1.1, R1.1, R12.2, R16.1, R17.1, R18.1, R19.1, SV2.1, SV6.6, U$2.1
- net 5V: now also R12.2, R26.2, R27.2, R29.1, SV14.3, T1.3, U$3.VOUT; no longer 5V.P$1, JP11.1, R11.1, R20.2, R21.2, R22.2, R23.1
- net 5VM: now also SV1.5, SV16.11, SV16.12; no longer JP1.P$4, SV9.6
- net 5VM2: now also SV2.5, SV6.11, SV6.12; no longer JP5.P$4, SV11.6
- net 5VM3: now also SV18.11, SV18.12, SV8.5; no longer JP2.P$4, SV3.6
- net 5VM4: now also SV17.11, SV17.12, SV5.5; no longer JP7.P$4, SV7.6
- net 5VM5: now also SV10.11, SV10.12, SV4.5; no longer JP9.P$4, SV14.6
- net A_1: now also SV16.19, SV16.20; no longer SV9.10
- net A_2: now also SV6.19, SV6.20; no longer SV11.10
- net A_3: now also SV18.19, SV18.20; no longer SV3.10
- net A_4: now also SV17.19, SV17.20; no longer SV7.10
- net A_5: now also SV10.19, SV10.20; no longer SV14.10
- net BATT_LEVEL: now also U$2.NO, U$5.P$1; no longer U$3.P$1, U3.1, U3.3
- net BOT_COLOR: now also S10.2, S10.5, U$1.1; no longer SW1.1, U$1.4
- net B_1: now also SV16.23, SV16.24; no longer SV9.12
- net B_2: now also SV6.23, SV6.24; no longer SV11.12
- net B_3: now also SV18.23, SV18.24; no longer SV3.12
- net B_4: now also SV17.23, SV17.24; no longer SV7.12
- net B_5: now also SV10.23, SV10.24; no longer SV14.12
- net CE: now also TP5.TP; no longer M1.3
- net CSN: now also TP6.TP; no longer M1.4
- net DIN1_1: now also SV9.7, SV9.8; no longer SV10.4
- net DIN1_2: now also SV3.7, SV3.8; no longer SV12.4
- net DIN1_3: now also SV11.7, SV11.8; no longer SV4.4
- net DIN1_4: now also SV12.7, SV12.8; no longer SV8.4
- net DIN1_5: now also SV7.7, SV7.8; no longer SV15.4
- net DIN2_1: now also SV9.5, SV9.6; no longer SV10.3
- net DIN2_2: now also SV3.5, SV3.6; no longer SV12.3
- net DIN2_3: now also SV11.5, SV11.6; no longer SV4.3
- net DIN2_4: now also SV12.5, SV12.6; no longer SV8.3
- net DIN2_5: now also SV7.5, SV7.6; no longer SV15.3
- net DIN3_1: now also SV9.3, SV9.4; no longer SV10.2
- net DIN3_2: now also SV3.3, SV3.4; no longer SV12.2
- net DIN3_3: now also SV11.3, SV11.4; no longer SV4.2
- net DIN3_4: now also SV12.3, SV12.4; no longer SV8.2
- net DIN3_5: now also SV7.3, SV7.4; no longer SV15.2
- net DIN4_1: now also SV9.1, SV9.2; no longer SV10.1
- net DIN4_2: now also SV3.1, SV3.2; no longer SV12.1
- net DIN4_3: now also SV11.1, SV11.2; no longer SV4.1
- net DIN4_4: now also SV12.1, SV12.2, U$1.69; no longer SV8.1, U$1.65
- net DIN4_5: now also SV7.1, SV7.2, U$1.70; no longer SV15.1, U$1.66
- net GND: now also 12V.C, 3.3V.C, 5V.C, BATTERY.C, C14.1, C15.1, C16.-, C17.-, C18.-, C19.-, C20.-, D2.A, JP12.P$3, JP12.P$4, JP13.P$10, JP6.P$4, S10.1, S10.4, S7.1, S7.4, S8.1, S8.4, S9.1, S9.4, SV1.4, SV10.10, SV10.9, SV11.10, SV11.9, SV12.10, SV12.9, SV13.1, SV14.1, SV16.10, SV16.9, SV17.10, SV17.9, SV18.10, SV18.9, SV2.4, SV3.10, SV3.9, SV4.4, SV5.4, SV6.10, SV6.9, SV7.10, SV7.9, SV8.4, SV9.10, SV9.9, TESTLED1.C, TESTLED2.C, TP19.TP, TP3.TP, U$2.2, U$3.GND, U$3.GNDO, U$4.GNDO; no longer GND.P$1, GND2.P$1, GND_12V.P$1, GND_5V.P$1, JP11.3, JP6.P$2, LED8.C, LED9.C, LED_12V.C, LED_3.3V.C, LED_5V.C, LED_8V.C, M1.1, R26.2, SV1.5, SV10.5, SV11.5, SV12.5, SV14.5, SV15.5, SV2.2, SV3.5, SV4.5, SV6.5, SV7.5, SV8.5, SV9.5, SW1.5, SW1.6, SW1.7, SW1.8, U$2.10
- net H1_1: now also SV1.3, SV16.13, SV16.14; no longer JP1.P$6, SV9.7
- net H1_2: now also SV2.3, SV6.13, SV6.14; no longer JP5.P$6, SV11.7
- net H1_3: now also SV18.13, SV18.14, SV8.3; no longer JP2.P$6, SV3.7
- net H1_4: now also SV17.13, SV17.14, SV5.3; no longer JP7.P$6, SV7.7
- net H1_5: now also SV10.13, SV10.14, SV4.3; no longer JP9.P$6, SV14.7
- net H2_1: now also SV1.2, SV16.15, SV16.16; no longer JP1.P$7, SV9.8
- net H2_2: now also SV2.2, SV6.15, SV6.16; no longer JP5.P$7, SV11.8
- net H2_3: now also SV18.15, SV18.16, SV8.2; no longer JP2.P$7, SV3.8
- net H2_4: now also SV17.15, SV17.16, SV5.2; no longer JP7.P$7, SV7.8
- net H2_5: now also SV10.15, SV10.16, SV4.2; no longer JP9.P$7, SV14.8
- net H3_1: now also SV1.1, SV16.17, SV16.18; no longer JP1.P$8, SV9.9
- net H3_2: now also SV2.1, SV6.17, SV6.18; no longer JP5.P$8, SV11.9
- net H3_3: now also SV18.17, SV18.18, SV8.1; no longer JP2.P$8, SV3.9
- net H3_4: now also SV17.17, SV17.18, SV5.1; no longer JP7.P$8, SV7.9
- net H3_5: now also SV10.17, SV10.18, SV4.1; no longer JP9.P$8, SV14.9
- net ID_0: now also S9.2, S9.5, U$1.2; no longer SW1.2, U$1.3
- net ID_1: now also S8.2, S8.5, U$1.3; no longer SW1.3, U$1.2
- net ID_2: now also S7.2, S7.5, U$1.4; no longer SW1.4, U$1.1
- net IRQ: now also TP10.TP; no longer M1.8, U$1.7
- net M1_1: now also SV1.8, SV16.1, SV16.2; no longer JP1.P$1, SV9.1
- net M1_2: now also SV2.8, SV6.1, SV6.2; no longer JP5.P$1, SV11.1
- net M1_3: now also SV18.1, SV18.2, SV8.8; no longer JP2.P$1, SV3.1
- net M1_4: now also SV17.1, SV17.2, SV5.8; no longer JP7.P$1, SV7.1
- net M1_5: now also SV10.1, SV10.2, SV4.8; no longer JP9.P$1, SV14.1
- net M2_1: now also SV1.7, SV16.3, SV16.4; no longer JP1.P$2, SV9.2
- net M2_2: now also SV2.7, SV6.3, SV6.4; no longer JP5.P$2, SV11.2
- net M2_3: now also SV18.3, SV18.4, SV8.7; no longer JP2.P$2, SV3.2
- net M2_4: now also SV17.3, SV17.4, SV5.7; no longer JP7.P$2, SV7.2
- net M2_5: now also SV10.3, SV10.4, SV4.7; no longer JP9.P$2, SV14.2
- net M3_1: now also SV1.6, SV16.5, SV16.6; no longer JP1.P$3, SV9.3
- net M3_2: now also SV2.6, SV6.5, SV6.6; no longer JP5.P$3, SV11.3
- net M3_3: now also SV18.5, SV18.6, SV8.6; no longer JP2.P$3, SV3.3
- net M3_4: now also SV17.5, SV17.6, SV5.6; no longer JP7.P$3, SV7.3
- net M3_5: now also SV10.5, SV10.6, SV4.6; no longer JP9.P$3, SV14.3
- net MISO: now also TP9.TP, U$1.90; no longer M1.7, U$1.79, U$2.2
- net MOSI: now also TP8.TP, U$1.91; no longer M1.6, U$1.80
- net N$10: now also C15.2, R2.1; no longer R12.1, R8.2
- net N$12: now also 5V.A, R12.1; no longer D3.A, U$2.3
- net N$13: now also J1.BATT, U$2.C, U$5.P$2, U3.1, U3.3; no longer LED1.A, R11.2
- net N$14: now also 12V.A, R7.2; no longer LED_12V.A, R24.2
- net N$15: now also SV13.6; no longer LED_8V.A, R29.1
- net N$18: now also BATTERY.A, R14.2; no longer LED_5V.A, R28.1
- net N$19: now also 3.3V.A; no longer LED_3.3V.A
- net N$2: now also TESTLED2.A; no longer LED9.A
- net N$21: now also R1.2, T1.2; no longer R18.2, T3.2
- net N$22: now also D2.C, T1.1, U$2.1; no longer U$1.91
- net N$24: now also TP26.TP; no longer U$1.67
- net N$25: now also S2.2, S2.5, U3.2; no longer R17.2, T2.2
- net N$9: now also TESTLED1.A; no longer LED8.A
- net NRST: now also JP12.P$2, R6.2; no longer R1.2, SV6.4
- net SCK: now also TP7.TP, U$1.89; no longer D3.C, M1.5, U$1.78
- net SWCLK: now also JP12.P$5; no longer SV6.2
- net SWDIO: now also JP12.P$1; no longer SV6.1
- net VDC_1: now also C16.+, C17.+, R14.1, SV16.7, SV16.8, SV6.7, SV6.8, U$4.VIN; no longer SV7.4, SV9.4
- net VDC_2: now also C19.+, C20.+, SV17.7, SV17.8, SV18.7, SV18.8, U2.2; no longer SV11.4, SV3.4, U3.2
- net ~A_1: now also SV16.21, SV16.22; no longer SV9.11
- net ~A_2: now also SV6.21, SV6.22; no longer SV11.11
- net ~A_3: now also SV18.21, SV18.22; no longer SV3.11
- net ~A_4: now also SV17.21, SV17.22; no longer SV7.11
- net ~A_5: now also SV10.21, SV10.22; no longer SV14.11
- net ~B_1: now also SV16.25, SV16.26; no longer SV9.13
- net ~B_2: now also SV6.25, SV6.26; no longer SV11.13
- net ~B_3: now also SV18.25, SV18.26; no longer SV3.13
- net ~B_4: now also SV17.25, SV17.26; no longer SV7.13
- net ~B_5: now also SV10.25, SV10.26; no longer SV14.13
Routing:
- net GND: track 415.3 -> 877.6 mm, vias 3 -> 4
- net V_BAT: track 421.2 -> 0.00 mm
- net PA10: track 199.2 -> 0.00 mm
- net PA9: track 198.2 -> 0.00 mm
- net PE1: track 27.8 -> 200.1 mm, vias 0 -> 2
- net IR_SENSOR_ADC: track 0.00 -> 170.2 mm, vias 0 -> 1
- net SD_CARD_DAT0: track 0.00 -> 154.5 mm, vias 0 -> 2
- net SDA: track 152.9 -> 0.00 mm
- net SCL: track 152.3 -> 0.00 mm
- net 3.3V: track 513.2 -> 656.4 mm, vias 3 -> 9
- net SD_CARD_CMD: track 0.00 -> 122.4 mm
- net SWDIO: track 28.1 -> 148.0 mm
- net BATTERY: track 119.8 -> 0.00 mm
- net SD_CARD_SCK: track 0.00 -> 117.0 mm
- net USB_DM: track 114.1 -> 0.00 mm, vias 2 -> 0
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- added copper zone on layer 15, net GND
- removed copper zone on layer 15, net BATT_LEVEL
Other:
- board size 163.3 x 159 mm -> 163.3 x 159.3 mm
