File: main_board/main_board-v2.1/main_board-v2.1.sch (EAGLE design)
At the start: 94 parts, among them J1 XT-60BATT_LABEL, M1 WIRELESS-NRF24L01, T1 BC547, T2 BC547, T3 BC547, T4 BC547

Commit message: main board
Parts:
- removed D3: BYD13, diode:BYD13
- removed GND, GND2, GND_12V, GND_5V, V_BAT, V_BAT_12V: PINHEAD_1, pinhead_1:PINHEAD_1
- removed JP1, JP2, JP5, JP7, JP9: FRC_SSL, frc:FRC_SSL
- removed JP11: (no value), adafruit:PINHD-1X3
- removed LED1, LED8, LED9, LED_12V, LED_3.3V, LED_5V, LED_8V: (no value), led:LEDCHIPLED_1206
- removed M1: WIRELESS-NRF24L01, diy-modules:WIRELESS-NRF24L01
- removed R11: 1k, resistor:R-EU_R1206
- removed R16, R17, R18, R19, R20, R21, R22, R23: 10k, resistor:R-EU_R1206
- removed R8: 47k, resistor:R-EU_R1206
- removed SV15: (no value), con-lsta:FE05-1
- removed SW1: (no value), special:SW_DIP-4
- removed T2, T3, T4: BC547, transistor:BC547
- added 3.3V, BATTERY, TESTLED1, TESTLED2: (no value), led:LEDCHIPLED_1206
- added C14, C15: 20pF, rcl:C-EUC1206
- added C16, C17, C18, C19, C20: 50uF, adafruit:CPOL-USE3.5-8
- added D2: 1N5817-B, diode:1N5817-B
- added JP12, JP13: FRC_25, mohit:FRC_25
- added R14: 4.7k, resistor:R-EU_R1206
- added R2: 220, resistor:R-EU_R1206
- added R3: 10k, resistor:R-EU_R1206
- added R6, R7: 1k, resistor:R-EU_R1206
- added S10, S2, S7, S8, S9: (no value), switch:A68-A31
- added SV13: (no value), con-lsta:FE06-1
- added SV16, SV17, SV18: (no value), con-lsta:FE13-2
- added SV5: (no value), con-lstb:MA08-1
- added T6, T7, T8, T9: BC547, transistor:BC547
- added TP10, TP19, TP20, TP21, TP22, TP23, TP24, TP25, TP26, TP3, TP4, TP5, TP6, TP7, TP8, TP9: PTR1PAD1-13, testpad:PTR1PAD1-13
- added U$5: (no value), switch_DA10:SWITCH_DA10
- 12V, 5V: value PINHEAD_1 -> (none); device pinhead_1:PINHEAD_1 -> led:LEDCHIPLED_1206
- Q1: device TRANSISTOR-NPN:TRANSISTOR-NPN-TO-92-EBC -> crystal:CRYSTALHC49U-V
- R1: value (none) -> 1k; device resistor:R-EU_M0805 -> resistor:R-EU_R1206
- R12: value (none) -> 1k
- R24, R28: value 1k -> 10k
- R26: value 27k -> 10k
- R27: value 140k -> 10k
- R29: value 4.7k -> 10k
- R4, R5: value 22 -> 10k
- SV1: device con-lstb:MA05-1 -> con-lstb:MA08-1
- SV10: device con-lsta:FE05-1 -> con-lsta:FE13-2
- SV11, SV3, SV7, SV9: device con-lsta:FE13-1 -> con-lsta:FE05-2
- SV12: device con-lsta:FE05-1 -> con-lsta:FE05-2
- SV14: device con-lsta:FE13-1 -> con-lstb:MA03-1
- SV2: device con-lsta:FE08-1 -> con-lstb:MA08-1
- SV4, SV8: device con-lsta:FE05-1 -> con-lstb:MA08-1
- SV6: device con-lstb:MA06-1 -> con-lsta:FE13-2
- T1: value BC547 -> 2N706; device transistor:BC547 -> transistor:2N706
- U$2: value XBEE-1B2 -> REL; device SparkFun:XBEE-1B2 -> rel:REL
- U$3: value (none) -> BUCK; device switch_DA10:SWITCH_DA10 -> BUCK:BUCK
- U$4: value USB-MICRO-B-FEMALE -> BUCK; device USB-MICRO-B-FEMALE:USB-MICRO-B-FEMALE -> BUCK:BUCK
Connections:
- removed net ADC: JP11.2, U$1G$1.PA1/USART2_RTS/USART4_RX
- removed net ADD: SV2.7
- removed net BATTERY: J1.+, U$3.P
- removed net BAT_ADC: R26.1, R27.2, U$1G$1.PA2/USART2_TX
- removed net INT: SV2.8, U$1G$2.PC4
- removed net KICKER_1: T1.E, U$1G$4.PD0/CAN1_RX
- removed net KICKER_2: T2.E, U$1G$4.PD1/CAN1_TX
- removed net KICKER_3: T3.E, U$1G$4.PD2/UART5_RX
- removed net KICKER_4: T4.E, U$1G$4.PD3/USART2_CTS
- removed net N$1: R5.2, U$4.3
- removed net N$11: LED1.C, Q1.C
- removed net N$16: U$1G$1.PC2/SPI2_MISO
- removed net N$17: U$1G$1.PC3/SPI2_MOSI
- removed net N$23: R16.2, T1.B
- removed net N$26: R19.2, T4.B
- removed net N$31: R20.1, SV1.1, T1.C
- removed net N$32: R21.1, SV1.2, T2.C
- removed net N$33: R22.1, SV1.3, T3.C
- removed net N$34: R23.2, SV1.4, T4.C
- removed net N$5: R4.2, U$4.2
- removed net PA10: U$1G$3.PA10/USART1_RX, U$4.4
- removed net PA9: R8.1, U$1G$3.PA9/USART1_TX/I2C3_SMBA, U$4.1
- removed net SCL: SV2.3, U$1G$4.PB6/I2C1_SCL/CAN2_TX/USART1_TX
- removed net SDA: SV2.4, U$1G$4.PB7/I2C1_SDA/USART1_RX
- removed net TRACESWO: SV6.3, U$1G$4.PB3/JTDO/TRACESWO/SPI3_SCK/SPI1_SCK
- removed net USB_DM: R4.1, U$1G$3.PA11/USART1_CTS/CAN1_RX/OTG_FS_D-
- removed net USB_DP: R5.1, U$1G$3.PA12/USART1_RTS/CAN1_TX/OTG_FS_DP+
- removed net V_BAT: R27.1, R29.2, U2.K, V_BAT.P$1, V_BAT_12V.P$1
- removed net XCL: SV2.6
- removed net XDA: SV2.5
- new net CE_SPI2: TP21.TP, U$1G$3.PD11/USART3_CTS
- new net CSN_SPI2: TP22.TP, U$1G$3.PD10/USART3_CK
- new net IRQ_SPI2: U$1G$1.PC14/OSC32_IN
- new net IR_SENSOR_ADC: SV14.2, U$1G$1.PA1/USART2_RTS/USART4_RX
- new net KICKER_GPIO1: T6.E, U$1G$1.PC0
- new net KICKER_GPIO2: T7.E, U$1G$1.PC1
- new net KICKER_GPIO3: T8.E, U$1G$1.PC2/SPI2_MISO
- new net KICKER_GPIO4: T9.E, U$1G$1.PC3/SPI2_MOSI
- new net KICKER_USART1_RX: JP13.1, U$1G$4.PB7/I2C1_SDA/USART1_RX
- new net KICKER_USART1_TX: JP13.3, U$1G$4.PB6/I2C1_SCL/CAN2_TX/USART1_TX
- new net MISO_SPI2: TP25.TP, U$1G$3.PB14/SPI2_MISO/USART3_RTS
- new net MOSI_SPI2: TP24.TP, U$1G$3.PB15/SPI2_MOSI
- new net N$35: R5.2, T8.B
- new net N$37: R3.2, T6.B
- new net N$38: R4.2, T7.B
- new net N$39: R24.2, T9.B
- new net N$40: JP13.2, R26.1, T6.C
- new net N$41: JP13.4, R27.1, T7.C
- new net N$42: JP13.6, R28.1, T8.C
- new net N$43: JP13.8, R29.2, T9.C
- new net PH0: C14.2, Q1.1, U$1G$1.PH0/OSC_IN
- new net PH1: R2.2, U$1G$1.PH1/OSC_OUT
- new net SCK_SPI2: TP23.TP, U$1G$3.PB13/SPI2_SCK_USART3_CTS_CAN2_TX
- new net SD_CARD_CMD: SV13.4, U$1G$4.PD2/UART5_RX
- new net SD_CARD_DAT0: SV13.3, U$1G$3.PC8/USART6_CK
- new net SD_CARD_SCK: SV13.5, U$1G$4.PC12/UART5_TX/SPI3_MOSI/USART3_CK
- new net V_CIRCUIT: S2A.S, S2B.S, U$3.VIN
- net 12V: now also C18.+, R7.1, SV10.7, SV10.8, U$4.VOUT; no longer 12V.P$1, R24.1, SV14.4
- net 3.3V: now also JP12.7, JP12.8, R24.1, R3.1, R4.1, R5.1, R6.1, S10A.S, S10B.S, S7A.S, S7B.S, S8A.S, S8B.S, S9A.S, S9B.S, SV13.2, TP20.TP, TP4.TP; no longer M1.VCC, Q1.E, R1.1, R12.2, R16.1, R17.1, R18.1, R19.1, SV2.1, SV6.6, U$2.VDD
- net 5V: now also R12.2, R26.2, R27.2, R29.1, SV14.3, T1.C, U$3.VOUT; no longer 5V.P$1, JP11.1, R11.1, R20.2, R21.2, R22.2, R23.1
- net 5VM: now also SV1.5, SV16.11, SV16.12; no longer JP1.4, SV9.6
- net 5VM2: now also SV2.5, SV6.11, SV6.12; no longer JP5.4, SV11.6
- net 5VM3: now also SV18.11, SV18.12, SV8.5; no longer JP2.4, SV3.6
- net 5VM4: now also SV17.11, SV17.12, SV5.5; no longer JP7.4, SV7.6
- net 5VM5: now also SV10.11, SV10.12, SV4.5; no longer JP9.4, SV14.6
- net A_1: now also SV16.19, SV16.20; no longer SV9.10
- net A_2: now also SV6.19, SV6.20; no longer SV11.10
- net A_3: now also SV18.19, SV18.20; no longer SV3.10
- net A_4: now also SV17.19, SV17.20; no longer SV7.10
- net A_5: now also SV10.19, SV10.20; no longer SV14.10
- net BATT_LEVEL: now also U$2.NO, U$5.S; no longer U$3.S, U3.A, U3.~A
- net BOT_COLOR: now also S10A.P, S10B.P, U$1G$1.PE2; no longer SW1.1, U$1G$1.PE5
- net B_1: now also SV16.23, SV16.24; no longer SV9.12
- net B_2: now also SV6.23, SV6.24; no longer SV11.12
- net B_3: now also SV18.23, SV18.24; no longer SV3.12
- net B_4: now also SV17.23, SV17.24; no longer SV7.12
- net B_5: now also SV10.23, SV10.24; no longer SV14.12
- net CE: now also TP5.TP; no longer M1.CE
- net CSN: now also TP6.TP; no longer M1.CSN
- net DIN1_1: now also SV9.7, SV9.8; no longer SV10.4
- net DIN1_2: now also SV3.7, SV3.8; no longer SV12.4
- net DIN1_3: now also SV11.7, SV11.8; no longer SV4.4
- net DIN1_4: now also SV12.7, SV12.8; no longer SV8.4
- net DIN1_5: now also SV7.7, SV7.8; no longer SV15.4
- net DIN2_1: now also SV9.5, SV9.6; no longer SV10.3
- net DIN2_2: now also SV3.5, SV3.6; no longer SV12.3
- net DIN2_3: now also SV11.5, SV11.6; no longer SV4.3
- net DIN2_4: now also SV12.5, SV12.6; no longer SV8.3
- net DIN2_5: now also SV7.5, SV7.6; no longer SV15.3
- net DIN3_1: now also SV9.3, SV9.4; no longer SV10.2
- net DIN3_2: now also SV3.3, SV3.4; no longer SV12.2
- net DIN3_3: now also SV11.3, SV11.4; no longer SV4.2
- net DIN3_4: now also SV12.3, SV12.4; no longer SV8.2
- net DIN3_5: now also SV7.3, SV7.4; no longer SV15.2
- net DIN4_1: now also SV9.1, SV9.2; no longer SV10.1
- net DIN4_2: now also SV3.1, SV3.2; no longer SV12.1
- net DIN4_3: now also SV11.1, SV11.2; no longer SV4.1
- net DIN4_4: now also SV12.1, SV12.2, U$1G$3.PA10/USART1_RX; no longer SV8.1, U$1G$3.PC8/USART6_CK
- net DIN4_5: now also SV7.1, SV7.2, U$1G$3.PA11/USART1_CTS/CAN1_RX/OTG_FS_D-; no longer SV15.1, U$1G$3.PC9/I2C3_SDA
- net GND: now also 12V.C, 3.3V.C, 5V.C, BATTERY.C, C14.1, C15.1, C16.-, C17.-, C18.-, C19.-, C20.-, D2.A, JP12.3, JP12.4, JP13.10, JP6.4, S10A.O, S10B.O, S7A.O, S7B.O, S8A.O, S8B.O, S9A.O, S9B.O, SV1.4, SV10.10, SV10.9, SV11.10, SV11.9, SV12.10, SV12.9, SV13.1, SV14.1, SV16.10, SV16.9, SV17.10, SV17.9, SV18.10, SV18.9, SV2.4, SV3.10, SV3.9, SV4.4, SV5.4, SV6.10, SV6.9, SV7.10, SV7.9, SV8.4, SV9.10, SV9.9, TESTLED1.C, TESTLED2.C, TP19.TP, TP3.TP, U$2.2, U$3.GND, U$3.GNDO, U$4.GND, U$4.GNDO; no longer GND.P$1, GND2.P$1, GND_12V.P$1, GND_5V.P$1, JP11.3, JP6.2, LED8.C, LED9.C, LED_12V.C, LED_3.3V.C, LED_5V.C, LED_8V.C, M1.GND, R26.2, SV1.5, SV10.5, SV11.5, SV12.5, SV14.5, SV15.5, SV2.2, SV3.5, SV4.5, SV6.5, SV7.5, SV8.5, SV9.5, SW1.5, SW1.6, SW1.7, SW1.8, U$2.GND, U$4.5
- net H1_1: now also SV1.3, SV16.13, SV16.14; no longer JP1.6, SV9.7
- net H1_2: now also SV2.3, SV6.13, SV6.14; no longer JP5.6, SV11.7
- net H1_3: now also SV18.13, SV18.14, SV8.3; no longer JP2.6, SV3.7
- net H1_4: now also SV17.13, SV17.14, SV5.3; no longer JP7.6, SV7.7
- net H1_5: now also SV10.13, SV10.14, SV4.3; no longer JP9.6, SV14.7
- net H2_1: now also SV1.2, SV16.15, SV16.16; no longer JP1.7, SV9.8
- net H2_2: now also SV2.2, SV6.15, SV6.16; no longer JP5.7, SV11.8
- net H2_3: now also SV18.15, SV18.16, SV8.2; no longer JP2.7, SV3.8
- net H2_4: now also SV17.15, SV17.16, SV5.2; no longer JP7.7, SV7.8
- net H2_5: now also SV10.15, SV10.16, SV4.2; no longer JP9.7, SV14.8
- net H3_1: now also SV1.1, SV16.17, SV16.18; no longer JP1.8, SV9.9
- net H3_2: now also SV2.1, SV6.17, SV6.18; no longer JP5.8, SV11.9
- net H3_3: now also SV18.17, SV18.18, SV8.1; no longer JP2.8, SV3.9
- net H3_4: now also SV17.17, SV17.18, SV5.1; no longer JP7.8, SV7.9
- net H3_5: now also SV10.17, SV10.18, SV4.1; no longer JP9.8, SV14.9
- net ID_0: now also S9A.P, S9B.P, U$1G$1.PE3; no longer SW1.2, U$1G$1.PE4
- net ID_1: now also S8A.P, S8B.P, U$1G$1.PE4; no longer SW1.3, U$1G$1.PE3
- net ID_2: now also S7A.P, S7B.P, U$1G$1.PE5; no longer SW1.4, U$1G$1.PE2
- net IRQ: now also TP10.TP; no longer M1.IRQ, U$1G$1.PC13/RTC_AF1
- net M1_1: now also SV1.8, SV16.1, SV16.2; no longer JP1.1, SV9.1
- net M1_2: now also SV2.8, SV6.1, SV6.2; no longer JP5.1, SV11.1
- net M1_3: now also SV18.1, SV18.2, SV8.8; no longer JP2.1, SV3.1
- net M1_4: now also SV17.1, SV17.2, SV5.8; no longer JP7.1, SV7.1
- net M1_5: now also SV10.1, SV10.2, SV4.8; no longer JP9.1, SV14.1
- net M2_1: now also SV1.7, SV16.3, SV16.4; no longer JP1.2, SV9.2
- net M2_2: now also SV2.7, SV6.3, SV6.4; no longer JP5.2, SV11.2
- net M2_3: now also SV18.3, SV18.4, SV8.7; no longer JP2.2, SV3.2
- net M2_4: now also SV17.3, SV17.4, SV5.7; no longer JP7.2, SV7.2
- net M2_5: now also SV10.3, SV10.4, SV4.7; no longer JP9.2, SV14.2
- net M3_1: now also SV1.6, SV16.5, SV16.6; no longer JP1.3, SV9.3
- net M3_2: now also SV2.6, SV6.5, SV6.6; no longer JP5.3, SV11.3
- net M3_3: now also SV18.5, SV18.6, SV8.6; no longer JP2.3, SV3.3
- net M3_4: now also SV17.5, SV17.6, SV5.6; no longer JP7.3, SV7.3
- net M3_5: now also SV10.5, SV10.6, SV4.6; no longer JP9.3, SV14.3
- net MISO: now also TP9.TP, U$1G$4.PB4/NJTRST/SPI3_MISO/SPI1_MISO; no longer M1.MISO, U$1G$4.PC11/UART4_RX/SPI3_MISO/USART3_RX, U$2.DOUT
- net MOSI: now also TP8.TP, U$1G$4.PB5/I2C1_SMBA/CAN2_RX/SPI1_MOSI/SPI3_MOSI; no longer M1.MOSI, U$1G$4.PC12/UART5_TX/SPI3_MOSI/USART3_CK
- net N$10: now also C15.2, Q1.2, R2.1; no longer Q1.B, R12.1, R8.2
- net N$12: now also 5V.A, R12.1; no longer D3.A, U$2.DIN
- net N$13: now also J1.+, U$2.C, U$5.P, U3.A, U3.~A; no longer LED1.A, R11.2
- net N$14: now also 12V.A, R7.2; no longer LED_12V.A, R24.2
- net N$15: now also SV13.6; no longer LED_8V.A, R29.1
- net N$18: now also BATTERY.A, R14.2; no longer LED_5V.A, R28.1
- net N$19: now also 3.3V.A; no longer LED_3.3V.A
- net N$2: now also TESTLED2.A; no longer LED9.A
- net N$21: now also R1.2, T1.B; no longer R18.2, T3.B
- net N$22: now also D2.C, T1.E, U$2.1; no longer U$1G$4.PB5/I2C1_SMBA/CAN2_RX/SPI1_MOSI/SPI3_MOSI
- net N$24: now also TP26.TP; no longer U$1G$3.PA8/USART1_CK/I2C3_SCL
- net N$25: now also S2A.P, S2B.P, U3.K; no longer R17.2, T2.B
- net N$9: now also TESTLED1.A; no longer LED8.A
- net NRST: now also JP12.2, R6.2; no longer R1.2, SV6.4
- net SCK: now also TP7.TP, U$1G$4.PB3/JTDO/TRACESWO/SPI3_SCK/SPI1_SCK; no longer D3.C, M1.SCK, U$1G$4.PC10/SPI3_SCK/UART4_TX/USART3_CK
- net SWCLK: now also JP12.5; no longer SV6.2
- net SWDIO: now also JP12.1; no longer SV6.1
- net VDC_1: now also C16.+, C17.+, R14.1, SV16.7, SV16.8, SV6.7, SV6.8, U$4.VIN; no longer SV7.4, SV9.4
- net VDC_2: now also C19.+, C20.+, SV17.7, SV17.8, SV18.7, SV18.8, U2.K; no longer SV11.4, SV3.4, U3.K
- net ~A_1: now also SV16.21, SV16.22; no longer SV9.11
- net ~A_2: now also SV6.21, SV6.22; no longer SV11.11
- net ~A_3: now also SV18.21, SV18.22; no longer SV3.11
- net ~A_4: now also SV17.21, SV17.22; no longer SV7.11
- net ~A_5: now also SV10.21, SV10.22; no longer SV14.11
- net ~B_1: now also SV16.25, SV16.26; no longer SV9.13
- net ~B_2: now also SV6.25, SV6.26; no longer SV11.13
- net ~B_3: now also SV18.25, SV18.26; no longer SV3.13
- net ~B_4: now also SV17.25, SV17.26; no longer SV7.13
- net ~B_5: now also SV10.25, SV10.26; no longer SV14.13
Other:
- note added: "CRYSTAL"
- note added: "IR SENSOR"
- note added: "NRF24L01+ receiver"
- note added: "NRF24L01+ transmitter"
- note added: "POWER SUPPLY"
- note added: "Power Supply 5V"
- note added: "SD CARD MODULE"
- note removed: "IMU MPU6050"
- note removed: "NRF24L01+"
- note removed: "POWER SUPPLY 5v"
- note removed: "Proximity"
- note removed: "USB MICRO"
- note removed: "X-Bee"
- moved on the sheet: C1, C10, C11, C12, C13, C2, C3, C4, C5, C6, C69, C7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
